File: ElectricalSchematics/IGCV/IGVC Controller v1.9.brd (EAGLE design)
At the start: 130 x 118.6 mm, 268 parts, among them IC14 ATMEGA2560-16AU, IC2 IC_FT230X-SSOP-16, K1 G5V-2, T3 TIP122TO220V, T4 TIP122TO220V, T5 TIP122TO220V, T6 TIP122TO220V, T7 TIP122TO220V, T8 TIP122TO220V, U1 TPS54540, U2 LM25119_RTV_32, Y1 CSTCE16M0V53-R0 16MHZ

Commit message: updated eagle
Parts:
- removed C34, C9: 0.1uF, rcl:C0603
- removed STEERL_SENSE: (no value), con-amp-quick:02P
- added STEER_SENSE: (no value), con-amp-quick:03P
- added SV1, SV2, SV7, SV8: GND, con-lstb:MA04-2
- added SV10, SV9: B_+36V, con-lstb:MA04-2
- added SV11, SV12: +24V, con-lstb:MA04-2
- added SV3, SV4: B_+12V, con-lstb:MA04-2
- added SV5, SV6: +12V, con-lstb:MA04-2
- B_+12V, B_+36V: value (none) -> 432550059; device con-amp-quick:03P -> custom:432550059
- IC14: device SmartPrj:TQFP100 -> SmartPrj2:TQFP100
- moved RFBT 101.8 mm to (148.8, 119.4), turned to 180 degrees
- moved RFBB 96.3 mm to (150.6, 117.1), turned to 180 degrees
- moved RCOMP 95.2 mm to (146.7, 115.0), turned to 0 degrees
- moved RT 94.4 mm to (154.2, 117.1), turned to 0 degrees
- moved CCOMP 91.3 mm to (145.3, 112.3), turned to 270 degrees
- moved CCOMP2 89.4 mm to (147.6, 112.3), turned to 270 degrees
- moved U1 84.1 mm to (152.4, 111.3), turned to 180 degrees
- moved CIN_B 79.1 mm to (157.7, 110.2), turned to 270 degrees
- moved CCOMP1 75.5 mm to (155.4, 107.7), turned to 270 degrees
- moved L1_B 73.4 mm to (148.1, 89.9), turned to 0 degrees
- moved D2 71.6 mm to (150.1, 103.6), turned to 180 degrees
- moved COUT 62.1 mm to (157.7, 101.6), turned to 90 degrees
- moved B_+12V 62.0 mm to (108.0, 95.2), turned to 0 degrees
- moved C26 57.8 mm to (178.3, 31.5)
- moved C27 57.8 mm to (181.6, 33.8)
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Connections:
- net N$39 renamed +3.3V
- removed net N$12: STEERL_SENSE.2
- net +12V: now also SV5.1, SV5.2, SV5.3, SV5.4, SV5.5, SV5.6, SV5.7, SV5.8, SV6.1, SV6.2, SV6.3, SV6.4, SV6.5, SV6.6, SV6.7, SV6.8
- net +24V: now also SV11.1, SV11.2, SV11.3, SV11.4, SV11.5, SV11.6, SV11.7, SV11.8, SV12.1, SV12.2, SV12.3, SV12.4, SV12.5, SV12.6, SV12.7, SV12.8
- net +5V: now also STEER_SENSE.1
- net B_+12V: now also SV3.1, SV3.2, SV3.3, SV3.4, SV3.5, SV3.6, SV3.7, SV3.8, SV4.1, SV4.2, SV4.3, SV4.4, SV4.5, SV4.6, SV4.7, SV4.8; no longer B_+12V.2, C9.1
- net B_+36V: now also B_+36V.1, SV10.1, SV10.2, SV10.3, SV10.4, SV10.5, SV10.6, SV10.7, SV10.8, SV9.1, SV9.2, SV9.3, SV9.4, SV9.5, SV9.6, SV9.7, SV9.8; no longer B_+36V.2, B_+36V.3, C34.2
- net GND: now also B_+12V.2, B_+36V.2, STEER_SENSE.3, SV1.1, SV1.2, SV1.3, SV1.4, SV1.5, SV1.6, SV1.7, SV1.8, SV2.1, SV2.2, SV2.3, SV2.4, SV2.5, SV2.6, SV2.7, SV2.8, SV7.1, SV7.2, SV7.3, SV7.4, SV7.5, SV7.6, SV7.7, SV7.8, SV8.1, SV8.2, SV8.3, SV8.4, SV8.5, SV8.6, SV8.7, SV8.8; no longer B_+12V.3, B_+36V.1, C34.1, C9.2
- net STEER_ENCODER: now also STEER_SENSE.2; no longer STEERL_SENSE.1
Routing:
- net GND: track 617.8 -> 954.8 mm, vias 52 -> 51
- net +12V: track 106.4 -> 352.1 mm, vias 5 -> 9
- net +24V: track 301.9 -> 406.5 mm, vias 22 -> 19
- net B_+12V: track 30.2 -> 127.3 mm, vias 1 -> 0
- net B_+36V: track 191.3 -> 250.5 mm, vias 21 -> 17
- net N$76: track 8.89 -> 0.00 mm
- net RESET: track 100.5 -> 92.6 mm
- net I2C_SCL: track 66.6 -> 73.3 mm, vias 2 -> 1
- net I2C_SDA: track 68.3 -> 74.4 mm, vias 2 -> 1
- net BRAKE_IN: track 114.2 -> 118.7 mm
- net USART_RX0: track 92.3 -> 88.2 mm
- net BRAKE_OUT: track 108.0 -> 111.3 mm
- net HALL_2: track 107.3 -> 110.2 mm
- net USART_TX0: track 93.5 -> 90.8 mm
- net HALL_1: track 99.2 -> 101.7 mm
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Other:
- board size 130 x 118.6 mm -> 200.2 x 122.9 mm
- board text added: "+ -"
- board text added: "+12V GND"
- board text added: "+36V GND"
- board text added: "- - -"
- board text added: "1 2 - W +"
- board text added: "12 -"
- board text added: "24 -"
- board text added: "5 -"
- board text added: "BRAKE IN"
- board text added: "BRAKE OUT"
- board text added: "Cal Poly Robotics IGVC Controller Board v1.9 Justin Ng April 8, 2014"
- board text added: "DPOT EN"
- board text added: "ESTOP SENSE"
- board text added: "F R"
- board text added: "FL FR"
- board text added: "HALL LEFT"
- board text added: "HALL RIGHT"
- board text added: "IN"
- board text added: "LIGHT"
- board text added: "OUT"
- board text added: "POT HIGH"
- board text added: "POT WIPER"
- board text added: "RL"
- board text added: "RR"
- board text added: "STEER"
- board text added: "THROT POT"
- board text added: "THROT1"
- board text added: "THROT2"
- board text added: "TX3 RX3"
- board text added: "USART"
- board text removed: "B_+12V B_+12V GND GND B_+36V B_+36V"
- board text removed: "FRONT OF CART"
- board text removed: "LEFT OF CART"
- board text removed: "OUT IN"
- board text removed: "REAR OF CART"
- board text removed: "RIGHT OF CART"
- board text removed: "THROTPOT"
