File: ElectricalSchematics/IGCV/IGVC Controller v1.9.sch (EAGLE design)
At the start: 268 parts, among them IC14 ATMEGA2560-16AU, IC2 IC_FT230X-SSOP-16, K1 G5V-2, T3 TIP122TO220V, T4 TIP122TO220V, T5 TIP122TO220V, T6 TIP122TO220V, T7 TIP122TO220V, T8 TIP122TO220V, U1 TPS54540, U2 LM25119_RTV_32, Y1 CSTCE16M0V53-R0 16MHZ

Commit message: updated eagle
Parts:
- removed C34, C9: 0.1uF, rcl:C-EUC0603
- removed STEERL_SENSE: (no value), con-amp-quick:M02
- added STEER_SENSE: (no value), con-amp-quick:M03
- added SV1, SV2, SV7, SV8: GND, con-lstb:MA04-2
- added SV10, SV9: B_+36V, con-lstb:MA04-2
- added SV11, SV12: +24V, con-lstb:MA04-2
- added SV3, SV4: B_+12V, con-lstb:MA04-2
- added SV5, SV6: +12V, con-lstb:MA04-2
- B_+12V, B_+36V: value (none) -> 432550059; device con-amp-quick:M03 -> custom:432550059
- IC14: device SmartPrj:ATMEGA25602560-16AU -> SmartPrj2:ATMEGA25602560-16AU
Connections:
- net N$39 renamed +3.3V
- removed net N$12: STEERL_SENSE.2
- net +12V: now also SV5.1, SV5.2, SV5.3, SV5.4, SV5.5, SV5.6, SV5.7, SV5.8, SV6.1, SV6.2, SV6.3, SV6.4, SV6.5, SV6.6, SV6.7, SV6.8
- net +24V: now also SV11.1, SV11.2, SV11.3, SV11.4, SV11.5, SV11.6, SV11.7, SV11.8, SV12.1, SV12.2, SV12.3, SV12.4, SV12.5, SV12.6, SV12.7, SV12.8
- net +5V: now also STEER_SENSE.1
- net B_+12V: now also SV3.1, SV3.2, SV3.3, SV3.4, SV3.5, SV3.6, SV3.7, SV3.8, SV4.1, SV4.2, SV4.3, SV4.4, SV4.5, SV4.6, SV4.7, SV4.8; no longer B_+12V.2, C9.1
- net B_+36V: now also B_+36V.1, SV10.1, SV10.2, SV10.3, SV10.4, SV10.5, SV10.6, SV10.7, SV10.8, SV9.1, SV9.2, SV9.3, SV9.4, SV9.5, SV9.6, SV9.7, SV9.8; no longer B_+36V.2, B_+36V.3, C34.2
- net GND: now also B_+12V.2, B_+36V.2, STEER_SENSE.3, SV1.1, SV1.2, SV1.3, SV1.4, SV1.5, SV1.6, SV1.7, SV1.8, SV2.1, SV2.2, SV2.3, SV2.4, SV2.5, SV2.6, SV2.7, SV2.8, SV7.1, SV7.2, SV7.3, SV7.4, SV7.5, SV7.6, SV7.7, SV7.8, SV8.1, SV8.2, SV8.3, SV8.4, SV8.5, SV8.6, SV8.7, SV8.8; no longer B_+12V.3, B_+36V.1, C34.1, C9.2
- net STEER_ENCODER: now also STEER_SENSE.2; no longer STEERL_SENSE.1
Other:
- note added: "Power connectors"
- note removed: "Battery Inputs"
- moved on the sheet: MISC_1, MISC_2, MISC_3
