File: Electrical Schematics/Version2/Schematics/boardv2.sch (EAGLE design)
At the start: 235 parts, among them IC14 ATMEGA2560-16AU, IC2 IC_FT230X-SSOP-16, K1 G5V-2, T3 TIP122TO220V, T4 TIP122TO220V, T5 TIP122TO220V, T6 TIP122TO220V, T7 TIP122TO220V, T8 TIP122TO220V, U3 TMS570LS0432_PZ_100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

Commit message: More Updates
Parts:
- removed U3: TMS570LS0432_PZ_100, roblib:TMS570LS0432_PZ_100
- added U1: TMS570LS0432_PZ_100, version2:TMS570LS0432_PZ_100
Connections:
- net GND: no longer U3.VSS, U3.VSS_10, U3.VSS_9
Changed lines of the file:
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@@
 <?xml version="1.0" encoding="utf-8"?>
 <!DOCTYPE eagle SYSTEM "eagle.dtd">
-<eagle version="7.1.0">
+<eagle version="6.6.0">
 <drawing>
 <settings>
@@
 <part name="R37" library="resistor" deviceset="R-US_" device="R0603" value="27"/>
 <part name="R38" library="resistor" deviceset="R-US_" device="R0603" value="27"/>
-<part name="U3" library="roblib" deviceset="TMS570LS0432_PZ_100" device=""/>
-<part name="SUPPLY4" library="supply2" deviceset="GND" device=""/>
+<part name="U1" library="version2" deviceset="TMS570LS0432_PZ_100" device=""/>
 </parts>
 <sheets>
@@
 </plain>
 <instances>
-<instance part="U3" gate="A" x="22.86" y="81.28"/>
-<instance part="SUPPLY4" gate="GND" x="154.94" y="30.48"/>
+<instance part="U1" gate="A" x="160.02" y="78.74"/>
 </instances>
 <busses>
 </busses>
 <nets>
-<net name="GND" class="0">
-<segment>
-<pinref part="U3" gate="A" pin="VSS"/>
-<wire x1="124.46" y1="81.28" x2="154.94" y2="81.28" width="0.1524" layer="91"/>
-<wire x1="154.94" y1="81.28" x2="154.94" y2="48.26" width="0.1524" layer="91"/>
-<pinref part="U3" gate="A" pin="VSS_10"/>
-<wire x1="154.94" y1="48.26" x2="154.94" y2="45.72" width="0.1524" layer="91"/>
-<wire x1="154.94" y1="45.72" x2="154.94" y2="33.02" width="0.1524" layer="91"/>
-<wire x1="124.46" y1="48.26" x2="154.94" y2="48.26" width="0.1524" layer="91"/>
-<pinref part="U3" gate="A" pin="VSS_9"/>
-<wire x1="124.46" y1="45.72" x2="154.94" y2="45.72" width="0.1524" layer="91"/>
-<pinref part="SUPPLY4" gate="GND" pin="GND"/>
-</segment>
-</net>
 </nets>
 </sheet>
