File: Electrical Schematics/Version2/Schematics/boardv2ftdi.sch (EAGLE design)
At the start: 0 parts

Commit message: Created schematics for USB to mcu com and added isolation
Parts:
- added 24OHM, 24OHMS: (no value), SparkFun-Passives:RESISTOR0603-RES
- added C1, C2, C3, C4: 0.1uF, eagle-ltspice:CC0603
- added C5: 4.7uf, eagle-ltspice:CC0603
- added IC1: ADUM4160BRW, kblom:ADUM4160BRW
- added JP1: USB-B, SparkFun-Connectors:USBPTH
- added L1, L2: BLM15HB121SN1, inductors:BLM15HB121SN1
- added TP1, TP10, TP11, TP12, TP13, TP2, TP3, TP4, TP5, TP6, TP7, TP8, TP9: TPB1,27, testpad:TPB1,27
- added U$1: ACM3225-2P, shit:ACM3225-2P
- added U1: CP2130-GM, shit:CP2130-GM
Connections:
- new net 3.3V: U1.VIO
- new net GND: C1.2, C2.1, C5.2, IC1.GND2@1, IC1.GND2@2, TP5.TP, TP7.TP, U1.EPAD, U1.GND
- new net MCU: TP10.TP, TP11.TP, TP13.TP, TP8.TP, TP9.TP
- new net N$1: IC1.UD-, U$1.P$3
- new net N$10: C1.1, C2.2, IC1.PIN, IC1.SPD, IC1.VBUS2, IC1.VDD2, TP6.TP, U1.REGIN
- new net N$11: 24OHMS.2, TP4.TP
- new net N$12: C4.2, IC1.PDEN, IC1.VDD1
- new net N$13: 24OHM.2, TP3.TP, U1.D+
- new net N$15: C5.1, TP12.TP, U1.VPP
- new net N$2: IC1.UD+, U$1.P$4
- new net N$3: C3.2, C4.1, IC1.GND1@1, IC1.GND1@2, L2.2, TP2.TP
- new net N$4: C3.1, IC1.VBUS1, L1.2, TP1.TP
- new net N$5: U$1.P$1
- new net N$6: 24OHM.1, IC1.DD+
- new net N$7: JP1.D+, U$1.P$2
- new net N$8: 24OHMS.1, IC1.DD-
- new net N$9: JP1.VBUS, L1.1, L2.1
Other:
- note added: "USB Isolation"
- note added: "USB to SPI"
