File: Electrical Schematics/Version2/Schematics/boardv2ftdi.sch (EAGLE design)
At the start: 26 parts, among them IC1 ADUM4160BRW, U1 CP2130-GM

Commit message: updated everything
Other:
- note added: "SPI to USB"
Changed lines of the file:
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@@
 <part name="TP12" library="testpad" deviceset="TP" device="B1,27"/>
 <part name="TP13" library="testpad" deviceset="TP" device="B1,27"/>
+<part name="FRAME1" library="frames" deviceset="DOCFIELD" device=""/>
 </parts>
 <sheets>
@@
 <text x="-91.44" y="71.12" size="1.778" layer="91">USB Isolation</text>
 <text x="81.28" y="81.28" size="1.778" layer="91">USB to SPI</text>
+<frame x1="-187.96" y1="-91.44" x2="302.26" y2="157.48" columns="8" rows="5" layer="91"/>
+<text x="-160.02" y="134.62" size="7.62" layer="91">SPI to USB</text>
 </plain>
 <instances>
@@
 <instance part="TP12" gate="G$1" x="167.64" y="45.72"/>
 <instance part="TP13" gate="G$1" x="15.24" y="68.58"/>
+<instance part="FRAME1" gate="G$1" x="193.04" y="-83.82"/>
 </instances>
 <busses>
-<bus name="MCU">
+<bus name="TOMCU">
 <segment>
 <wire x1="-7.62" y1="104.14" x2="203.2" y2="104.14" width="0.762" layer="92"/>

Commit message: cleaned up the ftdi code
Connections:
- new net N$14: U1.REGIN
- new net N$17: U1.GND
- net GND: no longer U1.GND
- net N$10: no longer U1.REGIN
- net N$11: no longer 24OHMS.2
- net N$12: now also IC1.SPU
- net N$13: no longer 24OHM.2
- net N$5: now also JP1.D-
- net N$9: now also JP1.GND
Other:
- moved on the sheet: 24OHM, 24OHMS, C1, C2, C3, C4, IC1, L1, L2, TP1, TP2, TP3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

Commit message: updated the spi to usb convert file
Parts:
- added 24OHMS1: 600Ohms, SparkFun-Passives:RESISTOR0603-RES
- added 24OHMS3, RES604: 24, SparkFun-Passives:RESISTOR0603-RES
- added C6, C7, C8: 0.1uF, eagle-ltspice:CC0603
- added LED1: (no value), eagle-ltspice:LED_E
- added TP14, TP15, TP16: TPB1,27, testpad:TPB1,27
- added TP17, TP18: TPB2,54, testpad:TPB2,54
- TP10, TP11, TP8, TP9: value TPB1,27 -> TPB2,54; device testpad:TPB1,27 -> testpad:TPB2,54
Connections:
- removed net 3.3V: U1.VIO
- removed net MCU: TP10.TP, TP11.TP, TP13.TP, TP8.TP, TP9.TP
- removed net N$10: C1.1, C2.2, IC1.PIN, IC1.SPD, IC1.VBUS2, IC1.VDD2, TP6.TP
- removed net N$14: U1.REGIN
- removed net N$17: U1.GND
- new net MCU_SPIBRIDGE_CS: TP10.TP
- new net MCU_SPIBRIDGE_CS1: TP11.TP, U1.GPIO.1/*CS1
- new net MCU_SPIBRIDGE_MOSI: TP9.TP, U1.MOSI
- new net MCU_SPIBRIDGE_SCK: TP3.TP, U1.SCK
- new net MCU_USBBRIDGE_MISO: TP8.TP, U1.MISO
- new net N$16: U1.GPIO.0/*CS0
- new net N$18: JP1.VBUS, L1.1
- new net N$21: 24OHMS1.1, U1.GPIO.8/*CS8/SPIACT
- new net N$22: U1.GPIO.7/*CS7
- new net N$23: U1.GPIO.6/*CS6
- new net N$24: 24OHMS1.2, LED1.A
- new net SPIBRIDGE_3.3V: C6.1, C7.1, C8.1, TP15.TP, U1.*RST, U1.VDD
- new net SPIBRIDGE_ISOLATION_D+: 24OHM.2, TP13.TP, U1.D+
- new net SPIBRIDGE_ISOLATION_D-: 24OHMS.2, TP14.TP, U1.D-
- new net SPIBRIDGE_ISOLATION_VBUS: C1.1, C2.2, IC1.PIN, IC1.SPD, IC1.VBUS2, IC1.VDD2, TP16.TP, TP6.TP, U1.VBUS
- net GND: now also C6.2, C7.2, C8.2, LED1.C, TP4.TP, U1.GND
- net N$1: now also RES604.1, TP17.TP; no longer IC1.UD-
- net N$11: now also IC1.UD-, RES604.2; no longer TP4.TP
- net N$13: now also 24OHMS3.1, TP18.TP, U$1.P$4; no longer TP3.TP, U1.D+
- net N$2: now also 24OHMS3.2; no longer U$1.P$4
- net N$9: no longer JP1.VBUS, L1.1
Other:
- note added: "B"
- note added: "CREATED BY MICHAEL ROBERTS"
- moved on the sheet: 24OHM, 24OHMS, TP10, TP11, TP13, TP3, TP4, TP8, TP9

Commit message: updated circuits
Other:
- moved on the sheet: TP4
Changed lines of the file:
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@@
 <instance part="LED1" gate="G$1" x="218.44" y="-17.78"/>
 <instance part="SUPPLY5" gate="GND" x="218.44" y="-30.48"/>
-<instance part="SUPPLY6" gate="GND" x="-101.6" y="43.18"/>
+<instance part="SUPPLY6" gate="GND" x="-83.82" y="58.42"/>
 <instance part="TP3" gate="G$1" x="-38.1" y="68.58"/>
-<instance part="TP4" gate="G$1" x="-38.1" y="48.26"/>
+<instance part="TP4" gate="G$1" x="-43.18" y="63.5"/>
 <instance part="TP13" gate="G$1" x="-30.48" y="43.18"/>
 <instance part="TP14" gate="G$1" x="-25.4" y="35.56"/>
@@
 </segment>
 <segment>
-<pinref part="U1" gate="A" pin="GND"/>
-<wire x1="27.94" y1="63.5" x2="-33.02" y2="63.5" width="0.1524" layer="91"/>
-<wire x1="-33.02" y1="63.5" x2="-33.02" y2="45.72" width="0.1524" layer="91"/>
-<wire x1="-33.02" y1="45.72" x2="-38.1" y2="45.72" width="0.1524" layer="91"/>
-<pinref part="SUPPLY6" gate="GND" pin="GND"/>
-<pinref part="TP4" gate="G$1" pin="TP"/>
-<wire x1="-38.1" y1="45.72" x2="-101.6" y2="45.72" width="0.1524" layer="91"/>
-<junction x="-38.1" y="45.72"/>
-<junction x="27.94" y="63.5"/>
-</segment>
-<segment>
 <pinref part="C6" gate="G$1" pin="2"/>
 <pinref part="C8" gate="G$1" pin="2"/>
@@
 <junction x="2.54" y="38.1"/>
 <junction x="17.78" y="33.02"/>
+</segment>
+<segment>
+<pinref part="U1" gate="A" pin="GND"/>
+<wire x1="27.94" y1="63.5" x2="-27.94" y2="63.5" width="0.1524" layer="91"/>
+<wire x1="-27.94" y1="63.5" x2="-27.94" y2="60.96" width="0.1524" layer="91"/>
+<wire x1="-27.94" y1="60.96" x2="-43.18" y2="60.96" width="0.1524" layer="91"/>
+<pinref part="TP4" gate="G$1" pin="TP"/>
+<wire x1="-43.18" y1="60.96" x2="-83.82" y2="60.96" width="0.1524" layer="91"/>
+<junction x="-43.18" y="60.96"/>
+<pinref part="SUPPLY6" gate="GND" pin="GND"/>
 </segment>
 </net>
@@
 <pinref part="U1" gate="A" pin="SCK"/>
 <wire x1="27.94" y1="66.04" x2="-38.1" y2="66.04" width="0.1524" layer="91"/>
-<wire x1="-38.1" y1="66.04" x2="-40.64" y2="66.04" width="0.1524" layer="91"/>
-<wire x1="-40.64" y1="66.04" x2="-40.64" y2="53.34" width="0.1524" layer="91"/>
-<wire x1="-40.64" y1="53.34" x2="-55.88" y2="53.34" width="0.1524" layer="91"/>
+<wire x1="-38.1" y1="66.04" x2="-55.88" y2="66.04" width="0.1524" layer="91"/>
 <pinref part="TP3" gate="G$1" pin="TP"/>
 <junction x="-38.1" y="66.04"/>
-<label x="-55.88" y="53.34" size="1.778" layer="95" rot="R180" xref="yes"/>
+<label x="-55.88" y="66.04" size="1.778" layer="95" rot="R180" xref="yes"/>
 <junction x="27.94" y="66.04"/>
 </segment>
