File: Electrical Schematics/Version2/Schematics/boardv2FNR.sch (EAGLE design)
At the start: 0 parts

Commit message: FNR
Parts:
- added AMTOG+, AMTOG-, GEARSHIFT_GND, POT_HIGH, POT_WIPER, THROTTLE1, THROTTLE2: (no value), adafruit:PINHD-1X1
- added D5: 1N4004, adafruit:1N4004
- added GS_C, GS_N: N, adafruit:PINHD-1X1
- added GS_F: F, adafruit:PINHD-1X1
- added GS_R: R, adafruit:PINHD-1X1
- added K1: G5V-2, relay:G5V-2
- added LED1: BLUE, adafruit:LED3MM
- added LED2: RED, adafruit:LED3MM
- added LED3: GREEN, adafruit:LED3MM
- added LED4: (no value), adafruit:LED3MM
- added POT_GND: POT_GND, adafruit:PINHD-1X1
- added R1, R13, R15, R16, R17, R4: 150, rcl:R-US_0204/5
- added R14: 10K, rcl:R-US_0204/5
- added R18, R20, R21: 1K, rcl:R-US_0204/5
- added R19: 1k, rcl:R-US_0204/5
- added T3, T4, T5, T6, T7, T8: TIP122TO220V, transistor modified:TIP122TO220V
- added U$19: MCP4131-502E, custom:MCP4131-502E
Connections:
- new net +5V: AMTOG+.1, D5.C, K1A.1, LED4.A, U$19.+5V
- new net AM_TOGGLE-: AMTOG-.1, LED1.A, LED2.A, LED3.A, R13.1, R14.1, R15.1, R17.1
- new net AUTO_SENSE: R14.2
- new net DPOT_ENABLE: R1.2
- new net FGND: GS_F.1, R19.1, T5.C
- new net GEARSHIFT_F: R16.1
- new net GEARSHIFT_R: R4.1
- new net GND: GEARSHIFT_GND.1, GS_C.1, POT_GND.1, U$19.A, U$19.GND
- new net N: GS_N.1, R20.2, T4.E, T6.E, T7.E
- new net N$1: T7.C, T8.E
- new net N$13: LED2.C, R18.2
- new net N$14: LED3.C, R19.2
- new net N$17: LED4.C, R21.1
- new net N$18: R13.2, T3.B
- new net N$19: R4.2, T4.B
- new net N$2: R1.1, T8.B
- new net N$20: R15.2, T5.B
- new net N$21: R16.2, T6.B
- new net N$22: T5.E, T6.C
- new net N$23: R17.2, T7.B
- new net N$5: T3.E, T4.C
- new net N$51: K12.S, U$19.B
- new net N$52: K11.S, U$19.W
- new net N$57: D5.A, K1A.2, R21.2, T8.C
- new net N$8: LED1.C, R20.1
- new net POT_HIGH: K12.O, POT_HIGH.1
- new net POT_WIPER: K11.O, POT_WIPER.1
- new net RGND: GS_R.1, R18.1, T3.C
- new net SPI_MOSI: U$19.MOSI
- new net SPI_SCK: U$19.SCK
- new net SPI_SS: U$19.SS
- new net THROTTLE1: K12.P, THROTTLE1.1
- new net THROTTLE2: K11.P, THROTTLE2.1
Other:
- note added: "AUTO/MANUAL TOGGLE"
- note added: "DP pin out: 1. SPI-CS 2. SPI-SCK 3. SPI-SDIO 4. GND 5. Pot A terminal 6. Pot wiper 7. Pot B terminal 8. Vcc"
- note added: "F"
- note added: "Gearshift"
- note added: "R"
- note added: "R N F"
- note added: "Solid-state FNR controller v1.5"
- note added: "Throttle Controller v1.3"
