File: Electrical Schematics/Version2/Schematics/boardv2FNR.sch (EAGLE design)
At the start: 36 parts, among them K1 G5V-2, T3 TIP122TO220V, T4 TIP122TO220V, T5 TIP122TO220V, T6 TIP122TO220V, T7 TIP122TO220V, T8 TIP122TO220V

Commit message: updated everything
Other:
- note added: "FNR Block"
Changed lines of the file:
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@@
 <part name="U$19" library="custom" deviceset="MCP4131-502E" device=""/>
 <part name="GS_C" library="adafruit" deviceset="PINHD-1X1" device="" value="N"/>
+<part name="FRAME1" library="frames" deviceset="DOCFIELD" device=""/>
 </parts>
 <sheets>
@@
 <text x="30.48" y="66.04" size="1.778" layer="97">F</text>
 <rectangle x1="116.84" y1="2.54" x2="132.08" y2="48.26" layer="97"/>
+<frame x1="-60.96" y1="-63.5" x2="269.24" y2="111.76" columns="8" rows="5" layer="91"/>
+<text x="-48.26" y="101.6" size="5.08" layer="91">FNR Block</text>
 </plain>
 <instances>
@@
 <attribute name="NAME" x="85.598" y="34.671" size="1.778" layer="95"/>
 </instance>
+<instance part="FRAME1" gate="G$1" x="162.56" y="-60.96"/>
 </instances>
 <busses>

Commit message: FNR except digipot
Parts:
- removed T3, T4, T5, T6, T7, T8: TIP122TO220V, transistor modified:TIP122TO220V
- added Q1, Q2, Q3, Q4, Q5, Q6: IRLML2060TRPBFBSS123LT1G, SparkFun-DiscreteSemi:IRLML2060TRPBFBSS123LT1G
Connections:
- removed net N$19: R4.2, T4.B
- removed net N$20: R15.2, T5.B
- removed net N$21: R16.2, T6.B
- new net N$3: Q2.G, R4.2
- new net N$4: Q3.G, R15.2
- new net N$6: Q4.G, R16.2
- net FGND: now also Q3.S; no longer T5.C
- net N: now also Q2.D, Q4.D, Q5.D; no longer T4.E, T6.E, T7.E
- net N$1: now also Q5.S, Q6.D; no longer T7.C, T8.E
- net N$18: now also Q1.G; no longer T3.B
- net N$2: now also Q6.G; no longer T8.B
- net N$22: now also Q3.D, Q4.S; no longer T5.E, T6.C
- net N$23: now also Q5.G; no longer T7.B
- net N$5: now also Q1.D, Q2.S; no longer T3.E, T4.C
- net N$57: now also Q6.S; no longer T8.C
- net RGND: now also Q1.S; no longer T3.C
Changed lines of the file:
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@@
 <part name="LED4" library="adafruit" deviceset="LED" device="3MM"/>
 <part name="R21" library="rcl" deviceset="R-US_" device="0204/5" value="1K"/>
-<part name="T3" library="transistor modified" deviceset="TIP122" device="TO220V"/>
-<part name="T4" library="transistor modified" deviceset="TIP122" device="TO220V"/>
-<part name="T5" library="transistor modified" deviceset="TIP122" device="TO220V"/>
-<part name="T6" library="transistor modified" deviceset="TIP122" device="TO220V"/>
-<part name="T7" library="transistor modified" deviceset="TIP122" device="TO220V"/>
-<part name="T8" library="transistor modified" deviceset="TIP122" device="TO220V"/>
 <part name="GS_R" library="adafruit" deviceset="PINHD-1X1" device="" value="R"/>
 <part name="GS_N" library="adafruit" deviceset="PINHD-1X1" device="" value="N"/>
@@
 <part name="GS_C" library="adafruit" deviceset="PINHD-1X1" device="" value="N"/>
 <part name="FRAME1" library="frames" deviceset="DOCFIELD" device=""/>
+<part name="Q1" library="SparkFun-DiscreteSemi" deviceset="IRLML2060TRPBF" device="BSS123LT1G"/>
+<part name="Q2" library="SparkFun-DiscreteSemi" deviceset="IRLML2060TRPBF" device="BSS123LT1G"/>
+<part name="Q3" library="SparkFun-DiscreteSemi" deviceset="IRLML2060TRPBF" device="BSS123LT1G"/>
+<part name="Q4" library="SparkFun-DiscreteSemi" deviceset="IRLML2060TRPBF" device="BSS123LT1G"/>
+<part name="Q5" library="SparkFun-DiscreteSemi" deviceset="IRLML2060TRPBF" device="BSS123LT1G"/>
+<part name="Q6" library="SparkFun-DiscreteSemi" deviceset="IRLML2060TRPBF" device="BSS123LT1G"/>
 </parts>
 <sheets>
@@
 <attribute name="VALUE" x="123.19" y="61.722" size="1.778" layer="96" rot="R180"/>
 </instance>
-<instance part="T3" gate="G$1" x="-12.7" y="48.26" rot="MR270"/>
-<instance part="T4" gate="G$1" x="2.54" y="48.26" rot="MR270"/>
-<instance part="T5" gate="G$1" x="15.24" y="48.26" rot="MR270"/>
-<instance part="T6" gate="G$1" x="30.48" y="48.26" rot="MR270"/>
-<instance part="T7" gate="G$1" x="48.26" y="48.26" rot="R270"/>
-<instance part="T8" gate="G$1" x="116.84" y="78.74" rot="R180"/>
 <instance part="GS_R" gate="G$1" x="63.5" y="35.56" smashed="yes" rot="R180">
 <attribute name="NAME" x="70.358" y="37.465" size="1.778" layer="95"/>
@@
 </instance>
 <instance part="FRAME1" gate="G$1" x="162.56" y="-60.96"/>
+<instance part="Q1" gate="G$1" x="-10.16" y="43.18" rot="R270"/>
+<instance part="Q2" gate="G$1" x="5.08" y="43.18" rot="R270"/>
+<instance part="Q3" gate="G$1" x="17.78" y="43.18" rot="R270"/>
+<instance part="Q4" gate="G$1" x="33.02" y="43.18" rot="R270"/>
+<instance part="Q5" gate="G$1" x="45.72" y="43.18" rot="MR270"/>
+<instance part="Q6" gate="G$1" x="111.76" y="81.28" rot="MR0"/>
 </instances>
 <busses>
@@
 <junction x="-15.24" y="35.56"/>
 <pinref part="R18" gate="G$1" pin="1"/>
-<pinref part="T3" gate="G$1" pin="C"/>
 <pinref part="GS_R" gate="G$1" pin="1"/>
 <wire x1="60.96" y1="35.56" x2="66.04" y2="35.56" width="0.1524" layer="91"/>
+<pinref part="Q1" gate="G$1" pin="S"/>
 </segment>
 </net>
@@
 <pinref part="R19" gate="G$1" pin="1"/>
 <wire x1="-15.24" y1="25.4" x2="12.7" y2="25.4" width="0.1524" layer="91" style="shortdash"/>
-<pinref part="T5" gate="G$1" pin="C"/>
 <pinref part="GS_F" gate="G$1" pin="1"/>
 <wire x1="60.96" y1="25.4" x2="66.04" y2="25.4" width="0.1524" layer="91"/>
+<pinref part="Q3" gate="G$1" pin="S"/>
 </segment>
 </net>
@@
 <wire x1="58.42" y1="50.8" x2="58.42" y2="30.48" width="0.1524" layer="91"/>
 <junction x="58.42" y="30.48"/>
-<pinref part="T4" gate="G$1" pin="E"/>
-<pinref part="T6" gate="G$1" pin="E"/>
-<pinref part="T7" gate="G$1" pin="E"/>
 <wire x1="40.64" y1="43.18" x2="40.64" y2="30.48" width="0.1524" layer="91"/>
 <pinref part="GS_N" gate="G$1" pin="1"/>
 <wire x1="60.96" y1="30.48" x2="66.04" y2="30.48" width="0.1524" layer="91"/>
+<pinref part="Q2" gate="G$1" pin="D"/>
+<pinref part="Q4" gate="G$1" pin="D"/>
+<pinref part="Q5" gate="G$1" pin="D"/>
 </segment>
 </net>
@@
 <wire x1="53.34" y1="93.98" x2="111.76" y2="93.98" width="0.1524" layer="91"/>
 <wire x1="111.76" y1="93.98" x2="111.76" y2="86.36" width="0.1524" layer="91"/>
-<pinref part="T7" gate="G$1" pin="C"/>
 <wire x1="50.8" y1="43.18" x2="53.34" y2="43.18" width="0.1524" layer="91"/>
 <wire x1="53.34" y1="43.18" x2="53.34" y2="93.98" width="0.1524" layer="91"/>
-<pinref part="T8" gate="G$1" pin="E"/>
+<pinref part="Q5" gate="G$1" pin="S"/>
+<pinref part="Q6" gate="G$1" pin="D"/>
 </segment>
 </net>
@@
 <net name="N$5" class="0">
 <segment>
-<pinref part="T3" gate="G$1" pin="E"/>
 <wire x1="-5.08" y1="43.18" x2="0" y2="43.18" width="0.1524" layer="91"/>
-<pinref part="T4" gate="G$1" pin="C"/>
+<pinref part="Q1" gate="G$1" pin="D"/>
+<pinref part="Q2" gate="G$1" pin="S"/>
 </segment>
 </net>
@@
 <wire x1="116.84" y1="63.5" x2="111.76" y2="63.5" width="0.1524" layer="91"/>
 <junction x="111.76" y="63.5"/>
-<pinref part="T8" gate="G$1" pin="C"/>
 <wire x1="111.76" y1="76.2" x2="111.76" y2="63.5" width="0.1524" layer="91"/>
 <pinref part="K1" gate="A" pin="2"/>
+<pinref part="Q6" gate="G$1" pin="S"/>
 </segment>
 </net>
@@
 <net name="N$18" class="0">
 <segment>
-<pinref part="T3" gate="G$1" pin="B"/>
 <pinref part="R13" gate="G$1" pin="2"/>
 <wire x1="-12.7" y1="60.96" x2="-12.7" y2="50.8" width="0.1524" layer="91"/>
-</segment>
-</net>
-<net name="N$19" class="0">
-<segment>
-<pinref part="R4" gate="G$1" pin="2"/>
-<pinref part="T4" gate="G$1" pin="B"/>
-</segment>
-</net>
-<net name="N$20" class="0">
-<segment>
-<pinref part="T5" gate="G$1" pin="B"/>
-<pinref part="R15" gate="G$1" pin="2"/>
-</segment>
-</net>
-<net name="N$21" class="0">
-<segment>
-<pinref part="R16" gate="G$1" pin="2"/>
-<pinref part="T6" gate="G$1" pin="B"/>
+<wire x1="-12.7" y1="50.8" x2="-10.16" y2="50.8" width="0.1524" layer="91"/>
+<pinref part="Q1" gate="G$1" pin="G"/>
 </segment>
 </net>
 <net name="N$22" class="0">
 <segment>
-<pinref part="T6" gate="G$1" pin="C"/>
-<pinref part="T5" gate="G$1" pin="E"/>
 <wire x1="27.94" y1="43.18" x2="22.86" y2="43.18" width="0.1524" layer="91"/>
+<pinref part="Q3" gate="G$1" pin="D"/>
+<pinref part="Q4" gate="G$1" pin="S"/>
 </segment>
 </net>
@@
 <segment>
 <pinref part="R17" gate="G$1" pin="2"/>
-<pinref part="T7" gate="G$1" pin="B"/>
 <wire x1="48.26" y1="53.34" x2="48.26" y2="50.8" width="0.1524" layer="91"/>
-<junction x="48.26" y="50.8"/>
+<wire x1="45.72" y1="50.8" x2="48.26" y2="50.8" width="0.1524" layer="91"/>
+<pinref part="Q5" gate="G$1" pin="G"/>
 </segment>
 </net>
@@
 <net name="N$2" class="0">
 <segment>
-<pinref part="T8" gate="G$1" pin="B"/>
 <pinref part="R1" gate="G$1" pin="1"/>
 <wire x1="119.38" y1="78.74" x2="121.92" y2="78.74" width="0.1524" layer="91"/>
+<wire x1="119.38" y1="78.74" x2="119.38" y2="81.28" width="0.1524" layer="91"/>
+<pinref part="Q6" gate="G$1" pin="G"/>
 </segment>
 </net>
@@
 </segment>
 </net>
+<net name="N$3" class="0">
+<segment>
+<pinref part="R4" gate="G$1" pin="2"/>
+<wire x1="2.54" y1="50.8" x2="5.08" y2="50.8" width="0.1524" layer="91"/>
+<pinref part="Q2" gate="G$1" pin="G"/>
+</segment>
+</net>
+<net name="N$4" class="0">
+<segment>
+<pinref part="R15" gate="G$1" pin="2"/>
+<wire x1="15.24" y1="50.8" x2="17.78" y2="50.8" width="0.1524" layer="91"/>
+<pinref part="Q3" gate="G$1" pin="G"/>
+</segment>
+</net>
+<net name="N$6" class="0">
+<segment>
+<pinref part="R16" gate="G$1" pin="2"/>
+<wire x1="30.48" y1="50.8" x2="33.02" y2="50.8" width="0.1524" layer="91"/>
+<pinref part="Q4" gate="G$1" pin="G"/>
+</segment>
+</net>

Commit message: FNR with digipot
Parts:
- removed U$19: MCP4131-502E, custom:MCP4131-502E
- added IC1: MCP41HVX1ST, microchip-mcp41hvx1:MCP41HVX1ST
Connections:
- removed net SPI_MOSI: U$19.MOSI
- removed net SPI_SCK: U$19.SCK
- removed net SPI_SS: U$19.SS
- new net MCU_!CS: IC1.!CS
- new net MCU_MISO: IC1.SDO
- new net MCU_MOSI: IC1.SDI
- new net MCU_SCK: IC1.SCK
- net +5V: now also IC1.VL; no longer U$19.+5V
- net GND: now also IC1.DGND, IC1.P0A, IC1.V-; no longer U$19.A, U$19.GND
- net N$51: now also IC1.P0B, IC1.V+; no longer U$19.B
- net N$52: now also IC1.P0W; no longer U$19.W
Other:
- note removed: "DP pin out: 1. SPI-CS 2. SPI-SCK 3. SPI-SDIO 4. GND 5. Pot A terminal 6. Pot wiper 7. Pot B terminal 8. Vcc"
- note removed: "Solid-state FNR controller v1.5"
- note removed: "Throttle Controller v1.3"
- moved on the sheet: GEARSHIFT_GND, LED4, Q6, R1, R21

Commit message: updated fnr
Parts:
- removed AMTOG+, AMTOG-: (no value), adafruit:PINHD-1X1
- removed GS_C, GS_N: N, adafruit:PINHD-1X1
- removed GS_F: F, adafruit:PINHD-1X1
- removed GS_R: R, adafruit:PINHD-1X1
- removed LED3: GREEN, adafruit:LED3MM
- removed Q4: IRLML2060TRPBFBSS123LT1G, SparkFun-DiscreteSemi:IRLML2060TRPBFBSS123LT1G
- removed R13, R15, R16, R17: 150, rcl:R-US_0204/5
- removed R14: 10K, rcl:R-US_0204/5
- removed R18, R20: 1K, rcl:R-US_0204/5
- removed R19: 1k, rcl:R-US_0204/5
- added IC2: SE555D, linear:SE555D
- added LED5: GREEN, adafruit:LED3MM
- added R2, R3, R5: 1K, rcl:R-US_0204/5
- LED1: value BLUE -> GREEN
- LED2: value RED -> GREEN
- R4: value 150 -> 1K
Connections:
- removed net AM_TOGGLE-: AMTOG-.1, LED1.A, LED2.A, LED3.A, R13.1, R14.1, R15.1, R17.1
- removed net AUTO_SENSE: R14.2
- removed net FGND: GS_F.1, Q3.S, R19.1
- removed net GEARSHIFT_F: R16.1
- removed net GEARSHIFT_R: R4.1
- removed net N: GS_N.1, Q2.D, Q4.D, Q5.D, R20.2
- removed net N$13: LED2.C, R18.2
- removed net N$14: LED3.C, R19.2
- removed net N$18: Q1.G, R13.2
- removed net N$22: Q3.D, Q4.S
- removed net N$23: Q5.G, R17.2
- removed net N$5: Q1.D, Q2.S
- removed net N$6: Q4.G, R16.2
- removed net N$8: LED1.C, R20.1
- removed net RGND: GS_R.1, Q1.S, R18.1
- new net FNR_CON_F: R5.2
- new net FNR_CON_R: R4.2
- net +5V: no longer AMTOG+.1
- net GND: no longer GS_C.1
- net N$1: no longer Q5.S
- net N$3: now also LED1.C, R4.1; no longer Q2.G, R4.2
- net N$4: now also LED2.C, R5.1; no longer Q3.G, R15.2
Other:
- note removed: "AUTO/MANUAL TOGGLE"
- note removed: "F"
- note removed: "Gearshift"
- note removed: "R"
- note removed: "R N F"
- moved on the sheet: LED1, LED2, Q1, Q2, Q3, Q5, R4
