File: Electrical Schematics/Version2/Schematics/boardv2temperature.sch (EAGLE design)
At the start: 0 parts

Commit message: updated power ethernet and tempatature
Parts:
- added R1, R2, R3, R4, R5, R6: (no value), SparkFun-Passives:RESISTOR0603-RES
- added X1, X2, X3, X4, X5, X6: (no value), con-molex:KK-156-2
Connections:
- new net N$1: R1.2, X1-1.S
- new net N$10: R4.1, X4-2.S
- new net N$11: R5.1, X5-2.S
- new net N$12: R6.1, X6-2.S
- new net N$2: R2.2, X2-1.S
- new net N$3: R3.2, X3-1.S
- new net N$4: R4.2, X4-1.S
- new net N$5: X5-1.S
- new net N$6: R6.2, X6-1.S
- new net N$8: R1.1, R2.1, R3.1, X1-2.S, X2-2.S, X3-2.S
Other:
- note added: "ESC temp"
- note added: "motor temp"
- note added: "motorcontroler"
- note added: "regular 3.3 temp"
- note added: "regulator 12v temp"
- note added: "regulator 5v temp"
