File: Electrical Schematics/Version2/Schematics/boardv2connectors.sch (EAGLE design)
At the start: 1 part

Commit message: updated everything
Other:
- note added: "Connector Block"
Changed lines of the file:
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@@
 <parts>
 <part name="U$1" library="connectors" deviceset="34830-2001" device=""/>
+<part name="FRAME1" library="frames" deviceset="DOCFIELD" device=""/>
 </parts>
 <sheets>
 <sheet>
 <plain>
+<frame x1="10.16" y1="-40.64" x2="193.04" y2="106.68" columns="8" rows="5" layer="91"/>
+<text x="33.02" y="88.9" size="5.08" layer="91">Connector Block</text>
 </plain>
 <instances>
 <instance part="U$1" gate="G$1" x="81.28" y="27.94"/>
+<instance part="FRAME1" gate="G$1" x="86.36" y="-35.56"/>
 </instances>
 <busses>
