File: Electrical Schematics/Version2/Schematics/boardv2steer.sch (EAGLE design)
At the start: 0 parts

Commit message: coimbineeded everything
Parts:
- added C4: 33nF, rcl:C-USC1206K
- added D1: ZENER_SOD123, Atlanta Robotics:ZENER_SOD123
- added IC3: VNH2SP30-E, st-microelectronics:VNH2SP30-E
- added J2: PHOENIX_2POS_1792863, Atlanta-Robotics LAPTOP:PHOENIX_2POS_1792863
- added LED3, LED4: (no value), led:LEDSML1206
- added Q1, Q2: IRFR3707Z, Atlanta Robotics:IRFR3707Z
- added R10: 100k, rcl:R-US_R1206W
- added R11, R12, R13, R14, R17, R21: 1k, rcl:R-US_R1206W
- added R15, R16: 3.3k, rcl:R-US_R1206W
- added R18: 10k, rcl:R-US_R1206W
- added R19: 1.5k, rcl:R-US_R1206W
- added U1: ADS1225_RGV_16, shit:ADS1225_RGV_16
Connections:
- new net +12V: IC3.VCC, IC3.VCC@1, IC3.VCC@2, R10.2
- new net +5V: R15.2, R16.2
- new net GND: C4.2, Q1.D, Q2.D, R19.1
- new net N$10: D1.A, IC3.GNDA, IC3.GNDA@1, IC3.GNDA@2, IC3.GNDB, IC3.GNDB@1, IC3.GNDB@2, Q1.S, Q2.S
- new net N$12: R14.1
- new net N$17: IC3.INA, R14.2
- new net N$18: IC3.INB, R13.2
- new net N$19: IC3.DIAGA, R11.2, R16.1
- new net N$20: IC3.DIAGB, R12.2, R15.1
- new net N$21: IC3.PWM, R17.2
- new net N$22: IC3.CS, R18.2, R19.2
- new net N$23: C4.1, R18.1
- new net N$24: IC3.OUTA, IC3.OUTA@1, IC3.OUTA@2, J2G$1.SK, LED3.A, LED4.C
- new net N$25: IC3.OUTB, IC3.OUTB@1, IC3.OUTB@2, J2G$2.SK, R21.1
- new net N$27: D1.C, Q1.G, Q2.G, R10.1
- new net N$28: LED3.C, LED4.A, R21.2
- new net N$29: R13.1
- new net N$30: R11.1
- new net N$31: R12.1
- new net N$32: R17.1
