File: Electrical Schematics/Version2/Schematics/boardv2mcu.sch (EAGLE design)
At the start: 12 parts, among them U1 TMS570LS0432_PZ_100

Commit message: MCU JTAG
Parts:
- added C1: 0.1uf, rcl:C-EUC0603
- added R1, R2, R3, R4, R5, R8: (no value), SparkFun-Passives:RESISTOR0603-RES
- added U$1: JTAG20PIN, connectors:JTAG20PIN
Connections:
- removed net TD: U1.TDI
- removed net TRSTN: U1.NTRST
- new net +3.3V: R1.1, U$1.P$1, U$1.P$2
- new net N$1: C1.1, R1.2, U$1.P$8
- new net NC/DBGACK: U$1.P$19
- new net NC/DBGRQ: U$1.P$17
- new net NRESET: R8.1, R8.2, U$1.P$15, U1.NRST
- new net NTRST: R2.1, R2.2, U$1.P$3, U1.NTRST
- new net RTCK: U$1.P$11
- new net TCK: R5.1, R5.2, U$1.P$9
- new net TDI: R3.1, R3.2, U$1.P$5, U1.TDI
- new net TDO: U$1.P$13
- net GND: now also C1.2, U$1.P$10, U$1.P$12, U$1.P$14, U$1.P$16, U$1.P$18, U$1.P$20, U$1.P$4, U$1.P$6
- net TMS: now also R4.1, R4.2, U$1.P$7

Commit message: updated mcu
Connections:
- new net B$2: U1.MIBSPI1NCS[0], U1.MIBSPI1NCS[2], U1.MIBSPI1SIMO, U1.SPI2SOMI
Other:
- note added: "Jtag programmer"
- note added: "MCU BLock"
Changed lines of the file:
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@@
 <part name="R5" library="SparkFun-Passives" deviceset="RESISTOR" device="0603-RES"/>
 <part name="R8" library="SparkFun-Passives" deviceset="RESISTOR" device="0603-RES"/>
+<part name="FRAME1" library="frames" deviceset="DOCFIELD" device=""/>
 </parts>
 <sheets>
 <sheet>
 <plain>
+<text x="203.2" y="30.48" size="1.778" layer="91">Jtag programmer</text>
+<text x="-30.48" y="111.76" size="5.08" layer="91">MCU BLock</text>
+<frame x1="-71.12" y1="-116.84" x2="358.14" y2="129.54" columns="8" rows="5" layer="91"/>
 </plain>
 <instances>
@@
 <instance part="R5" gate="G$1" x="195.58" y="-7.62"/>
 <instance part="R8" gate="G$1" x="195.58" y="7.62"/>
+<instance part="FRAME1" gate="G$1" x="251.46" y="-111.76"/>
 </instances>
 <busses>
+<bus name="TOMCU">
+<segment>
+<wire x1="144.78" y1="12.7" x2="144.78" y2="-53.34" width="0.762" layer="92"/>
+<label x="149.86" y="-35.56" size="1.778" layer="95"/>
+</segment>
+<segment>
+<wire x1="-2.54" y1="35.56" x2="-2.54" y2="-33.02" width="0.762" layer="92"/>
+<label x="-15.24" y="0" size="1.778" layer="95"/>
+</segment>
+</bus>
 </busses>
 <nets>
@@
 </segment>
 </net>
+<net name="B$2" class="0">
+<segment>
+<wire x1="144.78" y1="-50.8" x2="111.76" y2="-50.8" width="0.1524" layer="91"/>
+</segment>
+<segment>
+<wire x1="144.78" y1="-48.26" x2="111.76" y2="-48.26" width="0.1524" layer="91"/>
+</segment>
+<segment>
+<wire x1="144.78" y1="-45.72" x2="111.76" y2="-45.72" width="0.1524" layer="91"/>
+</segment>
+<segment>
+<wire x1="144.78" y1="-43.18" x2="111.76" y2="-43.18" width="0.1524" layer="91"/>
+</segment>
+<segment>
+<wire x1="144.78" y1="-40.64" x2="111.76" y2="-40.64" width="0.1524" layer="91"/>
+</segment>
+<segment>
+<wire x1="144.78" y1="-38.1" x2="111.76" y2="-38.1" width="0.1524" layer="91"/>
+</segment>
+<segment>
+<wire x1="144.78" y1="-33.02" x2="111.76" y2="-33.02" width="0.1524" layer="91"/>
+</segment>
+<segment>
+<wire x1="144.78" y1="-35.56" x2="111.76" y2="-35.56" width="0.1524" layer="91"/>
+</segment>
+<segment>
+<pinref part="U1" gate="A" pin="SPI2SOMI"/>
+<wire x1="144.78" y1="-30.48" x2="114.3" y2="-30.48" width="0.1524" layer="91"/>
+</segment>
+<segment>
+<wire x1="144.78" y1="-25.4" x2="111.76" y2="-25.4" width="0.1524" layer="91"/>
+</segment>
+<segment>
+<pinref part="U1" gate="A" pin="MIBSPI1NCS[2]"/>
+<wire x1="144.78" y1="-22.86" x2="114.3" y2="-22.86" width="0.1524" layer="91"/>
+</segment>
+<segment>
+<wire x1="144.78" y1="-20.32" x2="111.76" y2="-20.32" width="0.1524" layer="91"/>
+</segment>
+<segment>
+<pinref part="U1" gate="A" pin="MIBSPI1NCS[0]"/>
+<wire x1="144.78" y1="-17.78" x2="114.3" y2="-17.78" width="0.1524" layer="91"/>
+</segment>
+<segment>
+<wire x1="144.78" y1="-12.7" x2="111.76" y2="-12.7" width="0.1524" layer="91"/>
+</segment>
+<segment>
+<wire x1="144.78" y1="-15.24" x2="111.76" y2="-15.24" width="0.1524" layer="91"/>
+</segment>
+<segment>
+<pinref part="U1" gate="A" pin="MIBSPI1SIMO"/>
+<wire x1="144.78" y1="-10.16" x2="114.3" y2="-10.16" width="0.1524" layer="91"/>
+</segment>
+<segment>
+<wire x1="144.78" y1="-7.62" x2="111.76" y2="-7.62" width="0.1524" layer="91"/>
+</segment>
+</net>
