File: Electrical Schematics/Version2/Schematics/boardv2mcu.sch (EAGLE design)
At the start: 94 parts, among them U1 TMS570LS0432_PZ_100

Commit message: MCU
Connections:
- net NC/DBGACK renamed MCU_PROG_NC/DBGACK
- net NC/DBGRQ renamed MCU_PROG_NC/DBGRQ
- removed net +3.3V: U$1.P$1, U$1.P$2
- removed net N$1: TP29.TP, U1.NTRST
- removed net N$2: TP28.TP, U1.RTCK
- removed net N$3: TP27.TP, U1.TCK
- removed net N$37: C26.1, C27.1, C28.1, U1.VCC, U1.VCC_2, U1.VCC_3
- removed net N$4: TP26.TP, U1.TDO
- removed net N$5: TP25.TP, U1.TDI
- removed net N$6: TP24.TP, U1.TMS
- removed net RTCK: U$1.P$11
- removed net TDO: U$1.P$13
- new net MCU_+3.3V: C26.1, C27.1, C28.1, U$1.P$1, U$1.P$2, U1.VCC, U1.VCC_2, U1.VCC_3
- new net MCU_PROG_NRESET: R8.1
- new net MCU_PROG_NTRST: R2.2, TP29.TP, U$1.P$3, U1.NTRST
- new net MCU_PROG_RTCK: TP28.TP, U$1.P$11, U1.RTCK
- new net MCU_PROG_TCK: R5.2, TP27.TP, U$1.P$9, U1.TCK
- new net MCU_PROG_TDI: R3.2, TP25.TP, U$1.P$5, U1.TDI
- new net MCU_PROG_TDO: TP26.TP, U$1.P$13, U1.TDO
- new net MCU_PROG_TMS: R4.2, TP24.TP, U$1.P$7, U1.TMS
- net NRESET: no longer R8.1
- net NTRST: no longer R2.2, U$1.P$3
- net TCK: no longer R5.2, U$1.P$9
- net TDI: no longer R3.2, U$1.P$5
- net TMS: no longer R4.2, U$1.P$7
Other:
- moved on the sheet: TP28, TP29
