File: Electrical Schematics/Version2/Schematics/boardv2fpga.sch (EAGLE design)
At the start: 18 parts

Commit message: updated fpga
Parts:
- added Q1: ASFL1, crystal:ASFL1
Connections:
- new net 128MHZCLK_OUT_TO_GCLK_FPGA: U$1.IO_L30P_GCLK1_D13_2
- new net 3.3V: Q1.OE
- new net JTAGBUS: U$1.TCK, U$1.TDI, U$1.TDO, U$1.TMS
- net GND: now also Q1.GND
Changed lines of the file:
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@@
 <part name="C17" library="SparkFun-Capacitors" deviceset="CAP" device="0603-CAP" value="1uF"/>
 <part name="SUPPLY6" library="supply2" deviceset="GND" device=""/>
+<part name="Q1" library="crystal" deviceset="ASF*" device="" technology="L1"/>
+<part name="SUPPLY7" library="supply2" deviceset="GND" device=""/>
 </parts>
 <sheets>
@@
 <instance part="C17" gate="G$1" x="193.04" y="25.4"/>
 <instance part="SUPPLY6" gate="GND" x="180.34" y="20.32"/>
+<instance part="Q1" gate="G$1" x="-7.62" y="-30.48"/>
+<instance part="SUPPLY7" gate="GND" x="-38.1" y="-48.26"/>
 </instances>
 <busses>
+<bus name="JTAGBUS">
+<segment>
+<wire x1="60.96" y1="137.16" x2="60.96" y2="86.36" width="0.762" layer="92"/>
+<label x="60.96" y="119.38" size="1.778" layer="95"/>
+</segment>
+</bus>
+<bus name="FRONTENDIO">
+<segment>
+<wire x1="281.94" y1="116.84" x2="281.94" y2="7.62" width="0.762" layer="92"/>
+<label x="284.48" y="71.12" size="1.778" layer="95"/>
+</segment>
+</bus>
+<bus name="TOMCU">
+<segment>
+<wire x1="309.88" y1="109.22" x2="309.88" y2="2.54" width="0.762" layer="92"/>
+<label x="297.18" y="83.82" size="1.778" layer="95"/>
+</segment>
+</bus>
 </busses>
 <nets>
@@
 <pinref part="SUPPLY6" gate="GND" pin="GND"/>
 </segment>
+<segment>
+<pinref part="Q1" gate="G$1" pin="GND"/>
+<wire x1="-20.32" y1="-35.56" x2="-38.1" y2="-35.56" width="0.1524" layer="91"/>
+<wire x1="-38.1" y1="-35.56" x2="-38.1" y2="-45.72" width="0.1524" layer="91"/>
+<pinref part="SUPPLY7" gate="GND" pin="GND"/>
+</segment>
 </net>
 <net name="VCCINT" class="0">
@@
 </segment>
 </net>
+<net name="3.3V" class="0">
+<segment>
+<wire x1="-17.78" y1="-25.4" x2="-20.32" y2="-25.4" width="0.1524" layer="91"/>
+<pinref part="Q1" gate="G$1" pin="OE"/>
+<wire x1="-20.32" y1="-25.4" x2="-35.56" y2="-25.4" width="0.1524" layer="91"/>
+<wire x1="5.08" y1="-25.4" x2="10.16" y2="-25.4" width="0.1524" layer="91"/>
+<wire x1="10.16" y1="-25.4" x2="10.16" y2="-17.78" width="0.1524" layer="91"/>
+<wire x1="10.16" y1="-17.78" x2="-20.32" y2="-17.78" width="0.1524" layer="91"/>
+<wire x1="-20.32" y1="-17.78" x2="-20.32" y2="-25.4" width="0.1524" layer="91"/>
+<label x="-40.64" y="-22.86" size="1.778" layer="95"/>
+</segment>
+</net>
+<net name="128MHZCLK_OUT_TO_GCLK_FPGA" class="0">
+<segment>
+<wire x1="2.54" y1="-30.48" x2="25.4" y2="-30.48" width="0.1524" layer="91"/>
+<label x="15.24" y="-25.4" size="1.778" layer="95"/>
+</segment>
+<segment>
+<wire x1="86.36" y1="15.24" x2="83.82" y2="15.24" width="0.1524" layer="91"/>
+<pinref part="U$1" gate="G$1" pin="IO_L30P_GCLK1_D13_2"/>
+<junction x="83.82" y="15.24"/>
+<wire x1="83.82" y1="15.24" x2="73.66" y2="15.24" width="0.1524" layer="91"/>
+<label x="63.5" y="15.24" size="1.778" layer="95" rot="R270"/>
+</segment>
+</net>
+<net name="JTAGBUS" class="0">
+<segment>
+<pinref part="U$1" gate="G$1" pin="TDO"/>
+<wire x1="40.64" y1="93.98" x2="50.8" y2="93.98" width="0.1524" layer="91"/>
+<label x="45.72" y="93.98" size="1.778" layer="95"/>
+<wire x1="60.96" y1="96.52" x2="53.34" y2="96.52" width="0.1524" layer="91"/>
+<wire x1="53.34" y1="96.52" x2="50.8" y2="93.98" width="0.1524" layer="91"/>
+</segment>
+<segment>
+<pinref part="U$1" gate="G$1" pin="TMS"/>
+<wire x1="40.64" y1="91.44" x2="53.34" y2="91.44" width="0.1524" layer="91"/>
+<label x="45.72" y="91.44" size="1.778" layer="95"/>
+<wire x1="60.96" y1="93.98" x2="55.88" y2="93.98" width="0.1524" layer="91"/>
+<wire x1="55.88" y1="93.98" x2="53.34" y2="91.44" width="0.1524" layer="91"/>
+</segment>
+<segment>
+<pinref part="U$1" gate="G$1" pin="TCK"/>
+<wire x1="40.64" y1="86.36" x2="50.8" y2="86.36" width="0.1524" layer="91"/>
+<label x="45.72" y="86.36" size="1.778" layer="95"/>
+<wire x1="60.96" y1="91.44" x2="55.88" y2="91.44" width="0.1524" layer="91"/>
+<wire x1="55.88" y1="91.44" x2="50.8" y2="86.36" width="0.1524" layer="91"/>
+</segment>
+<segment>
+<pinref part="U$1" gate="G$1" pin="TDI"/>
+<wire x1="40.64" y1="83.82" x2="50.8" y2="83.82" width="0.1524" layer="91"/>
+<label x="45.72" y="83.82" size="1.778" layer="95"/>
+<wire x1="60.96" y1="88.9" x2="55.88" y2="88.9" width="0.1524" layer="91"/>
+<wire x1="55.88" y1="88.9" x2="50.8" y2="83.82" width="0.1524" layer="91"/>
+</segment>
+</net>
 </nets>
 </sheet>
+<sheet>
+<plain>
+</plain>
+<instances>
+</instances>
+<busses>
+<bus name="B$1">
+<segment>
+<wire x1="-2.54" y1="96.52" x2="-2.54" y2="22.86" width="0.762" layer="92"/>
+</segment>
+</bus>
+</busses>
+<nets>
+</nets>
+</sheet>

Commit message: Data Isolation FPGA
Parts:
- added JP1, JP10, JP11, JP12, JP13, JP14, JP15, JP16, JP17, JP18, JP19, JP2, JP20, JP21, JP22, JP23, JP24, JP25, JP26, JP27, JP28, JP29, JP3, JP30, JP31, JP32, JP33, JP34, JP35, JP36, JP37, JP38, JP39, JP4, JP40, JP41, JP42, JP43, JP44, JP45, JP46, JP47, JP48, JP49, JP5, JP50, JP51, JP52, JP53, JP54, JP55, JP56, JP6, JP7, JP8, JP9: (no value), jumper:JP2E
- added OK1, OK10, OK11, OK12, OK13, OK14, OK15, OK16, OK2, OK3, OK4, OK5, OK6, OK7, OK8, OK9: MOC3043S, optocoupler:MOC3043S
- added R1, R10, R11, R12, R13, R14, R15, R16, R17, R18, R19, R2, R20, R21, R22, R23, R24, R25, R26, R27, R28, R29, R3, R30, R31, R32, R4, R5, R6, R7, R8, R9: (no value), SparkFun-Passives:RESISTOR0603-RES
- added X1, X2, X3, X4, X5, X6, X7, X8: (no value), con-molex:KK-156-4
Connections:
- new net +3.3V: JP13.1, JP14.1, JP20.1, JP21.1, JP27.1, JP28.1, JP34.1, JP35.1, JP41.1, JP42.1, JP48.1, JP49.1, JP55.1, JP56.1, JP6.1, JP7.1
- new net +3.3VRAIL: JP1.3, JP15.3, JP22.3, JP29.3, JP36.3, JP43.3, JP50.3, JP8.3
- new net +5V: JP1.1, JP15.1, JP22.1, JP29.1, JP36.1, JP43.1, JP50.1, JP8.1
- new net FPGA_L33N_MODULED_ISOLATOR: JP23.3, JP24.3, U$1.IO_L33N_1
- new net FPGA_L33P_MODULED_ISOLATOR: JP25.3, JP26.3, U$1.IO_L33P_1
- new net FPGA_L34N_MODULEC_ISOLATOR: JP16.3, JP17.3, U$1.IO_L34N_1
- new net FPGA_L34P_MODULEC_ISOLATOR: JP18.3, JP19.3, U$1.IO_L34P_1
- new net FPGA_L40N_MODULEB_ISOLATOR: JP10.3, JP9.3, U$1.IO_L40N_GCLK10_1
- new net FPGA_L40P_MODULEB_ISOLATOR: JP11.3, JP12.3, U$1.IO_L40P_GCLK11_1
- new net FPGA_L41N_MODULEA_ISOLATOR: JP2.3, JP3.3, U$1.IO_L41N_GCLK8_1
- new net FPGA_L41P_MODULEA_ISOLATOR: U$1.IO_L41P_GCLK9_IRDY1_1
- new net FPGA_L41P_MODULEA_ISOLATOR1: JP4.3, JP5.3
- new net FPGA_L49N_MODULEH_ISOLATOR: JP51.3, JP52.3, U$1.IO_L49N_3
- new net FPGA_L49P_MODULEH_ISOLATOR: JP53.3, JP54.3, U$1.IO_L49P_3
- new net FPGA_L50N_MODULEG_ISOLATOR: JP44.3, JP45.3, U$1.IO_L50N_3
- new net FPGA_L50P_MODULEG_ISOLATOR: JP46.3, JP47.3, U$1.IO_L50P_3
- new net FPGA_L51N_MODULEF_ISOLATOR: JP37.3, JP38.3, U$1.IO_L51N_3
- new net FPGA_L51P_MODULEF_ISOLATOR: JP39.3, JP40.3, U$1.IO_L51P_3
- new net FPGA_L52N_MODULEE_ISOLATOR: JP30.3, JP31.3, U$1.IO_L52N_3
- new net FPGA_L52P_MODULEE_ISOLATOR: JP32.3, JP33.3, U$1.IO_L52P_3
- new net N$1: JP10.1, JP9.1, X2-2.S
- new net N$10: JP6.2, R3.2
- new net N$11: JP11.1, JP12.1, X2-3.S
- new net N$12: JP7.2, R4.2
- new net N$13: JP10.2, OK3.A2, R7.1
- new net N$14: OK4.A, R5.2
- new net N$15: JP11.2, R5.1
- new net N$16: OK3.A, R6.2
- new net N$17: JP9.2, R6.1
- new net N$18: JP13.2, R7.2
- new net N$19: JP12.2, OK4.A2, R8.1
- new net N$2: JP2.1, JP3.1, X1-2.S
- new net N$20: JP14.2, R8.2
- new net N$21: JP16.1, JP17.1, X3-2.S
- new net N$22: JP18.1, JP19.1, X3-3.S
- new net N$23: JP17.2, OK5.A2, R11.1
- new net N$24: OK6.A, R9.2
- new net N$25: JP18.2, R9.1
- new net N$26: OK5.A, R10.2
- new net N$27: JP16.2, R10.1
- new net N$28: JP20.2, R11.2
- new net N$29: JP19.2, OK6.A2, R12.1
- new net N$3: JP4.1, JP5.1, X1-3.S
- new net N$30: JP21.2, R12.2
- new net N$31: JP23.1, JP24.1, X4-2.S
- new net N$32: JP25.1, JP26.1, X4-3.S
- new net N$33: JP24.2, OK7.A2, R15.1
- new net N$34: OK8.A, R13.2
- new net N$35: JP25.2, R13.1
- new net N$36: OK7.A, R14.2
- new net N$37: JP23.2, R14.1
- new net N$38: JP27.2, R15.2
- new net N$39: JP26.2, OK8.A2, R16.1
- new net N$4: JP3.2, OK1.A2, R3.1
- new net N$40: JP28.2, R16.2
- new net N$41: JP30.1, JP31.1, X5-2.S
- new net N$42: JP32.1, JP33.1, X5-3.S
- new net N$43: JP31.2, OK9.A2, R19.1
- new net N$44: OK10.A, R17.2
- new net N$45: JP32.2, R17.1
- new net N$46: OK9.A, R18.2
- new net N$47: JP30.2, R18.1
- new net N$48: JP34.2, R19.2
- new net N$49: JP33.2, OK10.A2, R20.1
- new net N$5: OK2.A, R1.2
- new net N$50: JP35.2, R20.2
- new net N$51: JP37.1, JP38.1, X6-2.S
- new net N$52: JP39.1, JP40.1, X6-3.S
- new net N$53: JP38.2, OK11.A2, R23.1
- new net N$54: OK12.A, R21.2
- new net N$55: JP39.2, R21.1
- new net N$56: OK11.A, R22.2
- new net N$57: JP37.2, R22.1
- new net N$58: JP41.2, R23.2
- new net N$59: JP40.2, OK12.A2, R24.1
- new net N$6: OK1.A, R2.2
- new net N$60: JP42.2, R24.2
- new net N$61: JP44.1, JP45.1, X7-2.S
- new net N$62: JP46.1, JP47.1, X7-3.S
- new net N$63: JP45.2, OK13.A2, R27.1
- new net N$64: OK14.A, R25.2
- new net N$65: JP46.2, R25.1
- new net N$66: OK13.A, R26.2
- new net N$67: JP44.2, R26.1
- new net N$68: JP48.2, R27.2
- new net N$69: JP47.2, OK14.A2, R28.1
- new net N$7: JP4.2, R1.1
- new net N$70: JP49.2, R28.2
- new net N$71: JP51.1, JP52.1, X8-2.S
- new net N$72: JP53.1, JP54.1, X8-3.S
- new net N$73: JP52.2, OK15.A2, R31.1
- new net N$74: OK16.A, R29.2
- new net N$75: JP53.2, R29.1
- new net N$76: OK15.A, R30.2
- new net N$77: JP51.2, R30.1
- new net N$78: JP55.2, R31.2
- new net N$79: JP54.2, OK16.A2, R32.1
- new net N$8: JP2.2, R2.1
- new net N$80: JP56.2, R32.2
- new net N$9: JP5.2, OK2.A2, R4.1
- new net V1: JP1.2, JP6.3, JP7.3, X1-1.S
- new net V2: JP13.3, JP14.3, JP8.2, X2-1.S
- new net V3: JP15.2, JP20.3, JP21.3, X3-1.S
- new net V4: JP22.2, JP27.3, JP28.3, X4-1.S
- new net V5: JP29.2, JP34.3, JP35.3, X5-1.S
- new net V6: JP36.2, JP41.3, JP42.3, X6-1.S
- new net V7: JP43.2, JP48.3, JP49.3, X7-1.S
- new net V8: JP50.2, JP55.3, JP56.3, X8-1.S
- net GND: now also OK1.A1, OK1.C, OK10.A1, OK10.C, OK11.A1, OK11.C, OK12.A1, OK12.C, OK13.A1, OK13.C, OK14.A1, OK14.C, OK15.A1, OK15.C, OK16.A1, OK16.C, OK2.A1, OK2.C, OK3.A1, OK3.C, OK4.A1, OK4.C, OK5.A1, OK5.C, OK6.A1, OK6.C, OK7.A1, OK7.C, OK8.A1, OK8.C, OK9.A1, OK9.C, X1-4.S, X2-4.S, X3-4.S, X4-4.S, X5-4.S, X6-4.S, X7-4.S, X8-4.S
Other:
- note added: "1.Anode 4.Emitter 2.Cathode 5.Collector 3.NC 6.Base"

Commit message: added Programmer to fpga
Parts:
- added U$2: JTAG14PIN, connectors:JTAG14PIN
Connections:
- new net HALT: U$2.P$7
- new net TCK: U$2.P$3
- new net TDI: U$2.P$5
- new net TDO: U$2.P$4
- new net TMS: U$2.P$2
- new net VREF: U$2.P$1
- net GND: now also U$2.P$10, U$2.P$11, U$2.P$12, U$2.P$13, U$2.P$14, U$2.P$8, U$2.P$9
Changed lines of the file:
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@@
 <setting verticaltext="up"/>
 </settings>
-<grid distance="0.1" unitdist="inch" unit="inch" style="lines" multiple="1" display="no" altdistance="0.01" altunitdist="inch" altunit="inch"/>
+<grid distance="0.05" unitdist="inch" unit="inch" style="lines" multiple="1" display="no" altdistance="0.025" altunitdist="inch" altunit="inch"/>
 <layers>
 <layer number="1" name="Top" color="4" fill="1" visible="no" active="no"/>
@@
 <part name="JP56" library="jumper" deviceset="JP2E" device=""/>
 <part name="R32" library="SparkFun-Passives" deviceset="RESISTOR" device="0603-RES"/>
+<part name="U$2" library="connectors" deviceset="JTAG14PIN" device=""/>
+<part name="SUPPLY48" library="supply2" deviceset="GND" device=""/>
 </parts>
 <sheets>
@@
 <bus name="JTAGBUS">
 <segment>
-<wire x1="60.96" y1="137.16" x2="60.96" y2="86.36" width="0.762" layer="92"/>
+<wire x1="60.96" y1="137.16" x2="60.96" y2="82.55" width="0.762" layer="92"/>
 <label x="60.96" y="119.38" size="1.778" layer="95"/>
-</segment>
-</bus>
-<bus name="FRONTENDIO">
-<segment>
-<wire x1="281.94" y1="116.84" x2="281.94" y2="7.62" width="0.762" layer="92"/>
-<label x="284.48" y="71.12" size="1.778" layer="95"/>
-</segment>
-</bus>
-<bus name="TOMCU">
-<segment>
-<wire x1="309.88" y1="109.22" x2="309.88" y2="2.54" width="0.762" layer="92"/>
-<label x="297.18" y="83.82" size="1.778" layer="95"/>
 </segment>
 </bus>
@@
 <segment>
 <pinref part="U$1" gate="G$1" pin="TDO"/>
-<wire x1="40.64" y1="93.98" x2="50.8" y2="93.98" width="0.1524" layer="91"/>
+<wire x1="40.64" y1="93.98" x2="60.96" y2="93.98" width="0.1524" layer="91"/>
 <label x="45.72" y="93.98" size="1.778" layer="95"/>
-<wire x1="60.96" y1="96.52" x2="53.34" y2="96.52" width="0.1524" layer="91"/>
-<wire x1="53.34" y1="96.52" x2="50.8" y2="93.98" width="0.1524" layer="91"/>
 </segment>
 <segment>
 <pinref part="U$1" gate="G$1" pin="TMS"/>
-<wire x1="40.64" y1="91.44" x2="53.34" y2="91.44" width="0.1524" layer="91"/>
+<wire x1="40.64" y1="91.44" x2="60.96" y2="91.44" width="0.1524" layer="91"/>
 <label x="45.72" y="91.44" size="1.778" layer="95"/>
-<wire x1="60.96" y1="93.98" x2="55.88" y2="93.98" width="0.1524" layer="91"/>
-<wire x1="55.88" y1="93.98" x2="53.34" y2="91.44" width="0.1524" layer="91"/>
 </segment>
 <segment>
 <pinref part="U$1" gate="G$1" pin="TCK"/>
-<wire x1="40.64" y1="86.36" x2="50.8" y2="86.36" width="0.1524" layer="91"/>
+<wire x1="40.64" y1="86.36" x2="60.96" y2="86.36" width="0.1524" layer="91"/>
 <label x="45.72" y="86.36" size="1.778" layer="95"/>
-<wire x1="60.96" y1="91.44" x2="55.88" y2="91.44" width="0.1524" layer="91"/>
-<wire x1="55.88" y1="91.44" x2="50.8" y2="86.36" width="0.1524" layer="91"/>
 </segment>
 <segment>
 <pinref part="U$1" gate="G$1" pin="TDI"/>
-<wire x1="40.64" y1="83.82" x2="50.8" y2="83.82" width="0.1524" layer="91"/>
+<wire x1="40.64" y1="83.82" x2="60.96" y2="83.82" width="0.1524" layer="91"/>
 <label x="45.72" y="83.82" size="1.778" layer="95"/>
-<wire x1="60.96" y1="88.9" x2="55.88" y2="88.9" width="0.1524" layer="91"/>
-<wire x1="55.88" y1="88.9" x2="50.8" y2="83.82" width="0.1524" layer="91"/>
 </segment>
 </net>
@@
 </plain>
 <instances>
+<instance part="U$2" gate="G$1" x="63.5" y="68.58" rot="R90"/>
+<instance part="SUPPLY48" gate="GND" x="43.18" y="66.04"/>
 </instances>
 <busses>
-<bus name="B$1">
+<bus name="JTAG">
 <segment>
 <wire x1="-2.54" y1="96.52" x2="-2.54" y2="22.86" width="0.762" layer="92"/>
+<label x="2.54" y="85.09" size="1.778" layer="95"/>
 </segment>
 </bus>
 </busses>
 <nets>
+<net name="HALT" class="0">
+<segment>
+<wire x1="-2.54" y1="59.69" x2="60.96" y2="59.69" width="0.1524" layer="91"/>
+<pinref part="U$2" gate="G$1" pin="P$7"/>
+<label x="7.62" y="59.69" size="1.778" layer="95"/>
+</segment>
+</net>
+<net name="VREF" class="0">
+<segment>
+<pinref part="U$2" gate="G$1" pin="P$1"/>
+<wire x1="-2.54" y1="44.45" x2="60.96" y2="44.45" width="0.1524" layer="91"/>
+<label x="7.62" y="44.45" size="1.778" layer="95"/>
+</segment>
+</net>
+<net name="TMS" class="0">
+<segment>
+<pinref part="U$2" gate="G$1" pin="P$2"/>
+<wire x1="-2.54" y1="46.99" x2="60.96" y2="46.99" width="0.1524" layer="91"/>
+<label x="7.62" y="46.99" size="1.778" layer="95"/>
+</segment>
+</net>
+<net name="TCK" class="0">
+<segment>
+<pinref part="U$2" gate="G$1" pin="P$3"/>
+<wire x1="-2.54" y1="49.53" x2="60.96" y2="49.53" width="0.1524" layer="91"/>
+<label x="7.62" y="49.53" size="1.778" layer="95"/>
+</segment>
+</net>
+<net name="TDO" class="0">
+<segment>
+<pinref part="U$2" gate="G$1" pin="P$4"/>
+<wire x1="-2.54" y1="52.07" x2="60.96" y2="52.07" width="0.1524" layer="91"/>
+<label x="7.62" y="52.07" size="1.778" layer="95"/>
+</segment>
+</net>
+<net name="TDI" class="0">
+<segment>
+<pinref part="U$2" gate="G$1" pin="P$5"/>
+<wire x1="-2.54" y1="54.61" x2="60.96" y2="54.61" width="0.1524" layer="91"/>
+<label x="7.62" y="54.61" size="1.778" layer="95"/>
+</segment>
+</net>
+<net name="GND" class="0">
+<segment>
+<pinref part="U$2" gate="G$1" pin="P$8"/>
+<wire x1="60.96" y1="62.23" x2="55.88" y2="62.23" width="0.1524" layer="91"/>
+<wire x1="55.88" y1="62.23" x2="55.88" y2="64.77" width="0.1524" layer="91"/>
+<pinref part="U$2" gate="G$1" pin="P$9"/>
+<wire x1="55.88" y1="64.77" x2="60.96" y2="64.77" width="0.1524" layer="91"/>
+<pinref part="U$2" gate="G$1" pin="P$10"/>
+<wire x1="60.96" y1="67.31" x2="55.88" y2="67.31" width="0.1524" layer="91"/>
+<wire x1="55.88" y1="67.31" x2="55.88" y2="64.77" width="0.1524" layer="91"/>
+<pinref part="U$2" gate="G$1" pin="P$11"/>
+<wire x1="60.96" y1="69.85" x2="55.88" y2="69.85" width="0.1524" layer="91"/>
+<pinref part="U$2" gate="G$1" pin="P$12"/>
+<wire x1="55.88" y1="69.85" x2="55.88" y2="67.31" width="0.1524" layer="91"/>
+<wire x1="60.96" y1="72.39" x2="55.88" y2="72.39" width="0.1524" layer="91"/>
+<pinref part="U$2" gate="G$1" pin="P$13"/>
+<wire x1="55.88" y1="72.39" x2="55.88" y2="69.85" width="0.1524" layer="91"/>
+<wire x1="60.96" y1="74.93" x2="55.88" y2="74.93" width="0.1524" layer="91"/>
+<pinref part="U$2" gate="G$1" pin="P$14"/>
+<wire x1="55.88" y1="74.93" x2="55.88" y2="72.39" width="0.1524" layer="91"/>
+<wire x1="60.96" y1="77.47" x2="55.88" y2="77.47" width="0.1524" layer="91"/>
+<wire x1="55.88" y1="77.47" x2="55.88" y2="74.93" width="0.1524" layer="91"/>
+<wire x1="55.88" y1="72.39" x2="43.18" y2="72.39" width="0.1524" layer="91"/>
+<wire x1="43.18" y1="72.39" x2="43.18" y2="68.58" width="0.1524" layer="91"/>
+<pinref part="SUPPLY48" gate="GND" pin="GND"/>
+</segment>
+</net>
 </nets>
 </sheet>
