File: Electrical Schematics/Version2/Schematics/boardv2fpga.sch (EAGLE design)
At the start: 132 parts, among them Q1 ASFL1

Commit message: updated everything
Other:
- note added: "FPGA Block"
- note added: "JTAG Programmer"
- note added: "Modular Connector A With Isolation"
- note added: "Modular Connector B With Isolation"
- note added: "Modular Connector C With Isolation"
- note added: "Modular Connector D With Isolation"
- note added: "Modular Connector E With Isolation"
- note added: "Modular Connector F With Isolation"
- note added: "Modular Connector H With Isolation"
- note added: "Modular Connector N With Isolation"
- note added: "Primary FPGA"
Changed lines of the file:
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@@
 <setting verticaltext="up"/>
 </settings>
-<grid distance="0.05" unitdist="inch" unit="inch" style="lines" multiple="1" display="no" altdistance="0.025" altunitdist="inch" altunit="inch"/>
+<grid distance="0.1" unitdist="inch" unit="inch" style="lines" multiple="1" display="no" altdistance="0.01" altunitdist="inch" altunit="inch"/>
 <layers>
 <layer number="1" name="Top" color="4" fill="1" visible="no" active="no"/>
@@
 <part name="U$2" library="connectors" deviceset="JTAG14PIN" device=""/>
 <part name="SUPPLY48" library="supply2" deviceset="GND" device=""/>
+<part name="FRAME1" library="frames" deviceset="DOCFIELD" device=""/>
+<part name="FRAME2" library="frames" deviceset="DOCFIELD" device=""/>
+<part name="FRAME3" library="frames" deviceset="DOCFIELD" device=""/>
+<part name="FRAME4" library="frames" deviceset="DOCFIELD" device=""/>
+<part name="FRAME5" library="frames" deviceset="DOCFIELD" device=""/>
+<part name="FRAME6" library="frames" deviceset="DOCFIELD" device=""/>
+<part name="FRAME7" library="frames" deviceset="DOCFIELD" device=""/>
+<part name="FRAME8" library="frames" deviceset="DOCFIELD" device=""/>
+<part name="FRAME9" library="frames" deviceset="DOCFIELD" device=""/>
+<part name="FRAME10" library="frames" deviceset="DOCFIELD" device=""/>
 </parts>
 <sheets>
 <sheet>
 <plain>
+<frame x1="-124.46" y1="-91.44" x2="373.38" y2="175.26" columns="8" rows="5" layer="91"/>
+<text x="-109.22" y="160.02" size="5.08" layer="91">FPGA Block</text>
+<text x="-101.6" y="152.4" size="5.08" layer="91">Primary FPGA</text>
 </plain>
 <instances>
@@
 <instance part="Q1" gate="G$1" x="-7.62" y="-30.48"/>
 <instance part="SUPPLY7" gate="GND" x="-38.1" y="-48.26"/>
+<instance part="FRAME1" gate="G$1" x="269.24" y="-86.36"/>
 </instances>
 <busses>
@@
 <sheet>
 <plain>
+<frame x1="-20.32" y1="-20.32" x2="198.12" y2="109.22" columns="8" rows="5" layer="91"/>
+<text x="-12.7" y="99.06" size="5.08" layer="91">FPGA Block</text>
+<text x="20.32" y="91.44" size="5.08" layer="91">JTAG Programmer</text>
 </plain>
 <instances>
 <instance part="U$2" gate="G$1" x="63.5" y="68.58" rot="R90"/>
 <instance part="SUPPLY48" gate="GND" x="43.18" y="66.04"/>
+<instance part="FRAME2" gate="G$1" x="91.44" y="-15.24"/>
 </instances>
 <busses>
@@
 2.Cathode 5.Collector
 3.NC          6.Base</text>
+<frame x1="-88.9" y1="-35.56" x2="177.8" y2="124.46" columns="8" rows="5" layer="91"/>
+<text x="-81.28" y="111.76" size="5.08" layer="91">FPGA Block</text>
+<text x="-58.42" y="104.14" size="5.08" layer="91">Modular Connector A With Isolation</text>
 </plain>
 <instances>
@@
 <instance part="JP7" gate="1" x="43.18" y="38.1"/>
 <instance part="R4" gate="G$1" x="43.18" y="30.48" rot="R90"/>
+<instance part="FRAME3" gate="G$1" x="63.5" y="-25.4"/>
 </instances>
 <busses>
@@
 2.Cathode 5.Collector
 3.NC          6.Base</text>
+<frame x1="-40.64" y1="-30.48" x2="226.06" y2="129.54" columns="8" rows="5" layer="91"/>
+<text x="-33.02" y="116.84" size="5.08" layer="91">FPGA Block</text>
+<text x="-17.78" y="106.68" size="5.08" layer="91">Modular Connector B With Isolation</text>
 </plain>
 <instances>
@@
 <instance part="JP14" gate="1" x="96.52" y="33.02"/>
 <instance part="R8" gate="G$1" x="96.52" y="25.4" rot="R90"/>
+<instance part="FRAME4" gate="G$1" x="111.76" y="-20.32"/>
 </instances>
 <busses>
@@
 2.Cathode 5.Collector
 3.NC          6.Base</text>
+<frame x1="-25.4" y1="-33.02" x2="241.3" y2="127" columns="8" rows="5" layer="91"/>
+<text x="-15.24" y="114.3" size="5.08" layer="91">FPGA Block</text>
+<text x="-5.08" y="104.14" size="5.08" layer="91">Modular Connector C With Isolation</text>
 </plain>
 <instances>
@@
 <instance part="JP21" gate="1" x="96.52" y="43.18"/>
 <instance part="R12" gate="G$1" x="96.52" y="35.56" rot="R90"/>
+<instance part="FRAME5" gate="G$1" x="127" y="-22.86"/>
 </instances>
 <busses>
@@
 2.Cathode 5.Collector
 3.NC          6.Base</text>
+<frame x1="-27.94" y1="-40.64" x2="238.76" y2="119.38" columns="8" rows="5" layer="91"/>
+<text x="-20.32" y="106.68" size="5.08" layer="91">FPGA Block</text>
+<text x="-12.7" y="99.06" size="5.08" layer="91">Modular Connector D With Isolation</text>
 </plain>
 <instances>
@@
 <instance part="JP28" gate="1" x="99.06" y="27.94"/>
 <instance part="R16" gate="G$1" x="99.06" y="20.32" rot="R90"/>
+<instance part="FRAME6" gate="G$1" x="124.46" y="-30.48"/>
 </instances>
 <busses>
@@
 2.Cathode 5.Collector
 3.NC          6.Base</text>
+<frame x1="-30.48" y1="-45.72" x2="236.22" y2="114.3" columns="8" rows="5" layer="91"/>
+<text x="-22.86" y="101.6" size="5.08" layer="91">FPGA Block</text>
+<text x="-17.78" y="93.98" size="5.08" layer="91">Modular Connector E With Isolation</text>
 </plain>
 <instances>
@@
 <instance part="JP35" gate="1" x="101.6" y="25.4"/>
 <instance part="R20" gate="G$1" x="101.6" y="17.78" rot="R90"/>
+<instance part="FRAME7" gate="G$1" x="121.92" y="-35.56"/>
 </instances>
 <busses>
@@
 2.Cathode 5.Collector
 3.NC          6.Base</text>
+<frame x1="-27.94" y1="-48.26" x2="238.76" y2="111.76" columns="8" rows="5" layer="91"/>
+<text x="-17.78" y="99.06" size="5.08" layer="91">FPGA Block</text>
+<text x="-12.7" y="91.44" size="5.08" layer="91">Modular Connector F With Isolation</text>
 </plain>
 <instances>
@@
 <instance part="JP42" gate="1" x="96.52" y="27.94"/>
 <instance part="R24" gate="G$1" x="96.52" y="20.32" rot="R90"/>
+<instance part="FRAME8" gate="G$1" x="124.46" y="-38.1"/>
 </instances>
 <busses>
@@
 2.Cathode 5.Collector
 3.NC          6.Base</text>
+<frame x1="-35.56" y1="-48.26" x2="231.14" y2="111.76" columns="8" rows="5" layer="91"/>
+<text x="-25.4" y="96.52" size="5.08" layer="91">FPGA Block</text>
+<text x="-17.78" y="88.9" size="5.08" layer="91">Modular Connector N With Isolation</text>
 </plain>
 <instances>
@@
 <instance part="JP49" gate="1" x="96.52" y="27.94"/>
 <instance part="R28" gate="G$1" x="96.52" y="20.32" rot="R90"/>
+<instance part="FRAME9" gate="G$1" x="116.84" y="-38.1"/>
 </instances>
 <busses>
@@
 2.Cathode 5.Collector
 3.NC          6.Base</text>
+<frame x1="-40.64" y1="-45.72" x2="226.06" y2="114.3" columns="8" rows="5" layer="91"/>
+<text x="-30.48" y="99.06" size="5.08" layer="91">FPGA Block</text>
+<text x="-27.94" y="88.9" size="5.08" layer="91">Modular Connector H With Isolation</text>
 </plain>
 <instances>
@@
 <instance part="JP56" gate="1" x="99.06" y="27.94"/>
 <instance part="R32" gate="G$1" x="99.06" y="20.32" rot="R90"/>
+<instance part="FRAME10" gate="G$1" x="111.76" y="-35.56"/>
 </instances>
 <busses>

Commit message: Fixed Grounds
Parts:
- added JP57, JP59, JP60, JP61, JP64, JP65, JP66, JP68, JP69, JP71, JP72, JP74, JP75, JP77, JP78, JP80: (no value), jumper:JP2E
Connections:
- new net CONGND: JP57.1, JP59.1, JP60.1, JP61.1, JP64.1, JP65.1, JP66.1, JP68.1, JP69.1, JP71.1, JP72.1, JP74.1, JP75.1, JP77.1, JP78.1, JP80.1
- new net G1: JP57.2, OK1.C, OK2.C
- new net G2: JP60.2, OK3.C, OK4.C
- new net G3: JP65.2, OK5.C, OK6.C
- new net G4: JP66.2, OK7.C, OK8.C
- new net G5: JP69.2, OK10.C, OK9.C
- new net G6: JP72.2, OK11.C, OK12.C
- new net G7: JP75.2, OK13.C, OK14.C
- new net G8: JP78.2, OK15.C, OK16.C
- new net GSENSE1: JP59.2, OK1.A1, OK2.A1, X1-4.S
- new net GSENSE2: JP61.2, OK3.A1, OK4.A1, X2-4.S
- new net GSENSE3: JP64.2, OK5.A1, OK6.A1, X3-4.S
- new net GSENSE4: JP68.2, OK7.A1, OK8.A1, X4-4.S
- new net GSENSE5: JP71.2, OK10.A1, OK9.A1, X5-4.S
- new net GSENSE6: JP74.2, OK11.A1, OK12.A1, X6-4.S
- new net GSENSE7: JP77.2, OK13.A1, OK14.A1, X7-4.S
- new net GSENSE8: JP80.2, OK15.A1, OK16.A1, X8-4.S
- net GND: now also JP57.3, JP59.3, JP60.3, JP61.3, JP64.3, JP65.3, JP66.3, JP68.3, JP69.3, JP71.3, JP72.3, JP74.3, JP75.3, JP77.3, JP78.3, JP80.3; no longer OK1.A1, OK1.C, OK10.A1, OK10.C, OK11.A1, OK11.C, OK12.A1, OK12.C, OK13.A1, OK13.C, OK14.A1, OK14.C, OK15.A1, OK15.C, OK16.A1, OK16.C, OK2.A1, OK2.C, OK3.A1, OK3.C, OK4.A1, OK4.C, OK5.A1, OK5.C, OK6.A1, OK6.C, OK7.A1, OK7.C, OK8.A1, OK8.C, OK9.A1, OK9.C, X1-4.S, X2-4.S, X3-4.S, X4-4.S, X5-4.S, X6-4.S, X7-4.S, X8-4.S
Other:
- moved on the sheet: JP11, JP12, JP14, JP18, JP19, JP21, JP25, JP26, JP28, JP3, JP32, JP33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

Commit message: Saved Changes
Connections:
- net +3.3V renamed +3.3VFPGA
Changed lines of the file:
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@@
 </segment>
 </net>
-<net name="+3.3V" class="0">
+<net name="+3.3VFPGA" class="0">
 <segment>
 <pinref part="JP6" gate="1" pin="1"/>
@@
 </segment>
 </net>
-<net name="+3.3V" class="0">
+<net name="+3.3VFPGA" class="0">
 <segment>
 <pinref part="JP13" gate="1" pin="1"/>
@@
 </segment>
 </net>
-<net name="+3.3V" class="0">
+<net name="+3.3VFPGA" class="0">
 <segment>
 <pinref part="JP20" gate="1" pin="1"/>
@@
 </segment>
 </net>
-<net name="+3.3V" class="0">
+<net name="+3.3VFPGA" class="0">
 <segment>
 <pinref part="JP27" gate="1" pin="1"/>
@@
 </segment>
 </net>
-<net name="+3.3V" class="0">
+<net name="+3.3VFPGA" class="0">
 <segment>
 <pinref part="JP34" gate="1" pin="1"/>
@@
 </segment>
 </net>
-<net name="+3.3V" class="0">
+<net name="+3.3VFPGA" class="0">
 <segment>
 <pinref part="JP41" gate="1" pin="1"/>
@@
 </segment>
 </net>
-<net name="+3.3V" class="0">
+<net name="+3.3VFPGA" class="0">
 <segment>
 <pinref part="JP48" gate="1" pin="1"/>
@@
 </segment>
 </net>
-<net name="+3.3V" class="0">
+<net name="+3.3VFPGA" class="0">
 <segment>
 <pinref part="JP55" gate="1" pin="1"/>

Commit message: FPGA style and wiring io
Parts:
- removed JP77, JP78: (no value), jumper:JP2E
- added JP58, JP62, JP63, JP67, JP70: (no value), jumper:JP2E
- added JP79, JP89, JP90, JP91, JP92, JP93, JP94, JP95: (no value), pinhead:PINHD-1X8
- JP74, JP75, JP80: device jumper:JP2E -> pinhead:PINHD-1X8
Connections:
- net +3.3VRAIL renamed PP_3.3V_MODULARCONNECTOR
- net +5V renamed PP_5V_MODULARCONNECTOR
- net FPGA_L33N_MODULED_ISOLATOR renamed FPGA_L33N_1_MODULED_ISOLATOR
- net FPGA_L33P_MODULED_ISOLATOR renamed FPGA_L33P_1_MODULED_ISOLATOR
- net FPGA_L34N_MODULEC_ISOLATOR renamed FPGA_L34N_1_MODULEC_ISOLATOR
- net FPGA_L34P_MODULEC_ISOLATOR renamed FPGA_L34P_1_MODULEC_ISOLATOR
- net FPGA_L40N_MODULEB_ISOLATOR renamed FPGA_L40N_1_MODULEB_ISOLATOR
- net FPGA_L40P_MODULEB_ISOLATOR renamed FPGA_L40P_1_MODULEB_ISOLATOR
- net FPGA_L41N_MODULEA_ISOLATOR renamed FPGA_L41N_1_MODULEA_ISOLATOR
- net FPGA_L49N_MODULEH_ISOLATOR renamed FPGA_L49N_3_MODULEH_ISOLATOR
- net FPGA_L49P_MODULEH_ISOLATOR renamed FPGA_L49P_3_MODULEH_ISOLATOR
- net FPGA_L50N_MODULEG_ISOLATOR renamed FPGA_L50N_3_MODULEG_ISOLATOR
- net FPGA_L50P_MODULEG_ISOLATOR renamed FPGA_L50P_3_MODULEG_ISOLATOR
- net FPGA_L51N_MODULEF_ISOLATOR renamed FPGA_L51N_3_MODULEF_ISOLATOR
- net FPGA_L51P_MODULEF_ISOLATOR renamed FPGA_L51P_3_MODULEF_ISOLATOR
- net FPGA_L52N_MODULEE_ISOLATOR renamed FPGA_L52N_3_MODULEE_ISOLATOR
- net FPGA_L52P_MODULEE_ISOLATOR renamed FPGA_L52P_3_MODULEE_ISOLATOR
- removed net +3.3VFPGA: JP13.1, JP14.1, JP20.1, JP21.1, JP27.1, JP28.1, JP34.1, JP35.1, JP41.1, JP42.1, JP48.1, JP49.1, JP55.1, JP56.1, JP6.1, JP7.1
- removed net +3V3: C10.1, C11.1, C12.1, C13.1, C14.1, C15.1, C16.1, C17.1, C5.1, C6.1, C7.1, C8.1, C9.1, U$1.VCCAUX, U$1.VCCAUX@1, U$1.VCCAUX@2, U$1.VCCAUX@3, U$1.VCCAUX@4
- removed net FPGA_L41P_MODULEA_ISOLATOR: U$1.IO_L41P_GCLK9_IRDY1_1
- removed net FPGA_L41P_MODULEA_ISOLATOR1: JP4.3, JP5.3
- removed net JTAGBUS: U$1.TCK, U$1.TDI, U$1.TDO, U$1.TMS
- new net FPGA_CMPCS_B_2: U$1.CMPCS_B_2
- new net FPGA_DONE_2: U$1.DONE_2
- new net FPGA_L12N_2: JP90.2, U$1.IO_L12N_D2_MISO3_2
- new net FPGA_L12P_2: JP90.1, U$1.IO_L12P_D1_MISO2_2
- new net FPGA_L13N_2: JP90.4, U$1.IO_L13N_D10_2
- new net FPGA_L13P_2: JP90.3, U$1.IO_L13P_M1_2
- new net FPGA_L14N_2: JP90.6, U$1.IO_L14N_D12_2
- new net FPGA_L14P_2: JP90.5, U$1.IO_L14P_D11_2
- new net FPGA_L1N_0: JP94.2, U$1.IO_L1N_VREF_0
- new net FPGA_L1N_1: JP95.4, U$1.IO_L1N_VREF_1
- new net FPGA_L1N_2: JP91.4, U$1.IO_L1N_M0_CMPMISO_2
- new net FPGA_L1N_3: JP93.6, U$1.IO_L1N_VREF_3
- new net FPGA_L1P_0: JP94.1, U$1.IO_L1P_HSWAPEN_0
- new net FPGA_L1P_1: JP95.3, U$1.IO_L1P_1
- new net FPGA_L1P_2: JP91.3, U$1.IO_L1P_CCLK_2
- new net FPGA_L1P_3: JP93.5, U$1.IO_L1P_3
- new net FPGA_L2N_0: JP94.4, U$1.IO_L2N_0
- new net FPGA_L2N_2: JP91.6, U$1.IO_L2N_CMPMOSI_2
- new net FPGA_L2N_3: JP93.8, U$1.IO_L2N_3
- new net FPGA_L2P_0: JP94.3, U$1.IO_L2P_0
- new net FPGA_L2P_2: JP91.5, U$1.IO_L2P_CMPCLK_2
- new net FPGA_L2P_3: JP93.7, U$1.IO_L2P_3
- new net FPGA_L30N_2: JP90.8, U$1.IO_L30N_GCLK0_USERCCLK_2
- new net FPGA_L31N_2: JP89.2, U$1.IO_L31N_GCLK30_D15_2
- new net FPGA_L31P_2: JP89.1, U$1.IO_L31P_GCLK31_D14_2
- new net FPGA_L32N_1: JP95.6, U$1.IO_L32N_1
- new net FPGA_L32P_1: JP95.5, U$1.IO_L32P_1
- new net FPGA_L34N_0: JP74.2, U$1.IO_L34N_GCLK18_0
- new net FPGA_L34P_0: JP74.1, U$1.IO_L34P_GCLK19_0
- new net FPGA_L35N_0: JP74.4, U$1.IO_L35N_GCLK16_0
- new net FPGA_L35P_0: JP74.3, U$1.IO_L35P_GCLK17_0
- new net FPGA_L36N_0: JP74.6, U$1.IO_L36N_GCLK14_0
- new net FPGA_L36N_3: JP80.2, U$1.IO_L36N_3
- new net FPGA_L36P_0: JP74.5, U$1.IO_L36P_GCLK15_0
- new net FPGA_L36P_3: JP80.1, U$1.IO_L36P_3
- new net FPGA_L37N_0: JP74.8, U$1.IO_L37N_GCLK12_0
- new net FPGA_L37N_3: JP80.4, U$1.IO_L37N_3
- new net FPGA_L37P_0: JP74.7, U$1.IO_L37P_GCLK13_0
- new net FPGA_L37P_3: JP80.3, U$1.IO_L37P_3
- new net FPGA_L3N_0: JP94.6, U$1.IO_L3N_0
- new net FPGA_L3N_2: JP91.8, U$1.IO_L3N_MOSI_CSI_B_MISO0_2
- new net FPGA_L3P_0: JP94.5, U$1.IO_L3P_0
- new net FPGA_L3P_2: JP91.7, U$1.IO_L3P_D0_DIN_MISO_MISO1_2
- new net FPGA_L41N_3: JP80.6, U$1.IO_L41N_GCLK26_3
- new net FPGA_L41P_1_MODULEA_ISOLATOR: JP4.3, JP5.3, U$1.IO_L41P_GCLK9_IRDY1_1
- new net FPGA_L41P_3: JP80.5, U$1.IO_L41P_GCLK27_3
- new net FPGA_L42N_3: JP79.2, U$1.IO_L42N_GCLK24_3
- new net FPGA_L42N_GCLK6_TRDY1_1: JP95.8, U$1.IO_L42N_GCLK6_TRDY1_1
- new net FPGA_L42P_1: JP95.7, U$1.IO_L42P_GCLK7_1
- new net FPGA_L42P_3: JP79.1, U$1.IO_L42P_GCLK25_TRDY2_3
- new net FPGA_L43N_1: JP92.2, U$1.IO_L43N_GCLK4_1
- new net FPGA_L43N_3: JP79.4, U$1.IO_L43N_GCLK22_IRDY2_3
- new net FPGA_L43P_1: JP92.1, U$1.IO_L43P_GCLK5_1
- new net FPGA_L43P_3: JP79.3, U$1.IO_L43P_GCLK23_3
- new net FPGA_L44N_3: JP79.6, U$1.IO_L44N_GCLK20_3
- new net FPGA_L44P_3: JP79.5, U$1.IO_L44P_GCLK21_3
- new net FPGA_L45N_1: JP92.4, U$1.IO_L45N_1
- new net FPGA_L45P_1: JP92.3, U$1.IO_L45P_1
- new net FPGA_L46N_1: JP92.6, U$1.IO_L46N_1
- new net FPGA_L46P_1: JP92.5, U$1.IO_L46P_1
- new net FPGA_L47N_1: JP92.8, U$1.IO_L47N_1
- new net FPGA_L47P_1: JP92.7, U$1.IO_L47P_1
- new net FPGA_L48N_2: JP89.4, U$1.IO_L48N_RDWR_B_VREF_2
- new net FPGA_L48P_2: JP89.3, U$1.IO_L48P_D7_2
- new net FPGA_L49N_2: JP89.6, U$1.IO_L49N_D4_2
- new net FPGA_L49P_2: JP89.5, U$1.IO_L49P_D3_2
- new net FPGA_L4N_0: JP94.8, U$1.IO_L4N_0
- new net FPGA_L4P_0: JP94.7, U$1.IO_L4P_0
- new net FPGA_L62N_0: JP75.2, U$1.IO_L62N_VREF_0
- new net FPGA_L62N_2: JP89.8, U$1.IO_L62N_D6_2
- new net FPGA_L62P_0: JP75.1, U$1.IO_L62P_0
- new net FPGA_L62P_2: JP89.7, U$1.IO_L62P_D5_2
- new net FPGA_L63N_0: JP75.4, U$1.IO_L63N_SCP6_0
- new net FPGA_L63P_0: JP75.3, U$1.IO_L63P_SCP7_0
- new net FPGA_L64N_0: JP75.6, U$1.IO_L64N_SCP4_0
- new net FPGA_L64N_2: JP93.2, U$1.IO_L64N_D9_2
- new net FPGA_L64P_0: JP75.5, U$1.IO_L64P_SCP5_0
- new net FPGA_L64P_2: JP93.1, U$1.IO_L64P_D8_2
- new net FPGA_L65N_0: JP75.8, U$1.IO_L65N_SCP2_0
- new net FPGA_L65N_2: JP93.4, U$1.IO_L65N_CSO_B_2
- new net FPGA_L65P_0: JP75.7, U$1.IO_L65P_SCP3_0
- new net FPGA_L65P_2: JP93.3, U$1.IO_L65P_INIT_B_2
- new net FPGA_L66N_0: JP95.2, U$1.IO_L66N_SCP0_0
- new net FPGA_L66P_0: JP95.1, U$1.IO_L66P_SCP1_0
- new net FPGA_L74N_1: JP91.2, U$1.IO_L74N_DOUT_BUSY_1
- new net FPGA_L74P_1: JP91.1, U$1.IO_L74P_AWAKE_1
- new net FPGA_L83N_3: JP79.8, U$1.IO_L83N_VREF_3
- new net FPGA_L83P_3: JP79.7, U$1.IO_L83P_3
- new net FPGA_PROGRAM_B_2: U$1.PROGRAM_B_2
- new net FPGA_SUSPEND: U$1.SUSPEND
- new net N$87: JP80.7
- new net N$88: JP80.8
- new net NC: JP90.7
- new net PP_3.3V_FPGA: C10.1, C11.1, C12.1, C13.1, C14.1, C15.1, C16.1, C17.1, C5.1, C6.1, C7.1, C8.1, C9.1, JP13.1, JP14.1, JP20.1, JP21.1, JP27.1, JP28.1, JP34.1, JP35.1, JP41.1, JP42.1, JP48.1, JP49.1, JP55.1, JP56.1, JP6.1, JP7.1, U$1.VCCAUX, U$1.VCCAUX@1, U$1.VCCAUX@2, U$1.VCCAUX@3, U$1.VCCAUX@4, U$1.VCCO_0, U$1.VCCO_0@1, U$1.VCCO_0@2, U$1.VCCO_1, U$1.VCCO_1@1, U$1.VCCO_1@2, U$1.VCCO_2, U$1.VCCO_2@1, U$1.VCCO_3, U$1.VCCO_3@1, U$1.VCCO_3@2
- net CONGND: now also JP58.1, JP62.1, JP63.1, JP67.1, JP70.1; no longer JP74.1, JP75.1, JP77.1, JP78.1, JP80.1
- net G2: now also JP58.2; no longer JP60.2
- net G3: now also JP61.2; no longer JP65.2
- net G4: now also JP63.2; no longer JP66.2
- net G5: now also JP65.2; no longer JP69.2
- net G6: now also JP67.2; no longer JP72.2
- net G7: now also JP69.2; no longer JP75.2
- net G8: now also JP71.2; no longer JP78.2
- net GND: now also JP58.3, JP62.3, JP63.3, JP67.3, JP70.3; no longer JP74.3, JP75.3, JP77.3, JP78.3, JP80.3
- net GSENSE1: now also OK3.A1
- net GSENSE2: now also JP60.2; no longer JP61.2, OK3.A1
- net GSENSE3: now also JP62.2; no longer JP64.2
- net GSENSE4: now also JP64.2; no longer JP68.2
- net GSENSE5: now also JP66.2; no longer JP71.2
- net GSENSE6: now also JP68.2; no longer JP74.2
- net GSENSE7: now also JP70.2; no longer JP77.2
- net GSENSE8: now also JP72.2; no longer JP80.2
- net TCK: now also U$1.TCK
- net TDI: now also U$1.TDI
- net TDO: now also U$1.TDO
- net TMS: now also U$1.TMS

Commit message: updated circuits
Connections:
- net CONGND: now also JP59.2, OK1.A1; no longer JP57.1, JP59.1
- net GSENSE1: now also JP57.1, JP59.1; no longer JP59.2, OK1.A1
Changed lines of the file:
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@@
 <setting verticaltext="up"/>
 </settings>
-<grid distance="0.1" unitdist="inch" unit="inch" style="lines" multiple="1" display="no" altdistance="0.05" altunitdist="inch" altunit="inch"/>
+<grid distance="0.1" unitdist="inch" unit="inch" style="lines" multiple="1" display="no" altdistance="0.01" altunitdist="inch" altunit="inch"/>
 <layers>
 <layer number="1" name="Top" color="4" fill="1" visible="no" active="no"/>
@@
 <net name="CONGND" class="0">
 <segment>
+<label x="68.58" y="48.26" size="1.27" layer="95" xref="yes"/>
+<wire x1="68.58" y1="48.26" x2="68.58" y2="53.34" width="0.1524" layer="91"/>
+<pinref part="JP59" gate="1" pin="2"/>
+<wire x1="68.58" y1="53.34" x2="58.42" y2="53.34" width="0.1524" layer="91"/>
+<wire x1="58.42" y1="53.34" x2="58.42" y2="50.8" width="0.1524" layer="91"/>
+</segment>
+<segment>
+<pinref part="OK1" gate="-1" pin="A1"/>
+<wire x1="25.4" y1="58.42" x2="27.94" y2="58.42" width="0.1524" layer="91"/>
+<label x="27.94" y="58.42" size="1.27" layer="95" rot="R270" xref="yes"/>
+</segment>
+</net>
+<net name="GSENSE1" class="0">
+<segment>
+<pinref part="OK2" gate="-1" pin="A1"/>
+<wire x1="40.64" y1="7.62" x2="43.18" y2="7.62" width="0.1524" layer="91"/>
+<label x="43.18" y="7.62" size="1.27" layer="95" rot="R270" xref="yes"/>
+</segment>
+<segment>
+<pinref part="X1" gate="-4" pin="S"/>
+<wire x1="68.58" y1="63.5" x2="60.96" y2="63.5" width="0.1524" layer="91"/>
+<label x="60.96" y="55.88" size="1.27" layer="95" xref="yes"/>
+<pinref part="JP59" gate="1" pin="1"/>
+<wire x1="60.96" y1="50.8" x2="60.96" y2="63.5" width="0.1524" layer="91"/>
+</segment>
+<segment>
 <pinref part="JP57" gate="1" pin="1"/>
 <wire x1="-5.08" y1="55.88" x2="2.54" y2="55.88" width="0.1524" layer="91"/>
@@
 <wire x1="2.54" y1="55.88" x2="2.54" y2="50.8" width="0.1524" layer="91"/>
 </segment>
-<segment>
-<pinref part="JP59" gate="1" pin="1"/>
-<wire x1="60.96" y1="50.8" x2="68.58" y2="50.8" width="0.1524" layer="91"/>
-<wire x1="68.58" y1="50.8" x2="68.58" y2="48.26" width="0.1524" layer="91"/>
-<label x="68.58" y="48.26" size="1.27" layer="95" xref="yes"/>
-</segment>
-</net>
-<net name="GSENSE1" class="0">
-<segment>
-<pinref part="OK2" gate="-1" pin="A1"/>
-<wire x1="40.64" y1="7.62" x2="43.18" y2="7.62" width="0.1524" layer="91"/>
-<label x="43.18" y="7.62" size="1.27" layer="95" rot="R270" xref="yes"/>
-</segment>
-<segment>
-<pinref part="X1" gate="-4" pin="S"/>
-<wire x1="68.58" y1="63.5" x2="58.42" y2="63.5" width="0.1524" layer="91"/>
-<pinref part="JP59" gate="1" pin="2"/>
-<wire x1="58.42" y1="63.5" x2="58.42" y2="50.8" width="0.1524" layer="91"/>
-<label x="58.42" y="55.88" size="1.27" layer="95" xref="yes"/>
-</segment>
-<segment>
-<pinref part="OK1" gate="-1" pin="A1"/>
-<wire x1="25.4" y1="58.42" x2="27.94" y2="58.42" width="0.1524" layer="91"/>
-<label x="27.94" y="58.42" size="1.27" layer="95" rot="R270" xref="yes"/>
-</segment>
-</net>
+</net>
