File: Electrical Schematics/Version2/Schematics/boardv2fpga.sch (EAGLE design)
At the start: 159 parts, among them Q1 ASFL1

Commit message: FPGA and isolation
Parts:
- removed JP10, JP11, JP12, JP13, JP14, JP15, JP16, JP17, JP18, JP19, JP20, JP21, JP22, JP23, JP24, JP25, JP26, JP27, JP28, JP29, JP30, JP31, JP32, JP33, JP34, JP35, JP36, JP37, JP38, JP39, JP40, JP41, JP42, JP43, JP44, JP45, JP46, JP47, JP48, JP49, JP50, JP51, JP52, JP53, JP54, JP55, JP56, JP57, JP58, JP59, JP60, JP61, JP62, JP63, JP64, JP65, JP66, JP67, JP68, JP69, JP70, JP71, JP72, JP9: (no value), jumper:JP2E
- removed OK1, OK10, OK11, OK12, OK13, OK14, OK15, OK16, OK2, OK3, OK4, OK5, OK6, OK7, OK8, OK9: MOC3043S, optocoupler:MOC3043S
- removed R1, R10, R11, R12, R13, R14, R15, R16, R17, R18, R19, R2, R20, R21, R22, R23, R24, R25, R26, R27, R28, R29, R3, R30, R31, R32, R4, R5, R6, R7, R8, R9: (no value), SparkFun-Passives:RESISTOR0603-RES
- added C18: 10uF, SparkFun-Capacitors:CAP0603-CAP
- added C19: 1uF, SparkFun-Capacitors:CAP0603-CAP
- added C20, C21, C22, C23, C24, C25, C26, C27, C28, C29, C30, C31, C32, C33, C34, C35: .1uF, SparkFun-Capacitors:CAP0603-CAP
- added R33: 10k, SparkFun-Passives:RESISTOR0603-RES
- added U$10, U$11, U$12, U$13, U$14, U$15, U$16, U$17, U$18, U$19, U$4, U$5, U$6, U$7, U$8, U$9: DPDTSWITCH, shit:DPDTSWITCH
- added U$3: 1.2VREG, shit:1.2VREG
- added U1, U2, U3, U4, U5, U6, U7, U8: ADUM3442CRWZ, digital-isolator:ADUM3442CRWZ
Connections:
- removed net 3.3V: Q1.OE
- removed net G1: JP57.2, OK1.C, OK2.C
- removed net G2: JP58.2, OK3.C, OK4.C
- removed net G3: JP61.2, OK5.C, OK6.C
- removed net G4: JP63.2, OK7.C, OK8.C
- removed net G5: JP65.2, OK10.C, OK9.C
- removed net G6: JP67.2, OK11.C, OK12.C
- removed net G7: JP69.2, OK13.C, OK14.C
- removed net G8: JP71.2, OK15.C, OK16.C
- removed net GSENSE1: JP57.1, JP59.1, OK2.A1, OK3.A1, X1-4.S
- removed net GSENSE2: JP60.2, OK4.A1, X2-4.S
- removed net GSENSE3: JP62.2, OK5.A1, OK6.A1, X3-4.S
- removed net GSENSE4: JP64.2, OK7.A1, OK8.A1, X4-4.S
- removed net GSENSE5: JP66.2, OK10.A1, OK9.A1, X5-4.S
- removed net GSENSE6: JP68.2, OK11.A1, OK12.A1, X6-4.S
- removed net GSENSE7: JP70.2, OK13.A1, OK14.A1, X7-4.S
- removed net GSENSE8: JP72.2, OK15.A1, OK16.A1, X8-4.S
- removed net N$41: JP30.1, JP31.1, X5-2.S
- removed net N$42: JP32.1, JP33.1, X5-3.S
- removed net N$43: JP31.2, OK9.A2, R19.1
- removed net N$44: OK10.A, R17.2
- removed net N$45: JP32.2, R17.1
- removed net N$46: OK9.A, R18.2
- removed net N$47: JP30.2, R18.1
- removed net N$48: JP34.2, R19.2
- removed net N$49: JP33.2, OK10.A2, R20.1
- removed net N$50: JP35.2, R20.2
- removed net N$51: JP37.1, JP38.1, X6-2.S
- removed net N$52: JP39.1, JP40.1, X6-3.S
- removed net N$53: JP38.2, OK11.A2, R23.1
- removed net N$54: OK12.A, R21.2
- removed net N$55: JP39.2, R21.1
- removed net N$56: OK11.A, R22.2
- removed net N$57: JP37.2, R22.1
- removed net N$58: JP41.2, R23.2
- removed net N$59: JP40.2, OK12.A2, R24.1
- removed net N$60: JP42.2, R24.2
- removed net N$61: JP44.1, JP45.1, X7-2.S
- removed net N$62: JP46.1, JP47.1, X7-3.S
- removed net N$63: JP45.2, OK13.A2, R27.1
- removed net N$64: OK14.A, R25.2
- removed net N$65: JP46.2, R25.1
- removed net N$66: OK13.A, R26.2
- removed net N$67: JP44.2, R26.1
- removed net N$68: JP48.2, R27.2
- removed net N$69: JP47.2, OK14.A2, R28.1
- removed net N$70: JP49.2, R28.2
- removed net N$71: JP51.1, JP52.1, X8-2.S
- removed net N$72: JP53.1, JP54.1, X8-3.S
- removed net N$73: JP52.2, OK15.A2, R31.1
- removed net N$74: OK16.A, R29.2
- removed net N$75: JP53.2, R29.1
- removed net N$76: OK15.A, R30.2
- removed net N$77: JP51.2, R30.1
- removed net N$78: JP55.2, R31.2
- removed net N$79: JP54.2, OK16.A2, R32.1
- removed net N$80: JP56.2, R32.2
- new net 3.3V_SUPERVISED: C21.1, C23.1, C25.1, C27.1, C29.1, C31.1, C33.1, C35.1, U1.VDD1, U1.VE1, U2.VDD1, U2.VE1, U3.VDD1, U3.VE1, U4.VDD1, U4.VE1, U5.VDD1, U5.VE1, U6.VDD1, U6.VE1, U7.VDD1, U7.VE1, U8.VDD1, U8.VE1
- new net VIAA: U$5.4, U1.VIA
- new net VIAB: U$7.4, U2.VIA
- new net VIAC: U$9.4, U3.VIA
- new net VIAD: U$11.4, U4.VIA
- new net VIAE: U$13.4, U5.VIA
- new net VIAF: U$15.4, U6.VIA
- new net VIAG: U$17.4, U7.VIA
- new net VIAH: U$19.4, U8.VIA
- new net VIBA: U$4.4, U1.VIB
- new net VIBB: U$6.4, U2.VIB
- new net VIBC: U$8.4, U3.VIB
- new net VIBD: U$10.4, U4.VIB
- new net VIBE: U$12.4, U5.VIB
- new net VIBF: U$14.4, U6.VIB
- new net VIBG: U$16.4, U7.VIB
- new net VIBH: U$18.4, U8.VIB
- new net VOBA: U$4.1, U1.VOB
- new net VOBB: U$6.1, U2.VOB
- new net VOBC: U$8.1, U3.VOB
- new net VOBD: U$10.1, U4.VOB
- new net VOBE: U$12.1, U5.VOB
- new net VOBF: U$14.1, U6.VOB
- new net VOBG: U$16.1, U7.VOB
- new net VOBH: U$18.1, U8.VOB
- new net VOCA: U$5.6, U1.VOC
- new net VOCB: U$7.6, U2.VOC
- new net VOCC: U$9.6, U3.VOC
- new net VOCD: U$11.6, U4.VOC
- new net VOCE: U$13.6, U5.VOC
- new net VOCF: U$15.6, U6.VOC
- new net VOCG: U$17.6, U7.VOC
- new net VOCH: U$19.6, U8.VOC
- new net VODA: U$4.6, U1.VOD
- new net VODB: U$6.6, U2.VOD
- new net VODC: U$8.6, U3.VOD
- new net VODD: U$10.6, U4.VOD
- new net VODE: U$12.6, U5.VOD
- new net VODF: U$14.6, U6.VOD
- new net VODG: U$16.6, U7.VOD
- new net VODH: U$18.6, U8.VOD
- net CONGND: now also C20.2, C22.2, C24.2, C26.2, C28.2, C30.2, C32.2, C34.2, U1.GND2, U1.GND2_2, U2.GND2, U2.GND2_2, U3.GND2, U3.GND2_2, U4.GND2, U4.GND2_2, U5.GND2, U5.GND2_2, U6.GND2, U6.GND2_2, U7.GND2, U7.GND2_2, U8.GND2, U8.GND2_2, X1-4.S, X2-4.S, X3-4.S, X4-4.S, X5-4.S, X6-4.S, X7-4.S, X8-4.S; no longer JP58.1, JP59.2, JP60.1, JP61.1, JP62.1, JP63.1, JP64.1, JP65.1, JP66.1, JP67.1, JP68.1, JP69.1, JP70.1, JP71.1, JP72.1, OK1.A1
- net FPGA_L33N_1_MODULED_ISOLATOR: now also U$10.COM2; no longer JP23.3, JP24.3
- net FPGA_L33P_1_MODULED_ISOLATOR: now also U$11.COM2; no longer JP25.3, JP26.3
- net FPGA_L34N_1_MODULEC_ISOLATOR: now also U$8.COM2; no longer JP16.3, JP17.3
- net FPGA_L34P_1_MODULEC_ISOLATOR: now also U$9.COM2; no longer JP18.3, JP19.3
- net FPGA_L40N_1_MODULEB_ISOLATOR: now also U$6.COM2; no longer JP10.3, JP9.3
- net FPGA_L40P_1_MODULEB_ISOLATOR: now also U$7.COM2; no longer JP11.3, JP12.3
- net FPGA_L41N_1_MODULEA_ISOLATOR: now also U$4.COM2; no longer JP2.3, JP3.3
- net FPGA_L41P_1_MODULEA_ISOLATOR: now also U$5.COM2; no longer JP4.3, JP5.3
- net FPGA_L49N_3_MODULEH_ISOLATOR: now also U$18.COM2; no longer JP51.3, JP52.3
- net FPGA_L49P_3_MODULEH_ISOLATOR: now also U$19.COM2; no longer JP53.3, JP54.3
- net FPGA_L50N_3_MODULEG_ISOLATOR: now also U$16.COM2; no longer JP44.3, JP45.3
- net FPGA_L50P_3_MODULEG_ISOLATOR: now also U$17.COM2; no longer JP46.3, JP47.3
- net FPGA_L51N_3_MODULEF_ISOLATOR: now also U$14.COM2; no longer JP37.3, JP38.3
- net FPGA_L51P_3_MODULEF_ISOLATOR: now also U$15.COM2; no longer JP39.3, JP40.3
- net FPGA_L52N_3_MODULEE_ISOLATOR: now also U$12.COM2; no longer JP30.3, JP31.3
- net FPGA_L52P_3_MODULEE_ISOLATOR: now also U$13.COM2; no longer JP32.3, JP33.3
- net FPGA_SUSPEND: now also R33.1
- net GND: now also C18.2, C19.2, C21.2, C23.2, C25.2, C27.2, C29.2, C31.2, C33.2, C35.2, R33.2, U$3.GND, U1.GND1, U1.GND1_2, U2.GND1, U2.GND1_2, U3.GND1, U3.GND1_2, U4.GND1, U4.GND1_2, U5.GND1, U5.GND1_2, U6.GND1, U6.GND1_2, U7.GND1, U7.GND1_2, U8.GND1, U8.GND1_2; no longer JP57.3, JP58.3, JP59.3, JP60.3, JP61.3, JP62.3, JP63.3, JP64.3, JP65.3, JP66.3, JP67.3, JP68.3, JP69.3, JP70.3, JP71.3, JP72.3
- net N$1: now also U$7.COM1; no longer JP10.1, JP9.1
- net N$10: now also U$6.3, U2.VID; no longer JP6.2, R3.2
- net N$11: now also U$9.COM1, X3-2.S; no longer JP11.1, JP12.1, X2-3.S
- net N$12: now also U$8.COM1, X3-3.S; no longer JP7.2, R4.2
- net N$13: now also U$9.1, U3.VOA; no longer JP10.2, OK3.A2, R7.1
- net N$14: now also U$9.3, U3.VIC; no longer OK4.A, R5.2
- net N$15: now also U$8.3, U3.VID; no longer JP11.2, R5.1
- net N$16: now also U$11.COM1, X4-2.S; no longer OK3.A, R6.2
- net N$17: now also U$10.COM1, X4-3.S; no longer JP9.2, R6.1
- net N$18: now also U$11.1, U4.VOA; no longer JP13.2, R7.2
- net N$19: now also U$11.3, U4.VIC; no longer JP12.2, OK4.A2, R8.1
- net N$2: now also U$5.COM1; no longer JP2.1, JP3.1
- net N$20: now also U$10.3, U4.VID; no longer JP14.2, R8.2
- net N$21: now also U$13.COM1, X5-2.S; no longer JP16.1, JP17.1, X3-2.S
- net N$22: now also U$12.COM1, X5-3.S; no longer JP18.1, JP19.1, X3-3.S
- net N$23: now also U$13.1, U5.VOA; no longer JP17.2, OK5.A2, R11.1
- net N$24: now also U$13.3, U5.VIC; no longer OK6.A, R9.2
- net N$25: now also U$12.3, U5.VID; no longer JP18.2, R9.1
- net N$26: now also U$15.COM1, X6-2.S; no longer OK5.A, R10.2
- net N$27: now also U$14.COM1, X6-3.S; no longer JP16.2, R10.1
- net N$28: now also U$15.1, U6.VOA; no longer JP20.2, R11.2
- net N$29: now also U$15.3, U6.VIC; no longer JP19.2, OK6.A2, R12.1
- net N$3: now also U$5.1, U1.VOA; no longer JP4.1, JP5.1, X1-3.S
- net N$30: now also U$14.3, U6.VID; no longer JP21.2, R12.2
- net N$31: now also U$17.COM1, X7-2.S; no longer JP23.1, JP24.1, X4-2.S
- net N$32: now also U$16.COM1, X7-3.S; no longer JP25.1, JP26.1, X4-3.S
- net N$33: now also U$17.1, U7.VOA; no longer JP24.2, OK7.A2, R15.1
- net N$34: now also U$17.3, U7.VIC; no longer OK8.A, R13.2
- net N$35: now also U$16.3, U7.VID; no longer JP25.2, R13.1
- net N$36: now also U$19.COM1, X8-2.S; no longer OK7.A, R14.2
- net N$37: now also U$18.COM1, X8-3.S; no longer JP23.2, R14.1
- net N$38: now also U$19.1, U8.VOA; no longer JP27.2, R15.2
- net N$39: now also U$19.3, U8.VIC; no longer JP26.2, OK8.A2, R16.1
- net N$4: now also U$5.3, U1.VIC; no longer JP3.2, OK1.A2, R3.1
- net N$40: now also U$18.3, U8.VID; no longer JP28.2, R16.2
- net N$5: now also U$4.3, U1.VID; no longer OK2.A, R1.2
- net N$6: now also U$4.COM1, X1-3.S; no longer OK1.A, R2.2
- net N$7: now also U$6.COM1, X2-3.S; no longer JP4.2, R1.1
- net N$8: now also U$7.1, U2.VOA; no longer JP2.2, R2.1
- net N$9: now also U$7.3, U2.VIC; no longer JP5.2, OK2.A2, R4.1
- net PP_3.3V_FPGA: now also C19.1, Q1.OE, U$3.VIN; no longer JP13.1, JP14.1, JP20.1, JP21.1, JP27.1, JP28.1, JP34.1, JP35.1, JP41.1, JP42.1, JP48.1, JP49.1, JP55.1, JP56.1, JP6.1, JP7.1
- net PP_3.3V_MODULARCONNECTOR: now also JP2.3, JP3.3, JP4.3, JP5.3, JP6.3, JP7.3; no longer JP15.3, JP22.3, JP29.3, JP36.3, JP43.3, JP50.3
- net PP_5V_MODULARCONNECTOR: now also JP2.1, JP3.1, JP4.1, JP5.1, JP6.1, JP7.1; no longer JP15.1, JP22.1, JP29.1, JP36.1, JP43.1, JP50.1
- net V1: now also C20.1, U1.VDD2, U1.VE2; no longer JP6.3, JP7.3
- net V2: now also C22.1, JP2.2, U2.VDD2, U2.VE2; no longer JP13.3, JP14.3, JP8.2
- net V3: now also C24.1, JP3.2, U3.VDD2, U3.VE2; no longer JP15.2, JP20.3, JP21.3
- net V4: now also C26.1, JP4.2, U4.VDD2, U4.VE2; no longer JP22.2, JP27.3, JP28.3
- net V5: now also C28.1, JP5.2, U5.VDD2, U5.VE2; no longer JP29.2, JP34.3, JP35.3
- net V6: now also C30.1, JP6.2, U6.VDD2, U6.VE2; no longer JP36.2, JP41.3, JP42.3
- net V7: now also C32.1, JP7.2, U7.VDD2, U7.VE2; no longer JP43.2, JP48.3, JP49.3
- net V8: now also C34.1, JP8.2, U8.VDD2, U8.VE2; no longer JP50.2, JP55.3, JP56.3
- net VCCINT: now also C18.1, U$3.TAB, U$3.VOUT
Other:
- note added: "Modular Connector G With Isolation"
- note removed: "1.Anode 4.Emitter 2.Cathode 5.Collector 3.NC 6.Base"
- note removed: "Modular Connector N With Isolation"
