File: Electrical Schematics/Version2/Schematics/boardv2power.sch (EAGLE design)
At the start: 92 parts, among them U1 LM1085_KTT_3, U2 LM1085_KTT_3, U3 LM1084_KTT_3, U4 TPS3514_D_14

Commit message: Change shit's pot and updated power
Parts:
- removed R16, R20, R32, R7, R8: (no value), SparkFun-Passives:RESISTOR0603-RES
- added U$7, U$8, U$9: PVZ3A, shit:PVZ3A
- R17: value (none) -> 470k
- R18, R19, R33: value (none) -> .01
- R31: value (none) -> 1k
Connections:
- net N$19 renamed 12V_SUPERVISED
- net N$21 renamed 5V_SUPERVISED
- net N$22 renamed FAULT_PROTECTION
- net N$25 renamed ON_OFF_CONTROL_INPUT
- net N$29 renamed POWER_GOOD_OUT
- net N$53 renamed 3.3V_SUPERVISED
- removed net N$10: R8.1
- removed net N$17: R7.2, R8.2, TP11.TP, U4.PGI
- removed net N$18: R16.1, R18.1, TP10.TP
- removed net N$23: R17.1, TP20.TP, U4.VDD
- removed net N$26: R19.1, R20.2, TP19.TP
- removed net N$27: R31.2, R32.2, R33.1
- new net 12V_UNSUPERVISED: R18.1, TP10.TP, U$7.P$1
- new net 3.3V_UNSUPERVISED: R31.2, R33.1, U$8.P$2
- new net 5V_TO_SUPERVISOR: R17.1, TP11.TP, TP20.TP, U4.PGI, U4.VDD
- new net 5V_UNSUPERVISED: R19.1, TP19.TP, U$9.P$2
- new net N$55: U$9.P$1, U4.IS5
- net GND: now also U$7.P$3, U$8.P$3, U$9.P$3; no longer R7.1
- net N$28: no longer R20.1, U4.IS5
- net N$48: now also U$8.P$1; no longer R32.1
- net N$54: now also U$7.P$2; no longer R16.2
Other:
- note removed: "12V"
- note removed: "3.3V"
- note removed: "5V"
- note removed: "5V VSB"
- note removed: "PG"
- moved on the sheet: R15, TP16, TP18

Commit message: Updated Power
Parts:
- removed R14, R15, RS, RS1, RS2: (no value), SparkFun-Passives:RESISTOR0603-RES
- added C13, C14: 10u, eagle-ltspice:CC0603
- added JP6, JP7, JP8: (no value), jumper:JP1Q
- added R7, R8: 121, SparkFun-Passives:RESISTOR0603-RES
- added TP30, TP31: TPB1,27, testpad:TPB1,27
- added U$14, U$15, U$16: PVG3A, shit:PVG3A
- added U$17: PVZ3A, shit:PVZ3A
- added U5: LM1085_KTT_3, shit:LM1085_KTT_3
- C11, C12, C8: value (none) -> .1u
- C2, C3, C4, C5, C6, C7: value (none) -> 10u
- R10, R11, R12, R13, R4, R9: value (none) -> 121
- U$7, U$8, U$9: DIGI (none) -> 987-1549-ND
Connections:
- net N$48 renamed IS33
- net N$54 renamed IS12
- net N$8 renamed MCU_+3.3V
- removed net N$28: C11.2
- removed net N$34: R21.1, RS1.2, U$3.VIN
- removed net N$42: RS2.1, U$5.SENSE, U$6.D
- removed net N$43: R26.1, RS2.2, U$5.VIN
- removed net N$49: JP1.1, TP4.TP
- removed net N$50: C6.1, JP2.1, TP6.TP
- removed net N$51: JP3.1, TP7.TP
- removed net N$55: U$9.P$1, U4.IS5
- new net CONNECTOR_ELECTRONIC_BATTERY: JP4.2
- new net IS5: C11.2, U$9.P$1, U4.IS5
- new net N$10: JP6.2, R7.1, TP30.TP, U5.OUTPUT
- new net N$17: R7.2, R9.1, U5.ADJ/GND
- new net N$19: C3.1, JP7.1, U1.INPUT
- new net N$21: C13.1, JP8.1, U5.INPUT
- net 12V_UNSUPERVISED: now also JP1.1, TP4.TP
- net 3.3V_SUPERVISED: now also R1.1, R21.1, R26.1, TP28.TP, U$14.P$1, U$15.P$1, U$16.P$1, U$3.VIN, U$5.VIN
- net 3.3V_UNSUPERVISED: now also JP3.1, TP7.TP
- net 5V_TO_SUPERVISOR: now also C14.1, JP6.1, TP31.TP
- net 5V_UNSUPERVISED: now also C6.1, JP2.1, TP6.TP
- net GND: now also C13.2, C14.2, R11.2, R8.2, U$14.P$3, U$16.P$3, U$17.P$1, U$17.P$3, U5.EPAD; no longer R14.2, R15.1
- net N$11: now also R8.1; no longer R9.1
- net N$14: now also C7.1
- net N$15: now also R11.1; no longer R12.1
- net N$16: now also R12.1; no longer R14.1
- net N$20: now also U$17.P$2; no longer R15.2
- net N$33: now also U$16.P$2; no longer RS1.1
- net N$4: now also U$15.P$2, U$5.SENSE, U$6.D; no longer R1.1, RS.2, TP28.TP
- net N$5: now also U$14.P$2; no longer RS.1
- net N$52: now also JP5.1
- net VOLTAGEJMP_+_TO_INPUT_VREG: now also JP7.2, JP8.2; no longer C3.1, U1.INPUT
Other:
- moved on the sheet: C2, C3, C4, C5, C6, C7, JP1, JP2, JP3, JP4, JP5, R10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

Commit message: updated power and ethernet
Parts:
- removed C10: (no value), eagle-ltspice:CC0603
- removed R26, R27, R28, R29, R30: (no value), SparkFun-Passives:RESISTOR0603-RES
- removed U$15: PVG3A, shit:PVG3A
- removed U$5: LM25061_DGS_10, shit:LM25061_DGS_10
- removed U$6: FDD8874, transistor-fet:FDD8874
Connections:
- removed net N$39: C10.1, U$5.TIMER
- removed net N$4: U$15.P$2, U$5.SENSE, U$6.D
- removed net N$40: R27.2, U$5.PWR
- removed net N$41: R26.2, R28.2, U$5.UVLO/EN
- removed net N$44: U$5.GATE, U$6.G
- removed net N$45: R29.2, R30.1, U$5.FB
- removed net N$46: R29.1, U$5.OUT, U$6.S
- removed net N$47: U$5.PGD
- net 3.3V_SUPERVISED: no longer R26.1, U$15.P$1, U$5.VIN
- net GND: no longer C10.2, R27.1, R28.1, R30.2, U$5.GND
Other:
- note removed: "Protection circuit for the Battery Monitoring Circuit"
Changed lines of the file:
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@@
 <setting verticaltext="up"/>
 </settings>
-<grid distance="0.1" unitdist="inch" unit="inch" style="lines" multiple="1" display="yes" altdistance="0.05" altunitdist="inch" altunit="inch"/>
+<grid distance="0.1" unitdist="inch" unit="inch" style="lines" multiple="1" display="no" altdistance="0.01" altunitdist="inch" altunit="inch"/>
 <layers>
 <layer number="1" name="Top" color="4" fill="1" visible="no" active="no"/>
@@
 <part name="R25" library="SparkFun-Passives" deviceset="RESISTOR" device="0603-RES"/>
 <part name="SUPPLY21" library="supply2" deviceset="GND" device=""/>
-<part name="U$5" library="shit" deviceset="LM25061_DGS_10" device=""/>
-<part name="U$6" library="transistor-fet" deviceset="FDD8874" device=""/>
-<part name="R26" library="SparkFun-Passives" deviceset="RESISTOR" device="0603-RES"/>
-<part name="R27" library="SparkFun-Passives" deviceset="RESISTOR" device="0603-RES"/>
-<part name="R28" library="SparkFun-Passives" deviceset="RESISTOR" device="0603-RES"/>
-<part name="C10" library="eagle-ltspice" deviceset="C" device="C0603"/>
-<part name="SUPPLY22" library="supply2" deviceset="GND" device=""/>
-<part name="SUPPLY23" library="supply2" deviceset="GND" device=""/>
-<part name="SUPPLY24" library="supply2" deviceset="GND" device=""/>
-<part name="SUPPLY25" library="supply2" deviceset="GND" device=""/>
-<part name="R29" library="SparkFun-Passives" deviceset="RESISTOR" device="0603-RES"/>
-<part name="R30" library="SparkFun-Passives" deviceset="RESISTOR" device="0603-RES"/>
-<part name="SUPPLY26" library="supply2" deviceset="GND" device=""/>
 <part name="FRAME2" library="frames" deviceset="DOCFIELD" device=""/>
 <part name="FRAME3" library="frames" deviceset="DOCFIELD" device=""/>
 <part name="FRAME4" library="frames" deviceset="DOCFIELD" device=""/>
-<part name="FRAME5" library="frames" deviceset="DOCFIELD" device=""/>
 <part name="JP1" library="jumper" deviceset="JP1Q" device=""/>
 <part name="JP2" library="jumper" deviceset="JP1Q" device=""/>
@@
 <part name="SUPPLY33" library="supply2" deviceset="GND" device=""/>
 <part name="U$16" library="shit" deviceset="PVG3A" device="">
-<attribute name="BITECH" value="84WR10LF"/>
-</part>
-<part name="U$15" library="shit" deviceset="PVG3A" device="">
 <attribute name="BITECH" value="84WR10LF"/>
 </part>
@@
 </segment>
 </net>
-</nets>
-</sheet>
-<sheet>
-<description>power monitoring FPGA</description>
-<plain>
-<frame x1="-22.86" y1="-2.54" x2="172.72" y2="116.84" columns="8" rows="5" layer="91"/>
-<text x="-15.24" y="104.14" size="5.08" layer="91">Power Block</text>
-<text x="-15.24" y="96.52" size="1.778" layer="91">Protection circuit for the Battery Monitoring Circuit</text>
-</plain>
-<instances>
-<instance part="U$5" gate="A" x="17.78" y="66.04"/>
-<instance part="U$6" gate="A" x="88.9" y="78.74" rot="R90"/>
-<instance part="R26" gate="G$1" x="-5.08" y="68.58" rot="R270"/>
-<instance part="R27" gate="G$1" x="109.22" y="58.42" rot="R180"/>
-<instance part="R28" gate="G$1" x="-5.08" y="50.8" rot="R90"/>
-<instance part="C10" gate="G$1" x="93.98" y="55.88" rot="R90"/>
-<instance part="SUPPLY22" gate="GND" x="116.84" y="55.88"/>
-<instance part="SUPPLY23" gate="GND" x="101.6" y="53.34"/>
-<instance part="SUPPLY24" gate="GND" x="15.24" y="53.34"/>
-<instance part="SUPPLY25" gate="GND" x="-5.08" y="43.18"/>
-<instance part="R29" gate="G$1" x="121.92" y="73.66" rot="R270"/>
-<instance part="R30" gate="G$1" x="5.08" y="50.8" rot="R270"/>
-<instance part="SUPPLY26" gate="GND" x="5.08" y="40.64"/>
-<instance part="FRAME5" gate="G$1" x="66.04" y="2.54"/>
-<instance part="U$15" gate="G$1" x="5.08" y="68.58" rot="R90">
-<attribute name="BITECH" x="5.08" y="68.58" size="1.778" layer="96" rot="R90" display="off"/>
-</instance>
-</instances>
-<busses>
-</busses>
-<nets>
-<net name="N$39" class="0">
-<segment>
-<pinref part="U$5" gate="A" pin="TIMER"/>
-<pinref part="C10" gate="G$1" pin="1"/>
-<wire x1="88.9" y1="55.88" x2="91.44" y2="55.88" width="0.1524" layer="91"/>
-</segment>
-</net>
-<net name="N$40" class="0">
-<segment>
-<pinref part="U$5" gate="A" pin="PWR"/>
-<pinref part="R27" gate="G$1" pin="2"/>
-<wire x1="88.9" y1="58.42" x2="104.14" y2="58.42" width="0.1524" layer="91"/>
-</segment>
-</net>
-<net name="GND" class="0">
-<segment>
-<pinref part="R27" gate="G$1" pin="1"/>
-<pinref part="SUPPLY22" gate="GND" pin="GND"/>
-<wire x1="116.84" y1="58.42" x2="114.3" y2="58.42" width="0.1524" layer="91"/>
-</segment>
-<segment>
-<pinref part="C10" gate="G$1" pin="2"/>
-<pinref part="SUPPLY23" gate="GND" pin="GND"/>
-<wire x1="101.6" y1="55.88" x2="99.06" y2="55.88" width="0.1524" layer="91"/>
-</segment>
-<segment>
-<pinref part="U$5" gate="A" pin="GND"/>
-<pinref part="SUPPLY24" gate="GND" pin="GND"/>
-<wire x1="15.24" y1="55.88" x2="17.78" y2="55.88" width="0.1524" layer="91"/>
-</segment>
-<segment>
-<pinref part="R28" gate="G$1" pin="1"/>
-<pinref part="SUPPLY25" gate="GND" pin="GND"/>
-</segment>
-<segment>
-<pinref part="R30" gate="G$1" pin="2"/>
-<pinref part="SUPPLY26" gate="GND" pin="GND"/>
-<wire x1="5.08" y1="45.72" x2="5.08" y2="43.18" width="0.1524" layer="91"/>
-</segment>
-</net>
-<net name="N$41" class="0">
-<segment>
-<pinref part="R28" gate="G$1" pin="2"/>
-<pinref part="R26" gate="G$1" pin="2"/>
-<wire x1="-5.08" y1="55.88" x2="-5.08" y2="60.96" width="0.1524" layer="91"/>
-<pinref part="U$5" gate="A" pin="UVLO/EN"/>
-<wire x1="-5.08" y1="60.96" x2="-5.08" y2="63.5" width="0.1524" layer="91"/>
-<wire x1="17.78" y1="60.96" x2="-5.08" y2="60.96" width="0.1524" layer="91"/>
-<junction x="-5.08" y="60.96"/>
-</segment>
-</net>
-<net name="3.3V_SUPERVISED" class="0">
-<segment>
-<pinref part="R26" gate="G$1" pin="1"/>
-<wire x1="-5.08" y1="73.66" x2="-17.78" y2="73.66" width="0.1524" layer="91"/>
-<wire x1="-5.08" y1="73.66" x2="0" y2="73.66" width="0.1524" layer="91"/>
-<wire x1="0" y1="73.66" x2="0" y2="63.5" width="0.1524" layer="91"/>
-<pinref part="U$5" gate="A" pin="VIN"/>
-<wire x1="17.78" y1="63.5" x2="5.08" y2="63.5" width="0.1524" layer="91"/>
-<junction x="-5.08" y="73.66"/>
-<label x="-17.78" y="73.66" size="1.778" layer="95" rot="R180" xref="yes"/>
-<pinref part="U$15" gate="G$1" pin="P$1"/>
-<wire x1="5.08" y1="63.5" x2="0" y2="63.5" width="0.1524" layer="91"/>
-<junction x="5.08" y="63.5"/>
-</segment>
-</net>
-<net name="N$44" class="0">
-<segment>
-<pinref part="U$6" gate="A" pin="G"/>
-<wire x1="91.44" y1="76.2" x2="91.44" y2="66.04" width="0.1524" layer="91"/>
-<pinref part="U$5" gate="A" pin="GATE"/>
-<wire x1="91.44" y1="66.04" x2="88.9" y2="66.04" width="0.1524" layer="91"/>
-</segment>
-</net>
-<net name="N$45" class="0">
-<segment>
-<pinref part="U$5" gate="A" pin="FB"/>
-<wire x1="17.78" y1="58.42" x2="12.7" y2="58.42" width="0.1524" layer="91"/>
-<wire x1="12.7" y1="58.42" x2="12.7" y2="43.18" width="0.1524" layer="91"/>
-<wire x1="12.7" y1="43.18" x2="121.92" y2="43.18" width="0.1524" layer="91"/>
-<wire x1="121.92" y1="43.18" x2="121.92" y2="68.58" width="0.1524" layer="91"/>
-<pinref part="R29" gate="G$1" pin="2"/>
-<wire x1="12.7" y1="58.42" x2="5.08" y2="58.42" width="0.1524" layer="91"/>
-<wire x1="5.08" y1="58.42" x2="5.08" y2="55.88" width="0.1524" layer="91"/>
-<pinref part="R30" gate="G$1" pin="1"/>
-<junction x="12.7" y="58.42"/>
-</segment>
-</net>
-<net name="N$46" class="0">
-<segment>
-<pinref part="U$6" gate="A" pin="S"/>
-<wire x1="93.98" y1="81.28" x2="96.52" y2="81.28" width="0.1524" layer="91"/>
-<wire x1="96.52" y1="81.28" x2="96.52" y2="63.5" width="0.1524" layer="91"/>
-<pinref part="U$5" gate="A" pin="OUT"/>
-<wire x1="96.52" y1="63.5" x2="88.9" y2="63.5" width="0.1524" layer="91"/>
-<junction x="96.52" y="81.28"/>
-<wire x1="96.52" y1="81.28" x2="121.92" y2="81.28" width="0.1524" layer="91"/>
-<pinref part="R29" gate="G$1" pin="1"/>
-<wire x1="121.92" y1="81.28" x2="127" y2="81.28" width="0.1524" layer="91"/>
-<wire x1="121.92" y1="78.74" x2="121.92" y2="81.28" width="0.1524" layer="91"/>
-<junction x="121.92" y="81.28"/>
-</segment>
-</net>
-<net name="N$47" class="0">
-<segment>
-<pinref part="U$5" gate="A" pin="PGD"/>
-<wire x1="88.9" y1="60.96" x2="111.76" y2="60.96" width="0.1524" layer="91"/>
-</segment>
-</net>
-<net name="N$4" class="0">
-<segment>
-<pinref part="U$5" gate="A" pin="SENSE"/>
-<wire x1="5.08" y1="73.66" x2="17.78" y2="73.66" width="0.1524" layer="91"/>
-<wire x1="17.78" y1="73.66" x2="17.78" y2="66.04" width="0.1524" layer="91"/>
-<wire x1="17.78" y1="73.66" x2="17.78" y2="81.28" width="0.1524" layer="91"/>
-<pinref part="U$6" gate="A" pin="D"/>
-<wire x1="17.78" y1="81.28" x2="83.82" y2="81.28" width="0.1524" layer="91"/>
-<junction x="17.78" y="73.66"/>
-<pinref part="U$15" gate="G$1" pin="P$2"/>
-</segment>
-</net>
