File: Electrical Schematics/Version2/Schematics/boardv2battery.sch (EAGLE design)
At the start: 52 parts, among them K1 CB1A-P-12V, K2 CB1A-P-12V, K3 CB1A-P-12V, K4 CB1A-P-12V

Commit message: updated everything
Other:
- note added: "Battery Monitoring Block A"
- note added: "Battery Monitoring Block B"
- note added: "Battery Monitoring Block C"
- note added: "Battery Monitoring Block D"
Changed lines of the file:
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@@
 <setting verticaltext="up"/>
 </settings>
-<grid distance="0.05" unitdist="inch" unit="inch" style="lines" multiple="1" display="no" altdistance="0.025" altunitdist="inch" altunit="inch"/>
+<grid distance="0.1" unitdist="inch" unit="inch" style="lines" multiple="1" display="no" altdistance="0.01" altunitdist="inch" altunit="inch"/>
 <layers>
 <layer number="1" name="Top" color="4" fill="1" visible="no" active="no"/>
@@
 <part name="SUPPLY24" library="supply2" deviceset="GND" device=""/>
 <part name="JP4" library="jumper" deviceset="JP1E" device=""/>
+<part name="FRAME1" library="frames" deviceset="DOCFIELD" device=""/>
+<part name="FRAME2" library="frames" deviceset="DOCFIELD" device=""/>
+<part name="FRAME3" library="frames" deviceset="DOCFIELD" device=""/>
+<part name="FRAME4" library="frames" deviceset="DOCFIELD" device=""/>
 </parts>
 <sheets>
 <sheet>
 <plain>
+<frame x1="-17.78" y1="-10.16" x2="233.68" y2="157.48" columns="8" rows="5" layer="91"/>
+<text x="-7.62" y="139.7" size="5.08" layer="91">Battery Monitoring Block A</text>
 </plain>
 <instances>
@@
 <instance part="SUPPLY6" gate="GND" x="73.66" y="25.4"/>
 <instance part="JP1" gate="A" x="57.15" y="113.03"/>
+<instance part="FRAME1" gate="G$1" x="127" y="-7.62"/>
 </instances>
 <busses>
@@
 <sheet>
 <plain>
+<text x="-60.96" y="132.08" size="5.08" layer="91">Battery Monitoring Block B</text>
+<frame x1="-81.28" y1="-10.16" x2="170.18" y2="157.48" columns="8" rows="5" layer="91"/>
 </plain>
 <instances>
@@
 <instance part="SUPPLY12" gate="GND" x="5.08" y="30.48"/>
 <instance part="JP2" gate="A" x="-11.43" y="118.11"/>
+<instance part="FRAME2" gate="G$1" x="63.5" y="-7.62"/>
 </instances>
 <busses>
@@
 <sheet>
 <plain>
+<text x="-86.36" y="142.24" size="5.08" layer="91">Battery Monitoring Block C</text>
+<frame x1="-99.06" y1="0" x2="152.4" y2="167.64" columns="8" rows="5" layer="91"/>
 </plain>
 <instances>
@@
 <instance part="SUPPLY18" gate="GND" x="-20.32" y="43.18"/>
 <instance part="JP3" gate="A" x="-36.83" y="130.81"/>
+<instance part="FRAME3" gate="G$1" x="45.72" y="2.54"/>
 </instances>
 <busses>
@@
 <sheet>
 <plain>
+<text x="-68.58" y="129.54" size="5.08" layer="91">Battery Monitoring Block D</text>
+<frame x1="-86.36" y1="-17.78" x2="165.1" y2="149.86" columns="8" rows="5" layer="91"/>
 </plain>
 <instances>
@@
 <instance part="SUPPLY24" gate="GND" x="-3.81" y="30.48"/>
 <instance part="JP4" gate="A" x="-20.32" y="118.11"/>
+<instance part="FRAME4" gate="G$1" x="58.42" y="-15.24"/>
 </instances>
 <busses>

Commit message: updated circuits
Parts:
- added R10, R9: 100UOHMS, SparkFun-Passives:RESISTOR0603-RES
- C4: value (none) -> 220pf
- C5: value (none) -> 4.7UF
- R1: value (none) -> 2.2KOHM
- R2: value (none) -> 100UOHMS
Connections:
- removed net TO_MCU: C4.1, C4.2
- new net CONNECTOR_BATA_+: D1.A1, D1.A2, R1.2
- new net N$11: X1-1.S
- new net N$12: C4.1, X1-2.S
- new net N$45: R10.1, U$1.ISENSEH
- new net N$46: R9.1, U$1.ISENSEL
- new net N$47: C1.1, U$1.VDDA
- net BATA_+TO+_MON: no longer D1.A1, D1.A2, R1.2
- net GND: now also C4.2, R10.2, U$1.DGND1, U$1.GNDSUB, U$1.GNDSUB1, U$1.GNDSUB2, U$1.GNDSUB3; no longer U$1.ISENSEH
- net MON_ISENSEL_TO_-BATA: now also R9.2; no longer U$1.ISENSEL
Other:
- note added: "TEMP CONNECTOR"
- moved on the sheet: C4, C5, D1, R1, R2, X1-1, X1-2

Commit message: Battery Monitor Finished?
Parts:
- removed JP1, JP2, JP3, JP4: (no value), jumper:JP1E
- removed K1, K2, K3, K4: CB1A-P-12V, relay:CB1A-P-12V
- added R11, R12, R13, R14, R15, R16: 100UOHMS, SparkFun-Passives:RESISTOR0603-RES
- C1, C11, C16, C6: value (none) -> 47nF
- C10, C15, C20: value (none) -> 220pf
- C12, C17, C2, C7: value (none) -> 220nF
- C13, C18, C3, C8: value (none) -> 1uF
- C14, C19, C9: value (none) -> 4.7UF
- R3, R5, R7: value (none) -> 2.2KOHM
- R4, R6, R8: value (none) -> 100UOHMS
Connections:
- removed net BATA_+TO+_MON: D2.A1, D2.A2, D3.A1, D3.A2, D4.A1, D4.A2, JP1.2, JP2.2, JP3.2, JP4.2, R3.2, R5.2, R7.2
- removed net CHARGER_+_TO_+_RELAY: JP1.1, JP2.1, JP3.1, JP4.1, K11.1, K21.1, K31.1, K41.1
- removed net CONNECTOR_BATA_+: D1.A1, D1.A2, R1.2
- removed net MON_ISENSEL_TO_-BATA: R2.2, R4.2, R6.2, R8.2, R9.2, U$2.ISENSEL, U$3.ISENSEL, U$4.ISENSEL
- removed net N$13 (its old number): C10.1, D2.C, U$2.VSUP
- removed net N$24 (its old number): C15.1, D3.C, U$3.VSUP
- removed net N$35 (its old number): C20.1, D4.C, U$4.VSUP
- removed net N$9 (its old number): K22.P
- removed net RELAY_+_TO_+_BATA: K11.2, K21.2, K31.2, K41.2
- removed net TO_MCU1: C9.1, C9.2
- removed net TO_MCU2: C14.1, C14.2
- removed net TO_MCU3: C19.1, C19.2
- new net CON_MONB_+: D1.A1, D1.A2, D2.A1, D2.A2, R1.2, R3.2
- new net CON_MONB_-: R11.2, R2.2, R4.2, R9.2
- new net CON_MONC_+: D3.A1, D3.A2, R5.2
- new net CON_MONC_-: R13.2, R6.2
- new net CON_MOND_+: D4.A1, D4.A2, R7.2
- new net CON_MOND_-: R15.2, R8.2
- new net N$18: C10.1, X2-1.S
- new net N$19: X2-2.S
- new net N$21: R12.1, U$2.ISENSEH
- new net N$22: C6.1, U$2.VDDA
- new net N$30: C15.1, X3-1.S
- new net N$31: X3-2.S
- new net N$33: R14.1, U$3.ISENSEH
- new net N$41: C20.1, X4-1.S
- new net N$42: X4-2.S
- new net N$44: R16.1, U$4.ISENSEH
- new net N$48: C3.1, U$1.VDDD2D, U$1.VDDH
- new net N$49: R11.1, U$2.ISENSEL
- new net N$50: C8.1, U$2.VDDD2D, U$2.VDDH
- new net N$51: C11.1, U$3.VDDA
- new net N$52: R13.1, U$3.ISENSEL
- new net N$53: C13.1, U$3.VDDD2D, U$3.VDDH
- new net N$54: C16.1, U$4.VDDA
- new net N$55: R15.1, U$4.ISENSEL
- new net N$56: C18.1, U$4.VDDD2D, U$4.VDDH
- net GND: now also C1.2, C11.2, C13.2, C14.2, C16.2, C18.2, C19.2, C3.2, C6.2, C8.2, C9.2, R12.2, R14.2, R16.2, U$1.AGND, U$2.AGND, U$2.DGND1, U$2.GNDSUB, U$2.GNDSUB1, U$2.GNDSUB2, U$2.GNDSUB3, U$3.AGND, U$3.DGND1, U$3.GNDSUB, U$3.GNDSUB1, U$3.GNDSUB2, U$3.GNDSUB3, U$4.AGND, U$4.DGND1, U$4.GNDSUB, U$4.GNDSUB1, U$4.GNDSUB2, U$4.GNDSUB3; no longer K12.S, K22.S, K32.S, K42.S, U$2.ISENSEH, U$3.ISENSEH, U$4.ISENSEH
- net N$1: now also C9.1, D2.C, U$2.VSUP; no longer K12.P
- net N$11: now also C4.1
- net N$12: no longer C4.1
- net N$23: now also C14.1, D3.C, U$3.VSUP; no longer K32.P
- net N$34: now also C19.1, D4.C, U$4.VSUP; no longer K42.P
Other:
- note added: "Battery Monitor B"
- note removed: "Battery Monitoring Block B"
- moved on the sheet: C1, C10, C11, C12, C13, C14, C15, C16, C17, C18, C19, C2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
