File: Electrical Schematics/Version2/Schematics/boardv2a.brd (EAGLE design)
At the start: 160 x 100 mm, 506 parts, among them IC1 MCP41HVX1ST, IC2 ADUM4160BRW, K5 G5V-2, Q1 IRLML2060TRPBFBSS123LT1G, Q2 IRLML2060TRPBFBSS123LT1G, Q3 IRLML2060TRPBFBSS123LT1G, Q4 IRLML2060TRPBFBSS123LT1G, Q5 IRLML2060TRPBFBSS123LT1G, Q6 IRLML2060TRPBFBSS123LT1G, Q7 ASFL1, U1 CP2130-GM, U2 TMS570LS0432_PZ_100, U2401 VNH2SP30-E, U3 LM1085_KTT_3, U4 LM1085_KTT_3, U5 LM1084_KTT_3, U6 TPS3514_D_14, U7 LM1085_KTT_3

Commit message: updated more of the schematics
Parts:
- added U$14, U$16, U$17, U$18: 4PDT_SWITCH, shit:MMS42
- TP104: value TPB1,27 -> TPTP06R; device testpad:B1,27 -> testpad:TP06R
- moved R92 442.4 mm to (204.5, 108.0), turned to 270 degrees
- moved C3 440.2 mm to (205.7, 104.1)
- moved R93 439.7 mm to (203.2, 111.8)
- moved X1 426.3 mm to (214.6, 104.1), turned to 90 degrees
- moved C4 418.6 mm to (217.2, 109.2), turned to 90 degrees
- moved C17 414.6 mm to (181.6, 105.4)
- moved R2 407.9 mm to (189.2, 86.4)
- moved R4 406.1 mm to (189.2, 90.2)
- moved C19 406.1 mm to (200.7, 101.6)
- moved C16 405.1 mm to (199.4, 106.7)
- moved U$4 402.6 mm to (195.6, 108.0)
- moved R3 401.1 mm to (175.3, 96.5)
- moved R10 400.0 mm to (195.6, 101.6), turned to 180 degrees
- moved R1 393.1 mm to (181.6, 55.9), turned to 180 degrees
- moved R7 392.0 mm to (171.4, 91.4)
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Connections:
- net FPGA_L51P_3_MODULEF_ISOLATOR: now also U$18.P$4, U$18.P$9
Other:
- board size 160 x 100 mm -> 201.9 x 117.8 mm

Commit message: updated board
Parts:
- removed JP48, JP49, JP50, JP51, JP52, JP53, JP69: (no value), jumper:JP2
- removed OK13, OK14: MOC3043S, optocoupler:DIL6-SMD
- removed R92, R93: 100UOHMS, SparkFun-Passives:0603-RES
- removed U$11, U$13: FDD8874, transistor-fet:TO252
- added JP1, JP2: (no value), jumper:JP1
- added LED6, LED7: (no value), led:SML1206
- added Q8, Q9: IRLML2060TRPBFBSS123LT1G, SparkFun-DiscreteSemi:SOT23-3
- added U9: ADUM3442CRWZ, digital-isolator:RW_16
- C46, C47, C48, C49, C50, C51, C52, C53, C54, C55: device rcl:C0603 -> rcl:C0402
- R46, R47: value (none) -> 500ohm
- R48: value (none) -> 2.2KOHM
- R49: value (none) -> 100UOHMS
- R5, R6, R79, R80: value 100UOHMS -> 500ohm
- R81: value 2.2KOHM -> 560ohms
- R91: value 100UOHMS -> 560ohms
- moved C16 520.2 mm to (-220.5, -200.4)
- moved C19 510.2 mm to (-214.0, -195.6)
- moved C18 506.4 mm to (-215.0, -200.4)
- moved R80 505.2 mm to (-220.5, -204.2), turned to 0 degrees
- moved C17 502.3 mm to (-220.5, -195.6)
- moved J4 499.1 mm to (-215.5, -188.1), turned to 0 degrees
- moved U$4 496.4 mm to (-208.3, -180.7)
- moved R91 495.4 mm to (-227.3, -223.6)
- moved R79 488.4 mm to (-203.5, -199.4)
- moved R81 484.1 mm to (-220.5, -211.1), turned to 0 degrees
- moved C11 481.6 mm to (-220.5, -169.5)
- moved C20 475.6 mm to (-207.6, -195.6)
- moved C12 466.0 mm to (-220.5, -164.7)
- moved X4 465.3 mm to (-215.8, -180.1), turned to 0 degrees
- moved R8 461.5 mm to (-210.3, -168.5)
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Connections:
- removed net G7: JP69.2, OK13.2, OK14.2
- removed net N$124: JP48.1, JP49.1, X11.2
- removed net N$125: JP50.1, JP51.1, X11.3
- removed net N$128 (its old number): JP50.2, R46.1
- removed net N$129 (its old number): OK13.1, R47.2
- removed net N$130 (its old number): JP48.2, R47.1
- removed net N$132 (its old number): JP51.2, OK14.6, R49.1
- removed net N$133 (its old number): JP53.2, R49.2
- removed net N$217 (its old number): C15.1, X3.1
- removed net N$218 (its old number): X3.2
- removed net N$220 (its old number): R80.1, U$3.32
- removed net N$234: R93.1, U$4.32
- removed net N$236: R92.1, U$4.31
- removed net V7: JP47.2, JP52.3, JP53.3, X11.1
- new net CON_MONB_+_J: D2.1, D2.2, JP2.2, R3.2
- new net CON_MONC_+_J: D3.1, D3.2, JP1.2, LED6.A, R7.2
- new net CON_MONC_SP: R47.2, R8.1, U$5.P$17
- new net MCU_BATMON_LINGND: U$1.23, U$2.23, U$3.23, U$4.23
- new net N$210: C15.1, U$3.29, X3.1
- new net N$213: R47.1, U$3.32
- new net N$215: R46.1, U$3.31
- new net N$224: C20.1, U$4.29, X4.1
- new net N$225: U$4.28, X4.2
- new net N$227: R80.1, U$4.32
- new net VDD1: U9.1
- new net VDD2: U9.16
- net CONGND: no longer JP69.1
- net CON_MONA_+: now also D1.1, D1.2, R1.2
- net CON_MONA_-: now also C1.2, C2.2, C3.2, C4.2, C5.2, R2.2, R9.2, U$1.11, U$1.13, U$1.16, U$1.18, U$1.20, U$1.27, U$1.30, U$1.33, U$1.4, U$1.41, U$1.44
- net CON_MONB_+: now also R10.2, R2.1; no longer D1.1, D1.2, D2.1, D2.2, R1.2, R3.2
- net CON_MONB_-: now also C10.2, C6.2, C7.2, C8.2, C9.2, R91.1, U$2.11, U$2.13, U$2.16, U$2.18, U$2.20, U$2.27, U$2.30, U$2.33, U$2.4, U$2.41, U$2.44; no longer R2.2, R9.2
- net CON_MONC_+: now also R4.1, R49.1, R6.2, R80.2; no longer D3.1, D3.2, R7.2
- net CON_MONC_-: now also C11.2, C12.2, C13.2, C14.2, C15.2, R46.2, R81.1, U$3.11, U$3.13, U$3.16, U$3.18, U$3.20, U$3.27, U$3.30, U$3.33, U$3.4, U$3.41, U$3.44; no longer R79.2
- net CON_MOND_+: now also R48.2; no longer R81.2
- net CON_MOND_-: now also C16.2, C17.2, C18.2, C19.2, C20.2, R49.2, R79.2, U$4.11, U$4.13, U$4.16, U$4.18, U$4.20, U$4.27, U$4.30, U$4.33, U$4.4, U$4.41, U$4.44; no longer R91.2, R92.2
- net FPGA_L50N_3_MODULEG_ISOLATOR: no longer JP48.3, JP49.3
- net FPGA_L50P_3_MODULEG_ISOLATOR: no longer JP50.3, JP51.3
- net GND: no longer C1.2, C10.2, C11.2, C12.2, C13.2, C14.2, C15.2, C16.2, C17.2, C18.2, C19.2, C2.2, C20.2, C3.2, C4.2, C5.2, C6.2, C7.2, C8.2, C9.2, JP69.3, R10.2, R2.1, R4.1, R6.2, R8.1, R80.2, R91.1, R93.2, U$1.11, U$1.13, U$1.16, U$1.18, U$1.20, U$1.27, U$1.30, U$1.4, U$1.41, U$1.44, U$2.11, U$2.13, U$2.16, U$2.18, U$2.20, U$2.27, U$2.30, U$2.4, U$2.41, U$2.44, U$3.11, U$3.13, U$3.16, U$3.18, U$3.20, U$3.27, U$3.30, U$3.4, U$3.41, U$3.44, U$4.11, U$4.13, U$4.16, U$4.18, U$4.20, U$4.27, U$4.30, U$4.4, U$4.41, U$4.44
- net GSENSE7: no longer OK13.4, OK14.4
- net MCU_+3.3V: now also Q8.2; no longer U$11.4
- net MCU_BATMON_LIN: now also U$1.22, U$2.22, U$3.22, U$4.22
- net N$126: now also U9.15; no longer JP49.2, OK13.6, R48.1
- net N$127: now also U9.2, U9.8; no longer OK14.1, R46.2
- net N$13: now also U$1.28
- net N$131: now also JP47.2, X11.1; no longer JP52.2, R48.2
- net N$182: now also Q8.3; no longer U$11.3
- net N$183: now also Q8.1; no longer U$11.1
- net N$189: now also Q9.3; no longer U$13.3
- net N$190: now also Q9.1; no longer U$13.1
- net N$192: now also Q9.2; no longer U$13.4
- net N$211: now also U$3.28, X3.2; no longer U$5.P$17
- net N$222: now also R48.1, U$4.34; no longer R79.1, U$3.31
- net N$229: now also R79.1, U$4.31; no longer R81.1, U$4.34
- net N$231: now also LED6.C, R81.2; no longer C20.1, X4.1
- net N$232: now also LED7.C, R91.2; no longer X4.2
- net N$40: now also U$2.29
- net N$41: now also U$2.28
- net N$8: now also U$1.29
- net PP_3.3V_FPGA: no longer JP52.1, JP53.1
Routing:
- net FPGA_L37N_0: track 0.00 -> 30.3 mm
- net FPGA_L37P_0: track 0.00 -> 28.5 mm
- net FPGA_L62P_0: track 0.00 -> 28.3 mm
- net FPGA_L62N_0: track 0.00 -> 25.6 mm
- net FPGA_L36N_0: track 0.00 -> 24.7 mm
- net FPGA_L63P_0: track 0.00 -> 24.5 mm
- net FPGA_L36P_0: track 0.00 -> 22.0 mm
- net FPGA_L63N_0: track 0.00 -> 21.5 mm
- net N$200: track 0.00 -> 19.7 mm
- net FPGA_L64P_0: track 0.00 -> 19.0 mm
- net FPGA_L35N_0: track 0.00 -> 17.4 mm
- net FPGA_L35P_0: track 0.00 -> 14.7 mm
- net FPGA_L64N_0: track 0.00 -> 14.6 mm
- net FPGA_L65P_0: track 0.00 -> 12.8 mm
- net FPGA_L34N_0: track 0.00 -> 11.4 mm
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Other:
- board size 201.9 x 117.8 mm -> 202.2 x 117.8 mm

Commit message: added  relay fets
Parts:
- added C80, C81, C82, C83, C84, C85: 0.1uf, eagle-ltspice:C0603
- added IC3: 74AHCT1G04DCK, 74xx-little-de:SC70-5
- added JP3, JP4, JP48: (no value), jumper:JP1
- added LED10, LED8, LED9: (no value), led:SML1206
- added Q10, Q11, Q12, Q13: IRLML2060TRPBFBSS123LT1G, SparkFun-DiscreteSemi:SOT23-3
- added R92, R93, R94: 560ohms, SparkFun-Passives:0603-RES
- moved U9 290.9 mm to (26.5, 52.5)
- moved JP72 21.8 mm to (42.0, 55.1)
- moved OK16 18.4 mm to (-12.3, 12.1)
Connections:
- removed net N$163: C48.1, C49.1, C50.1, C51.1, C52.1, U2.13, U2.21, U2.30, U2.85
- removed net N$195: C74.1, C75.1, C76.1, C77.1, C78.1, C79.1, R84.2, R85.2, U8.12, U8.18, U8.2, U8.44
- new net 5V_SUPERVISE: Q10.3, Q11.3, Q12.3, Q13.3
- new net CON_BAT1: U2401.13, U2401.23, U2401.3
- new net CON_MONA_+_J: D1.1, D1.2, JP3.2, R1.2
- new net CON_MOND_+_J: D4.1, D4.2, JP4.2, R48.2
- new net CON_RELAYA: Q10.2, Q11.2, Q12.2, Q13.2
- new net ETHERNET_3.3_J_+: C74.1, C75.1, C76.1, C77.1, C78.1, C79.1, JP48.2, LED10.A, R84.2, R85.2, U8.12, U8.18, U8.2, U8.44
- new net MCU_+1.2V: C53.1, C54.1, C55.1, U2.61, U2.88, U2.99
- new net MCU_RELAY_IO: Q10.1, Q11.1, Q12.1, Q13.1
- new net N$233: LED8.C, R92.2
- new net N$234: LED9.C, R93.2
- net CON_MONA_+: no longer D1.1, D1.2, R1.2
- net CON_MONA_-: now also R92.1
- net CON_MOND_+: no longer D4.1, D4.2, R48.2
- net CON_MOND_-: now also R93.1
- net GND: now also C80.2, C81.2, C82.2, C83.2, C84.2, C85.2, IC3.3, R94.1
- net MCU_+3.3V: now also C48.1, C49.1, C50.1, C51.1, C52.1, U2.13, U2.21, U2.30, U2.85; no longer C53.1, C54.1, C55.1, U2.61, U2.88, U2.99
- net N$206: now also LED10.C, R94.2; no longer U8.74
- net N$207: now also C80.1, C81.1, C82.1, C83.1, C84.1, C85.1, U8.11, U8.7, U8.74
- net STEERCTRL_+12V: no longer U2401.13, U2401.23, U2401.3
- net VCC: now also IC3.5

Commit message: updated board2a
Parts:
- removed IC3: 74AHCT1G04DCK, 74xx-little-de:SC70-5
- added C86, C87: 0.1 uF, rcl:C0402
- added JP111, JP112: (no value), jumper:JP2
- added JP49, JP50, JP51, JP52, JP53, JP69: (no value), jumper:JP1
- added LED11, LED12, LED13, LED14, LED15, LED16, LED17, LED18, LED19, LED20: (no value), led:SML1206
- added PTC: (no value), resistor:R1206W
- added Q14, Q15, Q16, Q17: IRLML2060TRPBFBSS123LT1G, SparkFun-DiscreteSemi:SOT23-3
- added R100, R101, R102, R103, R104, R97, R98, R99: .01, SparkFun-Passives:0603-RES
- added R105, R106, R107, R108, R109, R110, R111, R112, R113, R114: (no value), SparkFun-Passives:0603-RES
- added R95, R96: 1k, SparkFun-Passives:0603-RES
- added TP126, TP127, TP128, TP129: TPB2,54, testpad:B2,54
- added TP130, TP131: TPB1,27, testpad:B1,27
- added U10: SN65HVDA100-Q1_D_8, shit:D8
- moved TP18 119.0 mm to (27.4, 93.0)
- moved C42 35.3 mm to (49.9, 112.4), turned to 270 degrees
- moved C41 32.9 mm to (35.7, 87.4), turned to 270 degrees
- moved C38 31.8 mm to (52.6, 98.4), turned to 90 degrees
- moved TP11 30.8 mm to (52.3, 106.0)
- moved TP2 30.0 mm to (33.0, 90.8)
- moved TP63 28.8 mm to (69.8, 67.8)
- moved U$8 25.6 mm to (31.6, 112.5), turned to 180 degrees
- moved TP16 25.6 mm to (58.3, 90.7)
- moved TP3 25.4 mm to (53.0, 103.9)
- moved TP12 25.3 mm to (54.7, 114.2)
- moved LED5 23.9 mm to (64.6, 114.0), turned to 0 degrees
- moved RES604 23.8 mm to (28.2, 87.1), turned to 270 degrees
- moved C74 23.5 mm to (20.8, 68.3), turned to 0 degrees
- moved R68 22.7 mm to (88.1, 108.8), turned to 180 degrees
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Connections:
- net CON_RELAY_GND renamed CON_RELAY_HIGHSIDE
- removed net 5V_SUPERVISE: Q10.3, Q11.3, Q12.3, Q13.3
- removed net CON_RELAYA: Q10.2, Q11.2, Q12.2, Q13.2
- removed net MCU_BATMON_LIN-: TP40.TP, U2.94
- removed net MCU_RELAY_IO: Q10.1, Q11.1, Q12.1, Q13.1
- new net 12V_SUPERVISEDB: C63.2, Q14.3, R68.2, TP103.TP, U6.10
- new net 3.3V_SUPERVISEDB: C66.1, Q16.3, R76.2, U6.11
- new net 5V_SUPERVISEDB: C65.1, Q15.3, R69.2, U6.12
- new net FPGA_+3.3V: JP69.1, LED20.A, TP131.TP
- new net MCU_+3.3VT: JP53.2, Q8.2, R62.1, TP116.TP, U$10.9
- new net MCU_+3.3VT1: JP69.2
- new net MCU_ANALOG_GND: JP111.1
- new net MCU_IO_RALAYA: R109.2
- new net MCU_IO_RALAYB: R110.2
- new net MCU_IO_RALAYC: R111.2
- new net MCU_IO_RALAYD: R112.2
- new net MCU_LINTX: TP41.TP, U2.95
- new net MCU_LIN_EN: TP39.TP, U10.2, U2.92
- new net MCU_STEERING_POT: JP111.2, TP76.TP, U2.43
- new net MCU__LINRX: TP40.TP, U10.1, U2.94
- new net N$163: JP49.2, Q14.2
- new net N$195: LED20.C, R114.1
- new net N$235: JP51.2, Q15.2
- new net N$236: JP52.2, Q16.2
- new net N$237: TP126.TP, U10.3
- new net N$238: Q15.1, R101.2
- new net N$239: Q16.1, R100.2
- new net N$240: LED14.C
- new net N$241: LED13.A, R99.1
- new net N$242: LED15.C, R106.1
- new net N$243: Q14.1, R102.2
- new net N$244: Q17.3
- new net N$245: LED12.A, R98.1
- new net N$246: LED11.A, R97.1
- new net N$247: LED14.A, R103.2
- new net N$248: Q17.1, R104.1
- new net N$249: LED16.C, R105.1
- new net N$250: R105.2
- new net N$251: LED17.C, R108.1
- new net N$252: Q13.1, R109.1
- new net N$253: LED18.C, R107.1
- new net N$254: R107.2
- new net N$255: Q11.1, R111.1
- new net N$256: Q12.1, R112.1
- new net N$257: Q10.1, R110.1
- new net N$258: LED19.C, R113.1
- new net N$259: R113.2
- new net N$260: R114.2
- new net N$262: PTC.1, U7.2
- new net N$266: JP111.3, JP112.2
- net 12V_SUPERVISED: now also JP49.1, R97.2; no longer C63.2, R68.2, TP103.TP, U6.10
- net 12V_UNSUPERVISED: now also LED15.A
- net 3.3V_SUPERVISED: now also JP112.3, JP52.1, R99.2; no longer C66.1, R76.2, U6.11
- net 3.3V_UNSUPERVISED: now also LED18.A
- net 5V_SUPERVISED: now also JP112.1, JP51.1, R98.2; no longer C65.1, R69.2, U6.12
- net 5V_TO_SUPERVISOR: now also LED16.A, R103.1
- net CON_RELAY_BAT1: now also Q13.3
- net CON_RELAY_BAT2: now also Q10.3
- net CON_RELAY_BAT3: now also Q11.3
- net CON_RELAY_BAT4: now also Q12.3
- net GND: now also LED11.C, LED12.C, LED13.C, Q10.2, Q11.2, Q12.2, Q13.2, R106.2, R108.2; no longer IC3.3
- net MCU_+3.3V: now also JP53.1, LED19.A, TP130.TP; no longer Q8.2, R62.1, TP116.TP, U$10.9
- net MCU_BATMON_LIN: now also C87.1, R95.1, TP129.TP; no longer TP41.TP, U2.95
- net MCU_BATMON_LINGND: now also C86.2, C87.2, U10.5
- net MCU_PROG_RTCK: now also R96.1
- net MCU_SPIBRIDGE_MISO: no longer TP32.TP, U2.67
- net MCU_SPIBRIDGE_SCK: now also TP32.TP, U2.67
- net N$174: now also PTC.2; no longer U7.2
- net N$63: no longer TP76.TP, U2.43
- net N$9: now also C86.1, R95.2, TP127.TP, TP128.TP, U10.7, U10.8; no longer TP39.TP, U2.92
- net ON_OFF_CONTROL_INPUT: now also R104.2
- net POWER_GOOD_OUT: now also R100.1, R101.1, R102.1
- net VCC: no longer IC3.5
Routing:
- net N$145: track 0.00 -> 56.9 mm
- net GND: track 0.00 -> 45.0 mm
- net N$144: track 0.00 -> 27.4 mm
- net SPIBRIDGE_ISOLATION_VBUS: track 0.00 -> 25.0 mm
- net N$146: track 0.00 -> 24.3 mm
- net N$161: track 0.00 -> 23.5 mm
- net N$160: track 0.00 -> 23.3 mm
- net N$159: track 0.00 -> 21.1 mm
- net N$149: track 0.00 -> 16.0 mm
- net N$148: track 0.00 -> 15.4 mm
- net SPIBRIDGE_ISOLATION_D+: track 0.00 -> 14.4 mm, vias 0 -> 2
- net SPIBRIDGE_ISOLATION_D-: track 0.00 -> 13.3 mm
- net N$202: track 0.00 -> 9.38 mm
- net N$151: track 0.00 -> 8.62 mm
- net N$162: track 0.00 -> 8.60 mm
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- added copper zone on layer 16, net GND

Commit message: ls
Parts:
- removed JP13, JP14, JP15, JP16, JP17, JP18, JP19, JP20, JP21, JP22, JP23, JP24, JP25, JP26, JP27, JP28, JP29, JP30, JP31, JP32, JP33, JP34, JP35, JP36, JP37, JP38, JP39, JP40, JP41, JP42, JP43, JP44, JP45, JP46, JP47, JP54, JP55, JP56, JP57, JP58, JP59, JP60, JP61, JP62, JP63, JP64, JP65, JP66, JP67, JP68, JP70, JP71, JP72, JP73, JP74, JP76: (no value), jumper:JP2
- removed JP77, JP78: (no value), pinhead:1X08
- removed OK1, OK10, OK11, OK12, OK15, OK16, OK2, OK3, OK4, OK5, OK6, OK7, OK8, OK9: MOC3043S, optocoupler:DIL6-SMD
- removed R22, R23, R24, R25, R26, R27, R28, R29, R30, R31, R32, R34, R35, R36, R37, R38, R39, R40, R41, R42, R43, R44, R45, R50, R51, R52, R53: (no value), SparkFun-Passives:0603-RES
- added C100, C101, C102, C103, C104, C105, C90, C91, C92, C93, C94, C95, C96, C97, C98, C99: .1uF, SparkFun-Capacitors:0603-CAP
- added C88: 10uF, SparkFun-Capacitors:0603-CAP
- added C89: 1uF, SparkFun-Capacitors:0603-CAP
- added U$11: 1.2VREG, shit:SOT-223
- added U$13, U$19, U$20, U$23, U$24, U$25, U$26, U$27, U$28, U$29, U$30, U$31: DPDTSWITCH, shit:JS202011
- added U11, U12, U13, U14, U15, U16, U17: ADUM3442CRWZ, digital-isolator:RW_16
- JP75: device jumper:JP2 -> pinhead:1X08
- R33: value (none) -> 10k
- U$14, U$16, U$17, U$18: value 4PDT_SWITCH -> DPDTSWITCH; device shit:MMS42 -> shit:JS202011
- moved R80 567.4 mm to (242.1, 124.5), turned to 90 degrees
- moved C16 562.1 mm to (238.3, 124.5), turned to 90 degrees
- moved C18 560.9 mm to (238.3, 129.9), turned to 90 degrees
- moved R49 558.4 mm to (237.2, 134.6), turned to 90 degrees
- moved R48 557.7 mm to (237.2, 138.3), turned to 90 degrees
- moved R79 557.1 mm to (237.2, 141.5), turned to 90 degrees
- moved C17 555.4 mm to (233.4, 124.5), turned to 90 degrees
- moved C19 553.9 mm to (233.4, 130.9), turned to 90 degrees
- moved C20 552.6 mm to (233.4, 137.3), turned to 90 degrees
- moved J4 543.8 mm to (225.9, 129.4), turned to 90 degrees
- moved D4 542.8 mm to (226.6, 138.3), turned to 90 degrees
- moved X4 532.7 mm to (217.9, 129.2), turned to 90 degrees
- moved U$4 531.9 mm to (218.6, 136.7), turned to 90 degrees
- moved R47 524.4 mm to (211.2, 124.5), turned to 90 degrees
- moved C11 519.1 mm to (207.4, 124.5), turned to 90 degrees
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Connections:
- removed net 3.3V: Q7.1
- removed net FPGA_L34N_0: JP77.2, U$6.P133
- removed net FPGA_L34P_0: JP77.1, U$6.P134
- removed net FPGA_L35N_0: JP77.4, U$6.P131
- removed net FPGA_L35P_0: JP77.3, U$6.P132
- removed net FPGA_L36N_0: JP77.6, U$6.P126
- removed net FPGA_L36P_0: JP77.5, U$6.P127
- removed net FPGA_L37N_0: JP77.8, U$6.P123
- removed net FPGA_L37P_0: JP77.7, U$6.P124
- removed net G1: JP57.2, OK1.2, OK2.2
- removed net G2: JP58.2, OK3.2, OK4.2
- removed net G3: JP61.2, OK5.2, OK6.2
- removed net G4: JP63.2, OK7.2, OK8.2
- removed net G5: JP65.2, OK10.2, OK9.2
- removed net G6: JP67.2, OK11.2, OK12.2
- removed net G8: JP75.2, OK15.2, OK16.2
- removed net GSENSE1: JP57.1, JP59.1, OK2.4, OK3.4, X5.4
- removed net GSENSE2: JP60.2, OK4.4, X6.4
- removed net GSENSE3: JP62.2, OK5.4, OK6.4, X7.4
- removed net GSENSE4: JP64.2, OK7.4, OK8.4, X8.4
- removed net GSENSE5: JP66.2, OK10.4, OK9.4, X9.4
- removed net GSENSE6: JP68.2, OK11.4, OK12.4, X10.4
- removed net GSENSE7: JP70.2, X11.4
- removed net GSENSE8: JP76.2, OK15.4, OK16.4, X12.4
- removed net N$114: JP41.1, JP42.1, X10.2
- removed net N$115: JP43.1, JP44.1, X10.3
- removed net N$116: JP42.2, OK11.6, R44.1
- removed net N$117: OK12.1, R42.2
- removed net N$118: JP43.2, R42.1
- removed net N$119: OK11.1, R43.2
- removed net N$120: JP41.2, R43.1
- removed net N$121: JP45.2, R44.2
- removed net N$122: JP44.2, OK12.6, R45.1
- removed net N$123: JP46.2, R45.2
- removed net N$126: U9.15
- removed net N$127: U9.2, U9.8
- removed net N$131: JP47.2, X11.1
- removed net N$134: JP55.1, JP56.1, X12.2
- removed net N$135: JP71.1, JP72.1, X12.3
- removed net N$136: JP56.2, OK15.6, R52.1
- removed net N$137: OK16.1, R50.2
- removed net N$138: JP71.2, R50.1
- removed net N$139: OK15.1, R51.2
- removed net N$140: JP55.2, R51.1
- removed net N$141: JP73.2, R52.2
- removed net N$142: JP72.2, OK16.6, R53.1
- removed net N$143: JP74.2, R53.2
- removed net VDD1: U9.1
- removed net VDD2: U9.16
- new net FPGA_MCU_RES1: TP61.TP, U$6.P140, U2.83
- new net FPGA_MCU_RES4: TP64.TP, U$6.P44, U2.97
- new net V7: C102.1, JP11.2, U16.10, U16.16, X11.1
- new net VIAA: U$14.4, U9.3
- new net VIAB: U$17.4, U11.3
- new net VIAC: U$19.4, U12.3
- new net VIAD: U$23.4, U13.3
- new net VIAE: U$25.4, U14.3
- new net VIAF: U$27.4, U15.3
- new net VIAG: U$29.4, U16.3
- new net VIAH: U$31.4, U17.3
- new net VIBA: U$13.4, U9.4
- new net VIBB: U$16.4, U11.4
- new net VIBC: U$18.4, U12.4
- new net VIBD: U$20.4, U13.4
- new net VIBE: U$24.4, U14.4
- new net VIBF: U$26.4, U15.4
- new net VIBG: U$28.4, U16.4
- new net VIBH: U$30.4, U17.4
- new net VOBA: U$13.1, U9.13
- new net VOBB: U$16.1, U11.13
- new net VOBC: U$18.1, U12.13
- new net VOBD: U$20.1, U13.13
- new net VOBE: U$24.1, U14.13
- new net VOBF: U$26.1, U15.13
- new net VOBG: U$28.1, U16.13
- new net VOBH: U$30.1, U17.13
- new net VOCA: U$14.6, U9.5
- new net VOCB: U$17.6, U11.5
- new net VOCC: U$19.6, U12.5
- new net VOCD: U$23.6, U13.5
- new net VOCE: U$25.6, U14.5
- new net VOCF: U$27.6, U15.5
- new net VOCG: U$29.6, U16.5
- new net VOCH: U$31.6, U17.5
- new net VODA: U$13.6, U9.6
- new net VODB: U$16.6, U11.6
- new net VODC: U$18.6, U12.6
- new net VODD: U$20.6, U13.6
- new net VODE: U$24.6, U14.6
- new net VODF: U$26.6, U15.6
- new net VODG: U$28.6, U16.6
- new net VODH: U$30.6, U17.6
- net 3.3V_SUPERVISED: now also C101.1, C103.1, C105.1, C91.1, C93.1, C95.1, C97.1, C99.1, U11.1, U11.7, U12.1, U12.7, U13.1, U13.7, U14.1, U14.7, U15.1, U15.7, U16.1, U16.7, U17.1, U17.7, U9.1, U9.7
- net CONGND: now also C100.2, C102.2, C104.2, C90.2, C92.2, C94.2, C96.2, C98.2, U11.15, U11.9, U12.15, U12.9, U13.15, U13.9, U14.15, U14.9, U15.15, U15.9, U16.15, U16.9, U17.15, U17.9, U9.15, U9.9, X10.4, X11.4, X12.4, X5.4, X6.4, X7.4, X8.4, X9.4; no longer JP58.1, JP59.2, JP60.1, JP61.1, JP62.1, JP63.1, JP64.1, JP65.1, JP66.1, JP67.1, JP68.1, JP70.1, JP75.1, JP76.1, OK1.4
- net FPGA_L30N_2: now also U$6.P55
- net FPGA_L31N_2: now also U$6.P50
- net FPGA_L31P_2: now also U$6.P51
- net FPGA_L33N_1_MODULED_ISOLATOR: now also U$20.5; no longer JP27.3, JP28.3
- net FPGA_L33P_1_MODULED_ISOLATOR: now also U$23.5; no longer JP29.3, JP30.3
- net FPGA_L34N_1_MODULEC_ISOLATOR: now also U$18.5; no longer JP20.3, JP21.3
- net FPGA_L34P_1_MODULEC_ISOLATOR: now also U$19.5; no longer JP22.3, JP23.3
- net FPGA_L40N_1_MODULEB_ISOLATOR: now also U$16.5; no longer JP13.3, JP14.3
- net FPGA_L40P_1_MODULEB_ISOLATOR: now also U$17.5; no longer JP15.3, JP16.3
- net FPGA_L41N_1_MODULEA_ISOLATOR: now also U$13.5; no longer JP6.3, JP7.3
- net FPGA_L41P_1_MODULEA_ISOLATOR: now also U$14.5; no longer JP8.3, JP9.3
- net FPGA_L48N_2: now also U$6.P47
- net FPGA_L48P_2: now also U$6.P48
- net FPGA_L49N_2: now also U$6.P45
- net FPGA_L49N_3_MODULEH_ISOLATOR: now also U$30.5; no longer JP55.3, JP56.3
- net FPGA_L49P_2: now also U$6.P46
- net FPGA_L49P_3_MODULEH_ISOLATOR: now also U$31.5; no longer JP71.3, JP72.3
- net FPGA_L50N_3_MODULEG_ISOLATOR: now also U$28.5
- net FPGA_L50P_3_MODULEG_ISOLATOR: now also U$29.5
- net FPGA_L51N_3_MODULEF_ISOLATOR: now also U$26.5; no longer JP41.3, JP42.3
- net FPGA_L51P_3_MODULEF_ISOLATOR: now also U$27.5; no longer JP43.3, JP44.3, U$18.P$4, U$18.P$9
- net FPGA_L52N_3_MODULEE_ISOLATOR: now also U$24.5; no longer JP34.3, JP35.3
- net FPGA_L52P_3_MODULEE_ISOLATOR: now also U$25.5; no longer JP36.3, JP37.3
- net FPGA_L62N_0: now also JP75.2; no longer JP78.2
- net FPGA_L62P_0: now also JP75.1; no longer JP78.1, U$6.P121
- net FPGA_L63N_0: now also JP75.4; no longer JP78.4
- net FPGA_L63P_0: now also JP75.3; no longer JP78.3
- net FPGA_L64N_0: now also JP75.6; no longer JP78.6
- net FPGA_L64P_0: now also JP75.5; no longer JP78.5
- net FPGA_L65N_0: now also JP75.8; no longer JP78.8
- net FPGA_L65P_0: now also JP75.7; no longer JP78.7
- net FPGA_MCU_AD1: now also U$6.P123; no longer U$6.P138
- net FPGA_MCU_AD2: now also U$6.P124; no longer U$6.P139
- net FPGA_MCU_AD3: now also U$6.P126; no longer U$6.P140
- net FPGA_MCU_AD4: now also U$6.P127; no longer U$6.P41
- net FPGA_MCU_AD5: now also U$6.P131; no longer U$6.P43
- net FPGA_MCU_AD6: now also U$6.P132; no longer U$6.P44
- net FPGA_MCU_AD7: now also U$6.P133; no longer U$6.P45
- net FPGA_MCU_ADO: now also U$6.P121; no longer U$6.P137
- net FPGA_MCU_CLK: now also U$6.P137; no longer U$6.P47
- net FPGA_MCU_RES: now also U$6.P139; no longer U$6.P50
- net FPGA_MCU_RES2: now also TP62.TP, U$6.P41, U2.89; no longer U$6.P51
- net FPGA_MCU_RES3: now also TP63.TP, U$6.P43, U2.90; no longer U$6.P55
- net FPGA_MCU_RW: now also U$6.P134; no longer U$6.P46
- net FPGA_MCU_STAT: now also U$6.P138; no longer U$6.P48
- net FPGA_SUSPEND: now also R33.1
- net GND: now also C101.2, C103.2, C105.2, C88.2, C89.2, C91.2, C93.2, C95.2, C97.2, C99.2, R33.2, U$11.1, U11.2, U11.8, U12.2, U12.8, U13.2, U13.8, U14.2, U14.8, U15.2, U15.8, U16.2, U16.8, U17.2, U17.8, U9.2, U9.8; no longer JP57.3, JP58.3, JP59.3, JP60.3, JP61.3, JP62.3, JP63.3, JP64.3, JP65.3, JP66.3, JP67.3, JP68.3, JP70.3, JP75.3, JP76.3
- net N$100: now also U$26.2, X10.3; no longer JP27.2, R35.1
- net N$101: now also U$27.1, U15.14; no longer JP31.2, R36.2
- net N$102: now also U$27.3, U15.12; no longer JP30.2, OK8.6, R37.1
- net N$103: now also U$26.3, U15.11; no longer JP32.2, R37.2
- net N$104: now also U$29.2, X11.2; no longer JP34.1, JP35.1, X9.2
- net N$105: now also U$28.2, X11.3; no longer JP36.1, JP37.1, X9.3
- net N$106: now also U$29.1, U16.14; no longer JP35.2, OK9.6, R40.1
- net N$107: now also U$29.3, U16.12; no longer OK10.1, R38.2
- net N$108: now also U$28.3, U16.11; no longer JP36.2, R38.1
- net N$109: now also U$31.2, X12.2; no longer OK9.1, R39.2
- net N$110: now also U$30.2, X12.3; no longer JP34.2, R39.1
- net N$111: now also U$31.1, U17.14; no longer JP38.2, R40.2
- net N$112: now also U$31.3, U17.12; no longer JP37.2, OK10.6, R41.1
- net N$113: now also U$30.3, U17.11; no longer JP39.2, R41.2
- net N$48: no longer TP61.TP, U2.83
- net N$49: no longer TP62.TP, U2.89
- net N$50: no longer TP63.TP, U2.90
- net N$51: no longer TP64.TP, U2.97
- net N$64: now also U$14.2; no longer JP6.1, JP7.1
- net N$65: now also U$13.2; no longer JP8.1, JP9.1
- net N$66: now also U$14.1, U9.14; no longer JP7.2, OK1.6, R24.1
- net N$67: now also U$14.3, U9.12; no longer OK2.1, R22.2
- net N$68: now also U$13.3, U9.11; no longer JP8.2, R22.1
- net N$69: now also U$17.2, X6.2; no longer OK1.1, R23.2
- net N$70: now also U$16.2, X6.3; no longer JP6.2, R23.1
- net N$71: now also U$17.1, U11.14; no longer JP10.2, R24.2
- net N$72: no longer JP9.2, OK2.6, R25.1
- net N$73: no longer JP11.2, R25.2
- net N$74: no longer JP13.1, JP14.1, X6.2
- net N$75: no longer JP15.1, JP16.1, X6.3
- net N$76: no longer JP14.2, OK3.6, R28.1
- net N$77: no longer OK4.1, R26.2
- net N$78: no longer JP15.2, R26.1
- net N$79: no longer OK3.1, R27.2
- net N$80: no longer JP13.2, R27.1
- net N$81: no longer JP17.2, R28.2
- net N$82: now also U$17.3, U11.12; no longer JP16.2, OK4.6, R29.1
- net N$83: now also U$16.3, U11.11; no longer JP18.2, R29.2
- net N$84: now also U$19.2; no longer JP20.1, JP21.1
- net N$85: now also U$18.2; no longer JP22.1, JP23.1
- net N$86: now also U$19.1, U12.14; no longer JP21.2, OK5.6, R32.1
- net N$87: now also U$19.3, U12.12; no longer OK6.1, R30.2
- net N$88: now also U$18.3, U12.11; no longer JP22.2, R30.1
- net N$89: now also U$23.2, X8.2; no longer OK5.1, R31.2
- net N$90: now also U$20.2, X8.3; no longer JP20.2, R31.1
- net N$91: now also U$23.1, U13.14; no longer JP24.2, R32.2
- net N$92: now also U$23.3, U13.12; no longer JP23.2, OK6.6, R33.1
- net N$93: now also U$20.3, U13.11; no longer JP25.2, R33.2
- net N$94: now also U$25.2, X9.2; no longer JP27.1, JP28.1, X8.2
- net N$95: now also U$24.2, X9.3; no longer JP29.1, JP30.1, X8.3
- net N$96: now also U$25.1, U14.14; no longer JP28.2, OK7.6, R36.1
- net N$97: now also U$25.3, U14.12; no longer OK8.1, R34.2
- net N$98: now also U$24.3, U14.11; no longer JP29.2, R34.1
- net N$99: now also U$27.2, X10.2; no longer OK7.1, R35.2
- net PP_3.3V_FPGA: now also C89.1, Q7.1, U$11.3; no longer JP10.1, JP11.1, JP17.1, JP18.1, JP24.1, JP25.1, JP31.1, JP32.1, JP38.1, JP39.1, JP45.1, JP46.1, JP73.1, JP74.1
- net PP_3.3V_MODULARCONNECTOR: now also JP10.3, JP11.3, JP6.3, JP7.3, JP8.3, JP9.3; no longer JP19.3, JP26.3, JP33.3, JP40.3, JP47.3, JP54.3
- net PP_5V_MODULARCONNECTOR: now also JP10.1, JP11.1, JP6.1, JP7.1, JP8.1, JP9.1; no longer JP19.1, JP26.1, JP33.1, JP40.1, JP47.1, JP54.1
- net V1: now also C90.1, U9.10, U9.16; no longer JP10.3, JP11.3
- net V2: now also C92.1, JP6.2, U11.10, U11.16; no longer JP12.2, JP17.3, JP18.3
- net V3: now also C94.1, JP7.2, U12.10, U12.16; no longer JP19.2, JP24.3, JP25.3
- net V4: now also C96.1, JP8.2, U13.10, U13.16; no longer JP26.2, JP31.3, JP32.3
- net V5: now also C98.1, JP9.2, U14.10, U14.16; no longer JP33.2, JP38.3, JP39.3
- net V6: now also C100.1, JP10.2, U15.10, U15.16; no longer JP40.2, JP45.3, JP46.3
- net V8: now also C104.1, JP12.2, U17.10, U17.16; no longer JP54.2, JP73.3, JP74.3
- net VCCINT: now also C88.1, U$11.2, U$11.4
Routing:
- net FPGA_L37N_0: track 30.3 -> 0.00 mm
- net FPGA_L37P_0: track 28.5 -> 0.00 mm
- net FPGA_L62P_0: track 28.3 -> 0.00 mm
- net FPGA_L62N_0: track 25.6 -> 0.00 mm
- net FPGA_L36N_0: track 24.7 -> 0.00 mm
- net FPGA_L63P_0: track 24.5 -> 0.00 mm
- net FPGA_L36P_0: track 22.0 -> 0.00 mm
- net FPGA_L63N_0: track 21.5 -> 0.00 mm
- net FPGA_L64P_0: track 19.0 -> 0.00 mm
- net FPGA_L35N_0: track 17.4 -> 0.00 mm
- net FPGA_L35P_0: track 14.7 -> 0.00 mm
- net FPGA_L64N_0: track 14.6 -> 0.00 mm
- net FPGA_L65P_0: track 12.8 -> 0.00 mm
- net FPGA_L34N_0: track 11.4 -> 0.00 mm
- net FPGA_L65N_0: track 9.10 -> 0.00 mm
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- added copper zone on layer 1, net GND
Other:
- board size 202.2 x 117.8 mm -> 202.7 x 118.5 mm
