File: Electrical Schematics/Version2/Schematics/boardv2a.brd (EAGLE design)
At the start: 202.7 x 118.5 mm, 514 parts, among them IC1 MCP41HVX1ST, IC2 ADUM4160BRW, K5 G5V-2, Q1 IRLML2060TRPBFBSS123LT1G, Q10 IRLML2060TRPBFBSS123LT1G, Q11 IRLML2060TRPBFBSS123LT1G, Q12 IRLML2060TRPBFBSS123LT1G, Q13 IRLML2060TRPBFBSS123LT1G, Q14 IRLML2060TRPBFBSS123LT1G, Q15 IRLML2060TRPBFBSS123LT1G, Q16 IRLML2060TRPBFBSS123LT1G, Q17 IRLML2060TRPBFBSS123LT1G, Q2 IRLML2060TRPBFBSS123LT1G, Q3 IRLML2060TRPBFBSS123LT1G, Q4 IRLML2060TRPBFBSS123LT1G, Q5 IRLML2060TRPBFBSS123LT1G, Q6 IRLML2060TRPBFBSS123LT1G, Q7 ASFL1, Q8 IRLML2060TRPBFBSS123LT1G, Q9 IRLML2060TRPBFBSS123LT1G, U1 CP2130-GM, U10 SN65HVDA100-Q1_D_8, U11 ADUM3442CRWZ, U12 ADUM3442CRWZ, U13 ADUM3442CRWZ, U14 ADUM3442CRWZ, U15 ADUM3442CRWZ, U16 ADUM3442CRWZ, U17 ADUM3442CRWZ, U2 TMS570LS0432_PZ_100, U2401 VNH2SP30-E, U3 LM1085_KTT_3, U4 LM1085_KTT_3, U5 LM1084_KTT_3, U6 TPS3514_D_14, U7 LM1085_KTT_3, U9 ADUM3442CRWZ

Commit message: updated schematatics
Parts:
- removed AMTOG+, AMTOG-, GEARSHIFT_GND, POT_HIGH, POT_WIPER, THROTTLE1, THROTTLE2: (no value), adafruit:1X01
- removed C16: 47nF, eagle-ltspice:C0603
- removed C17: 220nF, eagle-ltspice:C0603
- removed C18: 1uF, eagle-ltspice:C0603
- removed C19: 4.7UF, eagle-ltspice:C0603
- removed C20: 220pf, eagle-ltspice:C0603
- removed D4: BBY51, diode:SOT23
- removed D5: 1N4004, adafruit:DO41-10
- removed GS_C, GS_N: N, adafruit:1X01
- removed GS_F: F, adafruit:1X01
- removed GS_R: R, adafruit:1X01
- removed J2401: (no value), Atlanta-Robotics LAPTOP:PHOENIX_1792863
- removed J2402, J2403: (no value), jumper:JP1
- removed J4: (no value), con-lsta:JU05
- removed JP112: (no value), jumper:JP2
- removed K5: G5V-2, relay:G5V-2
- removed LED1: BLUE, adafruit:1206
- removed LED2401, LED2402, LED9: (no value), led:SML1206
- removed POT_GND: POT_GND, adafruit:1X01
- removed Q12: IRLML2060TRPBFBSS123LT1G, SparkFun-DiscreteSemi:SOT23-3
- removed R112, R54, R55, R56, R57, R58: (no value), SparkFun-Passives:0603-RES
- removed R12: 150, rcl:R0603
- removed R2406: 10k, rcl:R0603
- removed R2407, R2408: 3.3k, rcl:R0603
- removed R2409: 1.5k, rcl:R0603
- removed R2410: 1k, rcl:R0603
- removed R46, R47, R79, R80: 500ohm, SparkFun-Passives:0603-RES
- removed R48: 2.2KOHM, SparkFun-Passives:0603-RES
- removed R49: 100UOHMS, SparkFun-Passives:0603-RES
- removed R81, R91, R93: 560ohms, SparkFun-Passives:0603-RES
- removed U$4: (no value), freescalemod:QFN48
- removed U2401: VNH2SP30-E, st-microelectronics:MULTIPOWERSO-30
- added C106: 3.3uf, eagle-ltspice:C0603
- added C107, C108: 10uf, eagle-ltspice:C0603
- added C109, C110, C111: 0.1uf, eagle-ltspice:C0603
- added C112: 1uF, eagle-ltspice:C0603
- added C113: 0.1uF, eagle-ltspice:C0603
- added C114, C115: .1uF, rcl:C0402
- added C116, C117: 10u, eagle-ltspice:C0603
- added C118, C119: 10nF, SparkFun-Capacitors:0603-CAP
- added IC3: SE555D, linear:SO08
- added IC4, IC7: 4030D, 40xx:SO14
- added IC5, IC6: 74LVC1G04DBV, 74xx-little-us:SOT23-5
- added JP13, JP14, JP15, JP16, JP17, JP18, JP19, JP20, JP21, JP23, JP25, JP27: (no value), jumper:JP1
- added JP22, JP24, JP26: (no value), jumper:JP2
- added K1: G5V-2, relay:G5V-2
- added L3, L4, L5, L6, L7: BLM15HB121SN1, inductors:0402
- added LED23, LED24, LED25: (no value), eagle-ltspice:LED_1206
- added LED26: (no value), led:SML1206
- added PTC1: (no value), resistor:R1206W
- added Q18: BSP170P, transistor-fet:SOT223
- added Q19: IRLML2060TRPBFBSS123LT1G, SparkFun-DiscreteSemi:SOT23-3
- added R22, R23: (no value), resistor-bourns:4816P
- added R24, R25, R26, R27, R28: 1k, SparkFun-Passives:0603-RES
- added R31, R32, R34: 600, SparkFun-Passives:0603-RES
- added R35: (no value), SparkFun-Passives:0603-RES
- added R36, R39: 560ohms, SparkFun-Passives:0603-RES
- added R37, R38: 500ohm, SparkFun-Passives:0603-RES
- added R40: 10K, rcl:R0603
- added SV1, SV2: (no value), con-lsta:FE05-1
- added TP132, TP133, TP134, TP135, TP136, TP137, TP138, TP139, TP140: TPB2,54, testpad:B2,54
- added TP141, TP142, TP143, TP144, TP145, TP146, TP147, TP148, TP149, TP150, TP151, TP152, TP153, TP154, TP155, TP156, TP157, TP158, TP159, TP160, TP161, TP162, TP163, TP164: TPB1,27, testpad:B1,27
- added U18: LM1085_KTT_3, shit:KTT3
- added U19, U20: ADUM3442CRWZ, digital-isolator:RW_16
- C69: value 33nF -> .1uF; device rcl:C0603 -> SparkFun-Capacitors:0603-CAP
- C70, C71: value 0.1 -> 0.1uF
- D1, D2, D3: value BBY51 -> GF1; device diode:SOT23 -> diode:SMA-DO214AC
- LED2: value RED -> GREEN
- LED4: device adafruit:1206 -> adafruit:CHIPLED_1206
- Q4: value IRLML2060TRPBFBSS123LT1G -> BSP170P; device SparkFun-DiscreteSemi:SOT23-3 -> transistor-fet:SOT223
- R13, R17: value 150 -> 10K
- R14: value 10K -> 1K; device rcl:R0603 -> rcl:MINI_MELF-0102W
- R15, R16: value 150 -> 1K
- R18, R20: value 1K -> 10K
- R19: value 1k -> 10K
- R96: value 1k -> 10k
- X4: value (none) -> 5566-4; device con-molex:KK-156-2 -> con-molex:5566-4
- moved JP111 668.4 mm to (91.4, 52.8), flipped to the bottom, turned to 90 degrees
- moved R111 663.9 mm to (165.1, 57.7), turned to 180 degrees
- moved R110 657.9 mm to (164.8, 52.1), turned to 180 degrees
- moved R109 657.6 mm to (164.8, 54.1), turned to 180 degrees
- moved PTC 654.6 mm to (151.9, 18.0), turned to 90 degrees
- moved JP53 636.0 mm to (102.6, 69.1), turned to 270 degrees
- moved R107 629.8 mm to (139.2, 44.7)
- moved R106 627.4 mm to (143.0, 40.4), turned to 90 degrees
- moved R114 622.4 mm to (94.0, 31.2), turned to 270 degrees
- moved R103 622.4 mm to (145.8, 54.6), turned to 270 degrees
- moved LED20 621.0 mm to (98.6, 29.2)
- moved TP130 618.2 mm to (128.3, 17.0)
- moved TP131 618.0 mm to (100.6, 26.7), turned to 270 degrees
- moved JP69 618.0 mm to (100.6, 34.3)
- moved LED18 616.4 mm to (138.2, 35.8), turned to 180 degrees
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Connections:
- removed net +12V: J2402.1
- removed net +5V: AMTOG+.1, D5.C, IC1.1, J2403.1, K5.1, LED4.A
- removed net AM_TOGGLE-: AMTOG-.1, LED1.A, LED2.A, LED3.A, R13.1, R14.1, R15.1, R17.1
- removed net AUTO_SENSE: R14.2
- removed net CON_BAT1: U2401.13, U2401.23, U2401.3
- removed net CON_MOND_+_J: D4.1, D4.2, JP4.2, R48.2
- removed net CON_RELAY_BAT4: Q12.3, U$5.P$20
- removed net FGND: GS_F.1, Q3.2, R19.1
- removed net FNR_CON_GND: GEARSHIFT_GND.1, IC1.10, IC1.13, IC1.9, POT_GND.1
- removed net FNR_CON_THROTTLE1: K5.13, THROTTLE1.1
- removed net FNR_CON_THROTTLE2: K5.4, THROTTLE2.1
- removed net GEARSHIFT_F: R16.1
- removed net GEARSHIFT_R: R11.1
- removed net MCU_!CS: IC1.3
- removed net MCU_+3.3VT1: JP69.2
- removed net MCU_ANALOG_GND: JP111.1
- removed net MCU_IO_RALAYD: R112.2
- removed net MCU_STEERCTRL_CS: C69.1, R2406.1
- removed net MCU_STEERCTRL_CS_R: R2406.2, R2409.2, U2401.9
- removed net MCU_STEERCTRL_DIAGA_R: R2403.2, R2407.1, U2401.6
- removed net MCU_STEERCTRL_DIAGB_R: R2404.2, R2408.1, U2401.10
- removed net MCU_STEERCTRL_INA_R: R2401.2, U2401.5
- removed net MCU_STEERCTRL_INB_R: R2402.2, U2401.11
- removed net MCU_STEERCTRL_PWM_R: R2405.2, U2401.8
- removed net N: GS_N.1, Q2.3, Q4.3, Q5.3, R20.2
- removed net N$133: U$3.9
- removed net N$153: U1.22
- removed net N$19: TP29.TP, U2.27
- removed net N$194: C74.2, C75.2, C77.2, C78.2, C79.2
- removed net N$20: TP28.TP, U2.39
- removed net N$21: TP27.TP, U2.69
- removed net N$213: R47.1, U$3.32
- removed net N$215: R46.1, U$3.31
- removed net N$217: C19.1, D4.3, U$4.21
- removed net N$218: J4.5, U$4.10
- removed net N$219: U$4.9
- removed net N$220: U$4.8
- removed net N$221: J4.2, U$4.7
- removed net N$222: R48.1, U$4.34
- removed net N$223: C17.1, U$4.12, U$4.17
- removed net N$224: C20.1, U$4.29, X4.1
- removed net N$225: U$4.28, X4.2
- removed net N$226: U$4.45, U$4.46
- removed net N$227: R80.1, U$4.32
- removed net N$228: C16.1, U$4.26
- removed net N$229: R79.1, U$4.31
- removed net N$230: C18.1, U$4.14, U$4.19
- removed net N$231: LED6.C, R81.2
- removed net N$232: LED7.C, R91.2
- removed net N$234: LED9.C, R93.2
- removed net N$237: TP126.TP, U10.3
- removed net N$240: LED14.C
- removed net N$244: Q17.3
- removed net N$250: R105.2
- removed net N$254: R107.2
- removed net N$256: Q12.1, R112.1
- removed net N$259: R113.2
- removed net N$260: R114.2
- removed net N$266: JP111.3, JP112.2
- removed net N$3 (its old number): C5.1, D1.3, U$1.21
- removed net N$31 (its old number): U$2.9
- removed net N$32 (its old number): U$2.8
- removed net N$48: Q5.2, Q6.3
- removed net N$79 (its old number): TP92.TP, U2.81
- removed net N$9: C86.1, R95.2, TP127.TP, TP128.TP, U10.7, U10.8
- removed net NRESET: R58.2, U$9.P$15
- removed net NTRST: R54.1
- removed net POT_HIGH: K5.11, POT_HIGH.1
- removed net POT_WIPER: K5.6, POT_WIPER.1
- removed net RGND: GS_R.1, Q1.2, R18.1
- removed net STEERCTRL_+12V: J2402.2
- removed net STEERCTRL_+5V: J2403.2, R2407.2, R2408.2
- removed net STEERCTRL_OUTA: J2401.1, LED2401.A, LED2402.C, U2401.1, U2401.25, U2401.30
- removed net STEERCTRL_OUTB: J2401.2, R2410.1, U2401.15, U2401.16, U2401.21
- removed net STEER_OUT_LED: LED2401.C, LED2402.A, R2410.2
- removed net TCK1: R57.1
- removed net TDI1: R55.1
- removed net THROTTLE-: U$5.P$4
- removed net TMS1: R56.1
- removed net VCC: Q7.4
- removed net VCCIO_2: U2.6
- removed net VCCIO_5: U2.28
- removed net VCCIO_7: U2.32
- removed net VCCIO_8: U2.60
- removed net VIN: U$10.2
- new net 1V8A: C108.1, C84.1, C85.1, L3.2, U8.7, U8.74
- new net 1V8D: C106.1, C107.1, L3.1
- new net 3V3A: C110.1, C111.1, L4.1, U8.2
- new net 5V_FNR: C117.1, D3.K, IC1.1, IC3.4, IC4.14, IC5.5, IC6.5, JP19.1, K1.1, LED2.A, LED26.A, LED3.A, LED4.A, Q5.2, R16.1, R17.1, TP142.TP, TP155.TP, U19.10, U19.16, U20.10, U20.16
- new net ADREFHI: C114.1, L5.2, TP68.TP, U2.46
- new net CON_FIN: JP4.2, U$5.P$14
- new net CON_FNR_HIGH: K1.11, U$5.P$19
- new net CON_FNR_POTGND: IC1.10, IC1.13, U$5.P$16
- new net CON_NIN: Q18.1, R17.2, TP146.TP, U$5.P$20
- new net CON_RIN: U$5.P$13
- new net FNR_CON_THROTTLE-: K1.13, TP161.TP, U$5.P$4
- new net FPGA_MCU_AD1_RES: TP134.TP, U2.45
- new net FPGA_MCU_AD2_RES: TP135.TP, U2.51
- new net FPGA_MCU_AD3_RES: TP136.TP, U2.52
- new net FPGA_MCU_AD4_RES: TP137.TP, U2.53
- new net FPGA_MCU_AD5_RES: TP138.TP, U2.54
- new net FPGA_MCU_AD6_RES: TP139.TP, U2.55
- new net FPGA_MCU_AD7_RES: R22.9, TP140.TP, TP38.TP, U2.56, U2.91
- new net FPGA_MCU_ADO_RES: TP133.TP, U2.44
- new net FPGA_MCU_RES1_RES: R23.16, U2.83
- new net FPGA_MCU_RES2_RES: R23.15, U2.89
- new net FPGA_MCU_RES3_RES: R23.14, U2.90
- new net FPGA_MCU_RES4_RES: R23.13, U2.97
- new net GNDA: C108.2, C110.2, C111.2, C84.2, C85.2, U8.10, U8.4, U8.77
- new net MCU_A_GND: C114.2, JP100.3, JP101.3, JP102.3, JP111.1, JP97.3, JP98.3, JP99.3, L6.1, TP69.TP, U2.47
- new net MCU_COMMS_MISO: JP13.2, TP35.TP, U2.66
- new net MCU_COMMS_MOSI: JP15.2, JP16.2, TP34.TP, U2.65
- new net MCU_COMMS_SCK: JP17.2, TP32.TP, U2.67
- new net MCU_DPOT_CLK: TP25.TP, U2.71, U20.3
- new net MCU_DPOT_CS: TP24.TP, U2.23, U20.6
- new net MCU_DPOT_CSO: IC1.3, U20.11
- new net MCU_DPOT_ENABLE: TP28.TP, U19.3, U2.39
- new net MCU_DPOT_MISO: TP27.TP, U19.6, U2.69
- new net MCU_DPOT_MOSI: TP26.TP, U19.4, U2.70
- new net MCU_FNR_DIRECTION: TP29.TP, TP86.TP, U2.27, U2.58, U20.4
- new net MCU_FNR_DIRECTIONO: IC5.2, IC6.2, IC7.2, R13.1, TP144.TP, U20.13
- new net MCU_FNR_ENABLE: TP37.TP, U2.63, U20.5
- new net MCU_FNR_ENABLEO: Q5.1, TP157.TP, U20.12
- new net MCU_SCREEN_CLK: SV1.3, TP21.TP, U2.36
- new net MCU_SCREEN_CS: SV1.4, TP19.TP, U2.38
- new net MCU_SCREEN_MISO: SV1.1, TP23.TP, U2.34
- new net MCU_SCREEN_MOSI: SV1.2, TP22.TP, U2.35
- new net MONA_AGND: C1.2, JP22.2, U$1.27, U$1.33
- new net MONB_AGND: C6.2, JP24.2, U$2.27, U$2.33
- new net MONC_AGND: C11.2, JP26.2, U$3.27, U$3.33
- new net N$115: LED14.C, Q17.2
- new net N$116: R27.1, TP126.TP, U10.3
- new net N$117: J3.4, U$3.9
- new net N$118: J3.3, U$3.8
- new net N$125: R38.1, U$3.32
- new net N$127: R37.1, U$3.31
- new net N$129: LED6.C, R39.2
- new net N$131: IC6.4, R18.1, TP153.TP
- new net N$132: Q18.2, Q18.4, Q4.3
- new net N$135: Q1.1, R18.2
- new net N$136: Q3.1, R13.2, TP152.TP
- new net N$137: Q2.1, R19.2, R20.2, TP147.TP
- new net N$138: Q18.3, R19.1, R40.2
- new net N$139: Q1.3, Q2.3
- new net N$141: Q19.2, Q3.3, TP151.TP
- new net N$142: Q19.1, R20.1, TP150.TP
- new net N$147: C118.1, IC3.5
- new net N$210: U19.5
- new net N$30: J2.3, U$2.8
- new net N$72: R2403.2, SV2.3
- new net NRST: R25.1, TP92.TP, U2.81
- new net TEST: R24.2, TP90.TP, U2.24
- new net V+: IC3.8
- new net VDD: IC7.14
- new net VSS: IC7.7
- net 0.1: now also U$22.R1
- net 128MHZCLK_OUT_TO_GCLK_FPGA: now also Q7.3
- net 3.3V_SUPERVISED: now also JP48.1, U$10.2; no longer JP112.3
- net 5V_SUPERVISED: now also C14.1, C5.1, C86.1, C9.1, JP21.1, JP21.2, JP23.1, JP23.2, JP25.1, JP25.2, R26.2, R95.2, TP127.TP, TP128.TP, U$1.21, U$2.21, U$3.21, U10.7, U10.8; no longer JP112.1
- net 5V_UNSUPERVISED: now also LED17.A
- net CONGND: now also L7.2
- net CON_MONA_+: now also JP3.1
- net CON_MONA_+_J: now also LED8.A; no longer D1.1, D1.2
- net CON_MONA_-: now also JP22.1; no longer C1.2, C4.2, C5.2, R92.1, U$1.16, U$1.20, U$1.27, U$1.30, U$1.33, U$1.4, U$1.41, U$1.44
- net CON_MONB_+: now also JP2.1, JP20.2
- net CON_MONB_+_J: now also LED7.A; no longer D2.1, D2.2
- net CON_MONB_-: now also C116.2, C117.2, C118.2, C119.2, C69.1, IC1.9, IC3.1, IC4.7, IC5.3, IC6.3, JP24.1, Q6.3, R35.2, U18.3, U18.4, U19.9, U20.9; no longer C10.2, C6.2, C9.2, R91.1, U$2.16, U$2.20, U$2.27, U$2.30, U$2.33, U$2.4, U$2.41, U$2.44
- net CON_MONC_+: now also JP1.1; no longer R49.1, R80.2
- net CON_MONC_+_J: no longer D3.1, D3.2
- net CON_MONC_-: now also JP26.1, R37.2; no longer C11.2, C14.2, C15.2, R46.2, R81.1, U$3.16, U$3.20, U$3.27, U$3.30, U$3.33, U$3.4, U$3.41, U$3.44
- net CON_MONC_SP: now also R38.2; no longer R47.2
- net CON_MOND_+: no longer U$5.P$13
- net CON_MOND_-: no longer C16.2, C17.2, C18.2, C19.2, C20.2, R49.2, R79.2, R93.1, U$4.11, U$4.13, U$4.16, U$4.18, U$4.20, U$4.27, U$4.30, U$4.33, U$4.4, U$4.41, U$4.44, U$5.P$14
- net CON_RELAY_BAT1: now also X4.3; no longer U$5.P$16
- net CON_RELAY_BAT2: now also X4.2; no longer U$5.P$18
- net CON_RELAY_BAT3: now also X4.1; no longer U$5.P$19
- net CON_RELAY_HIGHSIDE: now also X4.4; no longer U$5.P$15
- net DPOT_ENABLE: now also R11.2, U19.14; no longer R12.2
- net ETHERNET_3.3_J_+: now also C109.1, L4.2, R28.1; no longer U8.2
- net FNR_CON_F: now also D1.A, D2.K, JP4.1, Q2.2, R15.2
- net FNR_CON_GROUND: now also Q1.2, Q3.2, R40.1
- net FNR_CON_R: now also D1.K, D2.A, JP27.2, Q19.3, R14.2, TP149.TP
- net FNR_CON_THROTTLE+: now also K1.4, TP162.TP
- net FNR_CON_THROTTLEWIPER: now also K1.6, TP164.TP
- net FPGA_MCU_AD1: now also R22.2; no longer U2.45
- net FPGA_MCU_AD2: now also R22.3; no longer U2.51
- net FPGA_MCU_AD3: now also R22.4; no longer U2.52
- net FPGA_MCU_AD4: now also R22.5; no longer U2.53
- net FPGA_MCU_AD5: now also R22.6; no longer U2.54
- net FPGA_MCU_AD6: now also R22.7; no longer U2.55
- net FPGA_MCU_AD7: now also R22.8; no longer U2.56
- net FPGA_MCU_ADO: now also R22.1; no longer U2.44
- net FPGA_MCU_RES1: now also R23.1; no longer U2.83
- net FPGA_MCU_RES2: now also R23.2; no longer U2.89
- net FPGA_MCU_RES3: now also R23.3; no longer U2.90
- net FPGA_MCU_RES4: now also R23.4; no longer U2.97
- net GND: now also C10.2, C106.2, C107.2, C109.2, C112.1, C113.1, C115.2, C14.2, C15.2, C4.2, C5.2, C74.2, C75.2, C77.2, C78.2, C79.2, C9.2, JP22.3, JP24.3, JP26.3, L6.2, Q17.3, R105.2, R107.2, R113.2, R114.2, R24.1, R26.1, R27.2, R31.1, R32.1, R34.1, R36.1, R39.1, R92.1, SV1.5, U$1.16, U$1.20, U$1.30, U$1.4, U$1.41, U$1.44, U$2.16, U$2.20, U$2.30, U$2.4, U$2.41, U$2.44, U$3.16, U$3.20, U$3.30, U$3.4, U$3.41, U$3.44, U$9.P$8, U19.2, U19.8, U20.2, U20.8; no longer C69.2, C84.2, C85.2, GS_C.1, JP100.3, JP101.3, JP102.3, JP97.3, JP98.3, JP99.3, Q12.2, R2409.1, U2401.18, U2401.19, U2401.20, U2401.26, U2401.27, U2401.28
- net MCU_+3.3V: now also C115.1, JP111.3, L5.1, R25.2, R96.2, TP132.TP, U19.1, U19.7, U2.28, U2.32, U2.6, U2.60, U20.1, U20.7
- net MCU_BATMON_LIN: now also U10.6; no longer U$4.22
- net MCU_BATMON_LINGND: no longer U$4.23
- net MCU_ETHERNET_MISO: now also JP13.1
- net MCU_ETHERNET_MOSI: now also JP16.1
- net MCU_ETHERNET_SCLK: now also JP18.1
- net MCU_ETHERNET_SCS: now also TP30.TP, U2.93
- net MCU_ETHERNET_SEN: now also R28.2
- net MCU_IO_RALAYA: now also U$1.6
- net MCU_IO_RALAYC: now also U$3.6
- net MCU_LINTX: now also U10.4
- net MCU_MISO: now also U19.11
- net MCU_MOSI: now also U19.13
- net MCU_PROG_NRESET: now also U$9.P$15; no longer R58.1
- net MCU_PROG_NTRST: no longer R54.2
- net MCU_PROG_TCK: no longer R57.2
- net MCU_PROG_TDI: no longer R55.2
- net MCU_PROG_TMS: no longer R56.2
- net MCU_SCK: now also U20.14
- net MCU_SPIBRIDGE_CS: now also U1.22
- net MCU_SPIBRIDGE_MISO: now also JP14.2; no longer TP35.TP, U2.66
- net MCU_SPIBRIDGE_MOSI: now also JP15.1; no longer TP34.TP, U2.65
- net MCU_SPIBRIDGE_SCK: now also JP17.1; no longer TP32.TP, U2.67
- net N$10: now also JP19.2, PTC1.2, TP141.TP; no longer TP38.TP, U2.91
- net N$11: now also C116.1, JP20.1, U18.1; no longer TP37.TP, U2.63
- net N$12: now also LED25.A
- net N$130: now also Q4.2, Q4.4, Q5.3; no longer C14.1, D3.3, U$3.21
- net N$15: now also LED23.A
- net N$17: now also J2.4, U$2.9; no longer C9.1, D2.3, U$2.21
- net N$170: now also U19.12; no longer U$3.8
- net N$18: now also LED23.C, R31.2; no longer TP30.TP, U2.93
- net N$183: now also TP123.TP
- net N$192: now also JP69.2
- net N$207: no longer C84.1, C85.1, U8.7, U8.74
- net N$22: now also LED24.C, R32.2; no longer TP26.TP, U2.70
- net N$23: now also LED25.C, R34.2; no longer TP25.TP, U2.71
- net N$24: now also LED26.C, R35.1; no longer TP24.TP, U2.23
- net N$25: now also PTC1.1, U18.2; no longer TP23.TP, U2.34
- net N$26: now also SV2.1; no longer TP22.TP, U2.35
- net N$27: now also R2404.2, SV2.4; no longer TP21.TP, U2.36
- net N$28: now also LED24.A
- net N$29: now also R2402.2, SV2.2; no longer TP19.TP, U2.38
- net N$34: now also R22.16
- net N$35: now also R22.15
- net N$36: now also R22.14
- net N$39: now also R22.13
- net N$49: now also IC1.12, K1.8, TP163.TP; no longer Q1.3, Q2.2
- net N$5: now also J1.4
- net N$50: now also LED4.C, R21.1; no longer LED2.C, R18.2
- net N$51: now also IC1.11, IC1.14, K1.9; no longer LED3.C, R19.2
- net N$52: now also R22.12; no longer LED1.C, R20.1
- net N$53: now also R22.11; no longer IC1.11, IC1.14, K5.9
- net N$54: now also R22.10; no longer IC1.12, K5.8
- net N$55: now also Q6.1, R11.1; no longer LED4.C, R21.1, TP68.TP, U2.46
- net N$56: now also LED2.C, R14.1; no longer Q1.1, R13.2, TP69.TP, U2.47
- net N$57: now also D3.A, K1.16; no longer D5.A, K5.16
- net N$58: now also LED3.C, R15.1; no longer Q3.3, Q4.2
- net N$59: now also C119.1, IC3.6, R16.2, TP154.TP; no longer Q5.1, R17.2
- net N$6: now also J1.3
- net N$60: now also C69.2, IC5.4, IC7.1; no longer Q6.1, R12.1
- net N$61: now also IC7.3, TP156.TP; no longer Q2.1, R11.2
- net N$62: now also Q4.1, TP145.TP; no longer Q3.1, R15.2
- net N$63: now also JP27.1; no longer Q4.1, R16.2
- net N$73: now also LED7.C, R36.2; no longer TP86.TP, U2.58
- net N$77: now also R2405.2, SV2.5; no longer TP90.TP, U2.24
- net PP_3.3V_FPGA: now also Q7.4
- net SPIBRIDGE_ISOLATION_VBUS: now also C112.2, C113.2, U1.7
- net WIZNET_TO_GND: no longer U8.4, U8.77
Routing:
- net N$204: track 0.00 -> 43.8 mm, vias 0 -> 1
- net ETHERNET_3.3_J_+: track 0.00 -> 41.3 mm
- net N$205: track 0.00 -> 40.9 mm, vias 0 -> 1
- net 0.1: track 0.00 -> 38.3 mm
- net V3: track 0.00 -> 32.6 mm
- net N$87: track 0.00 -> 29.3 mm, vias 0 -> 1
- net N$86: track 0.00 -> 29.3 mm, vias 0 -> 1
- net N$202: track 9.38 -> 35.7 mm, vias 0 -> 2
- net VIBC: track 0.00 -> 26.3 mm, vias 0 -> 2
- net SPIBRIDGE_ISOLATION_VBUS: track 25.0 -> 0.00 mm
- net N$84: track 0.00 -> 24.5 mm
- net N$199: track 0.00 -> 23.2 mm, vias 0 -> 2
- net N$145: track 56.9 -> 34.3 mm
- net CON_MONC_SP: track 0.00 -> 21.4 mm, vias 0 -> 2
- net GNDA: track 0.00 -> 17.7 mm
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- removed copper zone on layer 1, net GND
Other:
- board size 202.7 x 118.5 mm -> 185.7 x 158.7 mm
- board text added: "C:/Users/michael roberts/Pictures/Untitled-1.BMP"

Commit message: updarted board
Parts:
- removed IC4: 4030D, 40xx:SO14
- removed JP50: (no value), jumper:JP1
- moved TP161 263.1 mm to (174.6, -8.66)
- moved TP164 262.8 mm to (178.0, -24.1)
- moved TP163 262.3 mm to (182.4, -24.9)
- moved TP160 257.6 mm to (172.1, -9.86)
- moved X4 254.4 mm to (202.1, 56.1), turned to 90 degrees
- moved TP162 253.6 mm to (172.9, -23.9)
- moved TP159 250.3 mm to (164.6, -9.04)
- moved TP158 234.4 mm to (164.6, -26.6)
- moved TP149 218.1 mm to (186.8, -44.6)
- moved TP153 210.8 mm to (163.3, -40.1)
- moved TP148 210.1 mm to (179.0, -43.2)
- moved TP150 209.8 mm to (180.0, -53.3)
- moved TP152 208.2 mm to (154.5, -29.8)
- moved TP151 206.8 mm to (174.5, -54.1)
- moved TP147 203.3 mm to (176.3, -47.8)
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Connections:
- removed net CON_MOND_+: JP85.2
- removed net CON_MOND_-: C57.2
- removed net N$63: JP27.1
- removed net V+: IC3.8
- removed net VDD: IC7.14
- removed net VSS: IC7.7
- new net FNR_CON_FD: D1.K, Q19.3, R14.2, TP149.TP
- new net FNR_CON_RD: D2.K, Q2.2, R15.2, TP148.TP
- net 5V_FNR: now also IC3.8, IC7.14, TP158.TP; no longer IC4.14
- net CON_FNR_POTGND: now also TP160.TP
- net CON_MONA_+: now also JP85.2
- net CON_MONA_-: now also C57.2
- net CON_MONB_-: now also IC7.7, TP159.TP; no longer IC4.7
- net CON_RIN: now also JP27.1
- net FNR_CON_F: no longer D2.K, Q2.2, R15.2
- net FNR_CON_R: no longer D1.K, Q19.3, R14.2, TP149.TP
- net N$59: now also IC3.7
- net N$61: now also IC3.2
- net N$62: now also IC3.3
Routing:
- net CON_NIN: track 0.00 -> 152.7 mm
- net V4: track 0.00 -> 84.7 mm
- net CON_MONB_-: track 0.00 -> 82.2 mm, vias 0 -> 2
- net 5V_FNR: track 0.00 -> 79.0 mm
- net CON_FNR_POTGND: track 0.00 -> 73.1 mm
- net GND: track 43.2 -> 111.8 mm, vias 9 -> 16
- net FNR_CON_R: track 0.00 -> 62.7 mm
- net CON_MONC_-: track 9.57 -> 63.6 mm
- net CONGND: track 3.24 -> 50.3 mm, vias 0 -> 1
- net FNR_CON_THROTTLE+: track 0.00 -> 44.8 mm
- net VOLTAGEJMP_+_TO_INPUT_VREG: track 0.00 -> 43.9 mm, vias 0 -> 1
- net MCU_SCK: track 0.00 -> 42.4 mm
- net MCU_FNR_ENABLEO: track 0.00 -> 42.2 mm
- net CON_FIN: track 0.00 -> 41.5 mm
- net CON_RIN: track 0.00 -> 41.4 mm
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Other:
- board size 185.7 x 158.7 mm -> 188.8 x 159.4 mm

Commit message: did some more routing
Parts:
- moved X4 98.0 mm to (112.4, 95.5), turned to 0 degrees
- moved JP14 81.9 mm to (62.9, 74.3)
- moved Q13 77.5 mm to (106.8, 92.6)
- moved TP106 76.8 mm to (108.2, 87.8)
- moved Q10 67.6 mm to (122.8, 90.0), turned to 90 degrees
- moved Q11 64.7 mm to (123.3, 93.3)
- moved R110 60.8 mm to (126.1, 88.6)
- moved TP109 58.3 mm to (117.7, 41.9)
- moved R111 54.4 mm to (127.5, 97.0), turned to 0 degrees
- moved TP58 50.8 mm to (57.4, 53.5)
- moved TP50 50.6 mm to (58.2, 63.4)
- moved TP70 47.2 mm to (74.2, 45.6)
- moved TP63 37.8 mm to (87.9, 27.9)
- moved TP136 32.6 mm to (94.6, 53.8)
- moved TP93 28.3 mm to (69.8, 45.2)
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Routing:
- net N$165: track 0.00 -> 20.9 mm
- net N$166: track 0.00 -> 20.2 mm
- net FPGA_MCU_AD6_RES: track 0.00 -> 17.2 mm
- net GND: track 111.8 -> 128.2 mm, vias 16 -> 17
- net MCU_COMMS_SCK: track 0.00 -> 15.8 mm
- net N$164: track 0.00 -> 15.6 mm
- net MCU_PROG_TMS: track 0.00 -> 14.9 mm
- net FPGA_MCU_AD3_RES: track 0.00 -> 13.9 mm
- net MCU_+1.2V: track 0.00 -> 13.5 mm
- net FPGA_MCU_AD2_RES: track 0.00 -> 13.0 mm
- net MCU_SPIBRIDGE_CS: track 0.00 -> 13.0 mm
- net MCU_FNR_DIRECTION: track 0.00 -> 12.6 mm
- net FPGA_MCU_AD4_RES: track 0.00 -> 12.5 mm
- net MCU_DPOT_MOSI: track 0.00 -> 11.2 mm
- net FPGA_MCU_AD5_RES: track 0.00 -> 10.9 mm
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