File: Electrical Schematics/Version2/Schematics/boardv2a.brd (EAGLE design)
At the start: 207.3 x 160.2 mm, 559 parts, among them IC1 MCP41HVX1ST, IC2 ADUM4160BRW, IC3 SE555D, IC5 74LVC1G04DBV, IC6 74LVC1G04DBV, IC7 4030D, K1 G5V-2, Q1 IRLML2060TRPBFBSS123LT1G, Q10 IRLML2060TRPBFBSS123LT1G, Q11 IRLML2060TRPBFBSS123LT1G, Q13 IRLML2060TRPBFBSS123LT1G, Q14 IRLML2060TRPBFBSS123LT1G, Q15 IRLML2060TRPBFBSS123LT1G, Q16 IRLML2060TRPBFBSS123LT1G, Q17 IRLML2060TRPBFBSS123LT1G, Q18 BSP170P, Q19 IRLML2060TRPBFBSS123LT1G, Q2 IRLML2060TRPBFBSS123LT1G, Q3 IRLML2060TRPBFBSS123LT1G, Q4 BSP170P, Q5 IRLML2060TRPBFBSS123LT1G, Q6 IRLML2060TRPBFBSS123LT1G, Q7 ASFL1, Q8 IRLML2060TRPBFBSS123LT1G, Q9 IRLML2060TRPBFBSS123LT1G, U1 CP2130-GM, U10 SN65HVDA100-Q1_D_8, U11 ADUM3442CRWZ, U12 ADUM3442CRWZ, U13 ADUM3442CRWZ, U14 ADUM3442CRWZ, U15 ADUM3442CRWZ, U16 ADUM3442CRWZ, U17 ADUM3442CRWZ, U18 LM1085_KTT_3, U19 ADUM3442CRWZ, U2 TMS570LS0432_PZ_100, U20 ADUM3442CRWZ, U3 LM1085_KTT_3, U4 LM1085_KTT_3, U5 LM1084_KTT_3, U6 TPS3514_D_14, U7 LM1085_KTT_3, U9 ADUM3442CRWZ, X4 5566-4

Commit message: Lots of routing and some lib updates
Parts:
- removed R22, R23: (no value), resistor-bourns:4816P
- removed TP117: TPB1,27, testpad:B1,27
- added U$32, U$4: RHM1620CT-ND, shit:MNR18
- moved C93 104.0 mm to (99.3, -37.3)
- moved C105 92.0 mm to (121.9, -37.2)
- moved C115 91.6 mm to (96.4, 50.0), turned to 180 degrees
- moved C103 86.2 mm to (67.3, -40.1), turned to 270 degrees
- moved JP53 85.1 mm to (102.9, 51.8), turned to 270 degrees
- moved JP11 82.4 mm to (76.2, -27.7)
- moved JP5 71.1 mm to (116.0, 6.86)
- moved C90 71.1 mm to (109.1, -3.94)
- moved C91 67.9 mm to (110.0, -1.65)
- moved C101 62.4 mm to (-0.89, -25.8), turned to 180 degrees
- moved C99 52.8 mm to (37.5, -40.1), turned to 270 degrees
- moved JP9 47.5 mm to (45.0, -26.0)
- moved TP122 45.1 mm to (112.8, 31.5)
- moved JP6 44.9 mm to (98.0, -28.8)
- moved C98 44.1 mm to (51.2, -31.6), turned to 270 degrees
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Connections:
- new net 5V_SU_J: JP25.2, U$3.21
- new net N$301: JP80.8
- new net N$302: JP80.7
- net 5V_SUPERVISED: no longer JP25.2, U$3.21
- net FPGA_MCU_AD1: now also U$4.P$13; no longer R22.2
- net FPGA_MCU_AD2: now also U$4.P$11; no longer R22.3
- net FPGA_MCU_AD3: now also U$4.P$9; no longer R22.4
- net FPGA_MCU_AD4: now also U$4.P$7; no longer R22.5
- net FPGA_MCU_AD5: now also U$4.P$5; no longer R22.6
- net FPGA_MCU_AD6: now also U$4.P$3; no longer R22.7
- net FPGA_MCU_AD7: now also U$4.P$1; no longer R22.8
- net FPGA_MCU_AD7_RES: now also U$4.P$2; no longer R22.9
- net FPGA_MCU_ADO: now also U$4.P$15; no longer R22.1
- net FPGA_MCU_RES1: now also U$32.P$1; no longer R23.1
- net FPGA_MCU_RES1_RES: now also U$32.P$2; no longer R23.16
- net FPGA_MCU_RES2: now also U$32.P$3; no longer R23.2
- net FPGA_MCU_RES2_RES: now also U$32.P$4; no longer R23.15
- net FPGA_MCU_RES3: now also U$32.P$5; no longer R23.3
- net FPGA_MCU_RES3_RES: now also U$32.P$6; no longer R23.14
- net FPGA_MCU_RES4: now also U$32.P$7; no longer R23.4
- net FPGA_MCU_RES4_RES: now also U$32.P$8; no longer R23.13
- net GND: now also L7.1
- net MCU_IO_RALAYB: now also U$2.6
- net N$185: no longer TP117.TP
- net N$34: now also U$4.P$16; no longer R22.16
- net N$35: now also U$4.P$14; no longer R22.15
- net N$36: now also U$4.P$12; no longer R22.14
- net N$39: now also U$4.P$10; no longer R22.13
- net N$52: now also U$4.P$8; no longer R22.12
- net N$53: now also U$4.P$6; no longer R22.11
- net N$54: now also U$4.P$4; no longer R22.10
- net N$87: no longer JP80.7
- net N$88: no longer JP80.8
Routing:
- net CONGND: track 50.3 -> 206.2 mm, vias 1 -> 4
- net 3.3V_SUPERVISED: track 16.9 -> 141.3 mm, vias 0 -> 4
- net GND: track 240.5 -> 310.3 mm, vias 23 -> 39
- net V6: track 0.00 -> 52.7 mm, vias 0 -> 1
- net V7: track 0.00 -> 41.0 mm, vias 0 -> 3
- net V5: track 0.00 -> 37.1 mm, vias 0 -> 3
- net N$99: track 0.00 -> 35.9 mm, vias 0 -> 1
- net N$141: track 0.00 -> 35.9 mm, vias 0 -> 2
- net V3: track 45.6 -> 79.2 mm
- net N$95: track 0.00 -> 32.7 mm
- net VIAE: track 0.00 -> 31.3 mm
- net VIAG: track 0.00 -> 28.1 mm
- net N$105: track 0.00 -> 27.0 mm
- net VOCE: track 0.00 -> 25.9 mm, vias 0 -> 2
- net VODF: track 0.00 -> 25.9 mm, vias 0 -> 2
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
Commit message: cleaned up FPGA
Parts:
- removed JP75, JP79, JP80, JP89, JP90, JP91, JP92, JP93, JP94, JP95: (no value), pinhead:1X08
- added TP117, TP143, TP165, TP166, TP167, TP168, TP169, TP170, TP171, TP172, TP173, TP174, TP175, TP176, TP177, TP178, TP179, TP180, TP181, TP182, TP183, TP184, TP185, TP186, TP187, TP188, TP189, TP190, TP191, TP192, TP193, TP194, TP195, TP196, TP197, TP198, TP199, TP200, TP201, TP202, TP203, TP204, TP205, TP206, TP207, TP208, TP209, TP210, TP211, TP212, TP213, TP214, TP215, TP216, TP217, TP218, TP219, TP220, TP221, TP222, TP223, TP224, TP225, TP228, TP229, TP230, TP231, TP232, TP233: TPPAD1-13, testpad:P1-13
- moved JP21 124.2 mm to (170.4, 70.2)
- moved JP102 36.6 mm to (40.6, 44.2)
- moved JP5 31.5 mm to (94.7, -16.4), turned to 90 degrees
- moved JP101 30.2 mm to (25.4, 36.1)
- moved JP100 28.9 mm to (39.9, 49.0)
- moved JP97 28.6 mm to (31.9, 45.0)
- moved C92 25.3 mm to (83.2, -44.3)
- moved TP71 24.7 mm to (47.4, 49.5)
- moved JP99 20.8 mm to (39.5, 37.2)
- moved Q7 20.2 mm to (55.1, -3.43), flipped to the bottom, turned to 270 degrees
- moved L7 20.1 mm to (127.1, -16.4)
- moved TP84 19.8 mm to (50.4, 27.8)
- moved C91 18.7 mm to (108.6, -20.3)
- moved C27 17.4 mm to (81.4, 2.67)
- moved C89 15.0 mm to (47.6, 7.87), turned to 180 degrees
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Connections:
- removed net N$301: JP80.8
- removed net N$302: JP80.7
- removed net NC: JP90.7
- net FPGA_L12N_2: now also TP185.TP; no longer JP90.2
- net FPGA_L12P_2: now also TP186.TP; no longer JP90.1
- net FPGA_L13N_2: now also TP183.TP; no longer JP90.4
- net FPGA_L13P_2: now also TP184.TP; no longer JP90.3
- net FPGA_L14N_2: now also TP181.TP; no longer JP90.6
- net FPGA_L14P_2: now also TP182.TP; no longer JP90.5
- net FPGA_L1N_0: now also TP204.TP; no longer JP94.2
- net FPGA_L1N_1: no longer JP95.4
- net FPGA_L1N_2: now also TP174.TP; no longer JP91.4
- net FPGA_L1N_3: now also TP215.TP; no longer JP93.6
- net FPGA_L1P_0: now also TP203.TP; no longer JP94.1
- net FPGA_L1P_1: no longer JP95.3
- net FPGA_L1P_2: now also TP176.TP; no longer JP91.3
- net FPGA_L1P_3: now also TP214.TP; no longer JP93.5
- net FPGA_L2N_0: now also TP206.TP; no longer JP94.4
- net FPGA_L2N_2: now also TP173.TP; no longer JP91.6
- net FPGA_L2N_3: now also TP217.TP; no longer JP93.8
- net FPGA_L2P_0: now also TP205.TP; no longer JP94.3
- net FPGA_L2P_2: now also TP175.TP; no longer JP91.5
- net FPGA_L2P_3: now also TP216.TP; no longer JP93.7
- net FPGA_L30N_2: now also TP179.TP; no longer JP90.8
- net FPGA_L31N_2: now also TP193.TP; no longer JP89.2
- net FPGA_L31P_2: now also TP194.TP; no longer JP89.1
- net FPGA_L32N_1: no longer JP95.6
- net FPGA_L32P_1: no longer JP95.5
- net FPGA_L36N_3: now also TP231.TP; no longer JP80.2
- net FPGA_L36P_3: now also TP233.TP; no longer JP80.1
- net FPGA_L37N_3: now also TP230.TP; no longer JP80.4
- net FPGA_L37P_3: now also TP232.TP; no longer JP80.3
- net FPGA_L3N_0: now also TP209.TP; no longer JP94.6
- net FPGA_L3N_2: now also TP117.TP; no longer JP91.8
- net FPGA_L3P_0: now also TP207.TP; no longer JP94.5
- net FPGA_L3P_2: now also TP172.TP; no longer JP91.7
- net FPGA_L41N_3: now also TP228.TP; no longer JP80.6
- net FPGA_L41P_3: now also TP229.TP; no longer JP80.5
- net FPGA_L42N_3: now also TP224.TP; no longer JP79.2
- net FPGA_L42N_GCLK6_TRDY1_1: no longer JP95.8
- net FPGA_L42P_1: no longer JP95.7
- net FPGA_L42P_3: now also TP225.TP; no longer JP79.1
- net FPGA_L43N_1: now also TP169.TP; no longer JP92.2
- net FPGA_L43N_3: now also TP222.TP; no longer JP79.4
- net FPGA_L43P_1: now also TP170.TP; no longer JP92.1
- net FPGA_L43P_3: now also TP223.TP; no longer JP79.3
- net FPGA_L44N_3: now also TP220.TP; no longer JP79.6
- net FPGA_L44P_3: now also TP221.TP; no longer JP79.5
- net FPGA_L45N_1: now also TP167.TP; no longer JP92.4
- net FPGA_L45P_1: now also TP168.TP; no longer JP92.3
- net FPGA_L46N_1: now also TP165.TP; no longer JP92.6
- net FPGA_L46P_1: now also TP166.TP; no longer JP92.5
- net FPGA_L47N_1: now also TP171.TP; no longer JP92.8
- net FPGA_L47P_1: now also TP143.TP; no longer JP92.7
- net FPGA_L48N_2: now also TP191.TP; no longer JP89.4
- net FPGA_L48P_2: now also TP192.TP; no longer JP89.3
- net FPGA_L49N_2: now also TP189.TP; no longer JP89.6
- net FPGA_L49P_2: now also TP190.TP; no longer JP89.5
- net FPGA_L4N_0: now also TP208.TP; no longer JP94.8
- net FPGA_L4P_0: now also TP180.TP; no longer JP94.7
- net FPGA_L62N_0: now also TP201.TP; no longer JP75.2
- net FPGA_L62N_2: now also TP187.TP; no longer JP89.8
- net FPGA_L62P_0: now also TP202.TP; no longer JP75.1
- net FPGA_L62P_2: now also TP188.TP; no longer JP89.7
- net FPGA_L63N_0: now also TP199.TP; no longer JP75.4
- net FPGA_L63P_0: now also TP200.TP; no longer JP75.3
- net FPGA_L64N_0: now also TP197.TP; no longer JP75.6
- net FPGA_L64N_2: now also TP211.TP; no longer JP93.2
- net FPGA_L64P_0: now also TP198.TP; no longer JP75.5
- net FPGA_L64P_2: now also TP210.TP; no longer JP93.1
- net FPGA_L65N_0: now also TP195.TP; no longer JP75.8
- net FPGA_L65N_2: now also TP213.TP; no longer JP93.4
- net FPGA_L65P_0: now also TP196.TP; no longer JP75.7
- net FPGA_L65P_2: now also TP212.TP; no longer JP93.3
- net FPGA_L66N_0: no longer JP95.2
- net FPGA_L66P_0: no longer JP95.1
- net FPGA_L74N_1: now also TP177.TP; no longer JP91.2
- net FPGA_L74P_1: now also TP178.TP; no longer JP91.1
- net FPGA_L83N_3: now also TP218.TP; no longer JP79.8
- net FPGA_L83P_3: now also TP219.TP; no longer JP79.7
Routing:
- net MCU_DPOT_CLK: track 9.56 -> 88.4 mm, vias 0 -> 1
- net MCU_FNR_ENABLE: track 8.25 -> 82.2 mm, vias 0 -> 1
- net MCU_FNR_DIRECTION: track 12.6 -> 85.3 mm, vias 0 -> 1
- net MCU_+3.3V: track 17.3 -> 48.3 mm
- net GND: track 310.3 -> 336.0 mm, vias 39 -> 42
- net MCU_DPOT_MISO: track 8.02 -> 33.2 mm, vias 0 -> 1
- net MCU_DPOT_MOSI: track 11.2 -> 32.9 mm, vias 0 -> 1
- net FPGA_L48P_2: track 0.00 -> 21.2 mm
- net MCU_DPOT_ENABLE: track 6.84 -> 27.5 mm, vias 0 -> 1
- net FPGA_L14P_2: track 0.00 -> 18.4 mm
- net FPGA_L14N_2: track 0.00 -> 16.1 mm
- net FPGA_L64N_2: track 0.00 -> 15.6 mm
- net FPGA_L48N_2: track 0.00 -> 15.3 mm
- net FPGA_L13N_2: track 0.00 -> 14.4 mm
- net FPGA_L12N_2: track 0.00 -> 14.2 mm
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
Commit message: did more work on  fpga
Parts:
- moved TP187 115.0 mm to (-39.0, -6.22)
- moved TP188 113.6 mm to (-34.2, -11.6)
- moved TP231 97.1 mm to (27.4, -2.79)
- moved TP232 95.5 mm to (33.3, -2.92)
- moved TP229 91.1 mm to (24.9, -0.38)
- moved TP230 90.2 mm to (30.1, -1.65)
- moved TP228 83.0 mm to (28.7, 1.02)
- moved TP225 78.6 mm to (20.6, 0.00)
- moved TP224 70.1 mm to (24.6, 3.17)
- moved TP10 65.6 mm to (96.9, 64.4)
- moved TP223 64.7 mm to (25.8, 5.59)
- moved TP49 39.1 mm to (47.0, 22.9)
- moved TP62 38.0 mm to (81.2, 21.6)
- moved JP18 35.7 mm to (26.2, 64.4), turned to 270 degrees
- moved TP90 31.2 mm to (77.0, 5.59)
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Routing:
- net FPGA_L42P_3: track 0.00 -> 24.2 mm
- net FPGA_L43N_3: track 0.00 -> 23.5 mm
- net FPGA_L46N_1: track 0.00 -> 23.3 mm
- net FPGA_L36P_3: track 0.00 -> 22.9 mm
- net FPGA_L46P_1: track 0.00 -> 21.1 mm
- net GND: track 336.0 -> 356.2 mm, vias 42 -> 43
- net FPGA_L47P_1: track 0.00 -> 20.2 mm
- net FPGA_L42N_3: track 0.00 -> 18.4 mm
- net FPGA_L2N_3: track 0.00 -> 18.1 mm
- net FPGA_L43P_3: track 0.00 -> 17.2 mm
- net FPGA_L41P_3: track 0.00 -> 17.2 mm
- net TDI: track 0.00 -> 16.8 mm
- net FPGA_L47N_1: track 0.00 -> 16.6 mm
- net FPGA_L83P_3: track 0.00 -> 15.8 mm
- net FPGA_L74N_1: track 0.00 -> 14.8 mm
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
Commit message: updated board
Parts:
- moved U$4 26.7 mm to (49.8, 30.2)
- moved U$32 26.7 mm to (56.4, 29.3)
- moved LED24 6.92 mm to (65.3, 33.9)
- moved R2 2.90 mm to (150.4, 81.5)
- moved Q10 2.17 mm to (111.9, 86.4)
- moved C8 0.74 mm to (142.2, 77.7)
- moved JP22 0.36 mm to (150.5, 88.5)
