File: Electrical Schematics/Version2/Schematics/boardv2a.sch (EAGLE design)
At the start: 629 parts, among them IC1 MCP41HVX1ST, IC2 ADUM4160BRW, IC3 SE555D, IC5 74LVC1G04DBV, IC6 74LVC1G04DBV, IC7 4030D, K1 G5V-2, K2 CP1SA-12V, Q1 IRLML2060TRPBFBSS123LT1G, Q10 IRLML2060TRPBFBSS123LT1G, Q11 IRLML2060TRPBFBSS123LT1G, Q12 IRLML2060TRPBFBSS123LT1G, Q13 IRLML2060TRPBFBSS123LT1G, Q17 IRLML2060TRPBFBSS123LT1G, Q18 MOSFET-PCHANNEL, Q19 IRLML2060TRPBFBSS123LT1G, Q2 IRLML2060TRPBFBSS123LT1G, Q3 IRLML2060TRPBFBSS123LT1G, Q4 MOSFET-PCHANNEL, Q5 MOSFET-PCHANNEL, Q6 IRLML2060TRPBFBSS123LT1G, Q7 ASFL1, Q8 IRLML2060TRPBFBSS123LT1G, Q9 IRLML2060TRPBFBSS123LT1G, U1 CP2130-GM, U10 SN65HVDA100-Q1_D_8, U11 ADUM3442CRWZ, U12 ADUM3442CRWZ, U13 ADUM3442CRWZ, U14 ADUM3442CRWZ, U15 ADUM3442CRWZ, U16 ADUM3442CRWZ, U17 ADUM3442CRWZ, U18 LM1085_KTT_3, U19 ADUM3442CRWZ, U2 TMS570LS0432_PZ_100, U20 ADUM3442CRWZ, U3 LM1085_KTT_3, U4 LM1085_KTT_3, U5 LM1084_KTT_3, U6 TPS3514_D_14, U7 LM1085_KTT_3, U9 ADUM3442CRWZ, X4 5566-4

Commit message: updaqted mcu
Connections:
- new net FPGA_MCU_CLKJ: U$32G$6.P$2, U2.GIOA[2]/INT[2]
- new net FPGA_MCU_RWJ: U$32G$8.P$2, U2.GIOA[0]/INT[0]
- new net FPGA_MCU_STATJ: U$32G$7.P$2, U2.GIOA[1]/INT[1]
- net FPGA_MCU_CLK: now also U$32G$6.P$1; no longer U2.GIOA[2]/INT[2]
- net FPGA_MCU_RW: now also U$32G$8.P$1; no longer U2.GIOA[0]/INT[0]
- net FPGA_MCU_STAT: now also U$32G$7.P$1; no longer U2.GIOA[1]/INT[1]
Changed lines of the file:
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@@
 <instance part="U$32" gate="G$4" x="-172.72" y="-27.94"/>
 <instance part="U$32" gate="G$5" x="-319.376290625" y="-42.0306"/>
-<instance part="U$32" gate="G$6" x="-304.8" y="-33.02"/>
-<instance part="U$32" gate="G$7" x="-307.34" y="-27.94"/>
-<instance part="U$32" gate="G$8" x="-307.34" y="-22.86"/>
+<instance part="U$32" gate="G$6" x="-149.86" y="78.74"/>
+<instance part="U$32" gate="G$7" x="-154.94" y="81.28"/>
+<instance part="U$32" gate="G$8" x="-154.94" y="83.82"/>
 <instance part="U$4" gate="G$1" x="-274.32" y="-5.08"/>
 <instance part="U$4" gate="G$2" x="-274.32" y="5.08"/>
@@
 <net name="FPGA_MCU_RW" class="0">
 <segment>
-<pinref part="U2" gate="A" pin="GIOA[0]/INT[0]"/>
-<wire x1="12.7" y1="83.82" x2="-170.18" y2="83.82" width="0.1524" layer="91"/>
-<wire x1="-170.18" y1="83.82" x2="-170.18" y2="71.12" width="0.1524" layer="91"/>
-<wire x1="-170.18" y1="71.12" x2="-180.34" y2="71.12" width="0.1524" layer="91"/>
-<label x="-213.36" y="71.12" size="1.778" layer="95" rot="R180" xref="yes"/>
 <pinref part="TP48" gate="G$1" pin="TP"/>
 <wire x1="-180.34" y1="71.12" x2="-208.28" y2="71.12" width="0.1524" layer="91"/>
 <junction x="-180.34" y="71.12"/>
-<junction x="12.7" y="83.82"/>
+<wire x1="-170.18" y1="71.12" x2="-180.34" y2="71.12" width="0.1524" layer="91"/>
+<wire x1="-170.18" y1="83.82" x2="-170.18" y2="71.12" width="0.1524" layer="91"/>
+<wire x1="-162.56" y1="83.82" x2="-170.18" y2="83.82" width="0.1524" layer="91"/>
+<pinref part="U$32" gate="G$8" pin="P$1"/>
+<label x="-213.36" y="71.12" size="1.778" layer="95" rot="R180" xref="yes"/>
 </segment>
 </net>
 <net name="FPGA_MCU_STAT" class="0">
 <segment>
-<pinref part="U2" gate="A" pin="GIOA[1]/INT[1]"/>
-<wire x1="12.7" y1="81.28" x2="-165.1" y2="81.28" width="0.1524" layer="91"/>
-<wire x1="-165.1" y1="81.28" x2="-165.1" y2="66.04" width="0.1524" layer="91"/>
-<wire x1="-165.1" y1="66.04" x2="-180.34" y2="66.04" width="0.1524" layer="91"/>
-<label x="-213.36" y="66.04" size="1.778" layer="95" rot="R180" xref="yes"/>
 <pinref part="TP49" gate="G$1" pin="TP"/>
 <wire x1="-180.34" y1="66.04" x2="-208.28" y2="66.04" width="0.1524" layer="91"/>
 <junction x="-180.34" y="66.04"/>
-<junction x="12.7" y="81.28"/>
-</segment>
-</net>
-<net name="FPGA_MCU_CLK" class="0">
-<segment>
-<wire x1="15.24" y1="78.74" x2="12.7" y2="78.74" width="0.1524" layer="91"/>
-<wire x1="12.7" y1="78.74" x2="-160.02" y2="78.74" width="0.1524" layer="91"/>
-<wire x1="-160.02" y1="78.74" x2="-160.02" y2="60.96" width="0.1524" layer="91"/>
-<wire x1="-160.02" y1="60.96" x2="-180.34" y2="60.96" width="0.1524" layer="91"/>
-<label x="-213.36" y="60.96" size="1.778" layer="95" rot="R180" xref="yes"/>
-<pinref part="TP50" gate="G$1" pin="TP"/>
-<wire x1="-180.34" y1="60.96" x2="-208.28" y2="60.96" width="0.1524" layer="91"/>
-<junction x="-180.34" y="60.96"/>
-<pinref part="U2" gate="A" pin="GIOA[2]/INT[2]"/>
-<junction x="12.7" y="78.74"/>
+<wire x1="-165.1" y1="66.04" x2="-180.34" y2="66.04" width="0.1524" layer="91"/>
+<wire x1="-165.1" y1="81.28" x2="-165.1" y2="66.04" width="0.1524" layer="91"/>
+<wire x1="-162.56" y1="81.28" x2="-165.1" y2="81.28" width="0.1524" layer="91"/>
+<pinref part="U$32" gate="G$7" pin="P$1"/>
+<label x="-213.36" y="66.04" size="1.778" layer="95" rot="R180" xref="yes"/>
 </segment>
 </net>
@@
 </segment>
 </net>
+<net name="FPGA_MCU_CLK" class="0">
+<segment>
+<pinref part="TP50" gate="G$1" pin="TP"/>
+<wire x1="-180.34" y1="60.96" x2="-208.28" y2="60.96" width="0.1524" layer="91"/>
+<junction x="-180.34" y="60.96"/>
+<wire x1="-160.02" y1="60.96" x2="-180.34" y2="60.96" width="0.1524" layer="91"/>
+<wire x1="-160.02" y1="78.74" x2="-160.02" y2="60.96" width="0.1524" layer="91"/>
+<wire x1="-157.48" y1="78.74" x2="-160.02" y2="78.74" width="0.1524" layer="91"/>
+<pinref part="U$32" gate="G$6" pin="P$1"/>
+<label x="-213.36" y="60.96" size="1.778" layer="95" rot="R180" xref="yes"/>
+</segment>
+</net>
+<net name="FPGA_MCU_RWJ" class="0">
+<segment>
+<pinref part="U2" gate="A" pin="GIOA[0]/INT[0]"/>
+<wire x1="12.7" y1="83.82" x2="-147.32" y2="83.82" width="0.1524" layer="91"/>
+<junction x="12.7" y="83.82"/>
+<pinref part="U$32" gate="G$8" pin="P$2"/>
+</segment>
+</net>
+<net name="FPGA_MCU_STATJ" class="0">
+<segment>
+<pinref part="U2" gate="A" pin="GIOA[1]/INT[1]"/>
+<wire x1="12.7" y1="81.28" x2="-147.32" y2="81.28" width="0.1524" layer="91"/>
+<junction x="12.7" y="81.28"/>
+<pinref part="U$32" gate="G$7" pin="P$2"/>
+</segment>
+</net>
+<net name="FPGA_MCU_CLKJ" class="0">
+<segment>
+<wire x1="15.24" y1="78.74" x2="12.7" y2="78.74" width="0.1524" layer="91"/>
+<wire x1="12.7" y1="78.74" x2="-142.24" y2="78.74" width="0.1524" layer="91"/>
+<pinref part="U2" gate="A" pin="GIOA[2]/INT[2]"/>
+<junction x="12.7" y="78.74"/>
+<pinref part="U$32" gate="G$6" pin="P$2"/>
+</segment>
+</net>
