File: Electrical Schematics/Version3/Schematics/boardv2a.sch (EAGLE design)
At the start: 629 parts, among them IC1 MCP41HVX1ST, IC2 ADUM4160BRW, IC3 SE555D, IC5 74LVC1G04DBV, IC6 74LVC1G04DBV, IC7 4030D, K1 G5V-2, K2 CP1SA-12V, Q1 IRLML2060TRPBFBSS123LT1G, Q10 IRLML2060TRPBFBSS123LT1G, Q11 IRLML2060TRPBFBSS123LT1G, Q12 IRLML2060TRPBFBSS123LT1G, Q13 IRLML2060TRPBFBSS123LT1G, Q17 IRLML2060TRPBFBSS123LT1G, Q18 MOSFET-PCHANNEL, Q19 IRLML2060TRPBFBSS123LT1G, Q2 IRLML2060TRPBFBSS123LT1G, Q3 IRLML2060TRPBFBSS123LT1G, Q4 MOSFET-PCHANNEL, Q5 MOSFET-PCHANNEL, Q6 IRLML2060TRPBFBSS123LT1G, Q7 ASFL1, Q8 IRLML2060TRPBFBSS123LT1G, Q9 IRLML2060TRPBFBSS123LT1G, U1 CP2130-GM, U10 SN65HVDA100-Q1_D_8, U11 ADUM3442CRWZ, U12 ADUM3442CRWZ, U13 ADUM3442CRWZ, U14 ADUM3442CRWZ, U15 ADUM3442CRWZ, U16 ADUM3442CRWZ, U17 ADUM3442CRWZ, U18 LM1085_KTT_3, U19 ADUM3442CRWZ, U2 TMS570LS0432_PZ_100, U20 ADUM3442CRWZ, U3 LM1085_KTT_3, U4 LM1085_KTT_3, U5 LM1084_KTT_3, U6 TPS3514_D_14, U7 LM1085_KTT_3, U9 ADUM3442CRWZ, X4 5566-4

Commit message: updated ldo library and some routing
Parts:
- removed C1, C11, C6: 47nF, eagle-ltspice:CC0603
- removed C10, C15, C4: 220pf, eagle-ltspice:CC0603
- removed C12, C2, C7: 220nF, eagle-ltspice:CC0603
- removed C13, C3, C8: 1uF, eagle-ltspice:CC0603
- removed C14, C5, C9: 4.7UF, eagle-ltspice:CC0603
- removed C86, C87: 0.1 uF, rcl:C-EUC0402
- removed J1, J2, J3: (no value), con-lsta:JU05
- removed JP1, JP2, JP21, JP23, JP25, JP28, JP29, JP3, JP30: (no value), jumper:JP1E
- removed JP22, JP24, JP26: (no value), jumper:JP2E
- removed LED6, LED7, LED8: (no value), led:LEDSML1206
- removed R1, R3, R7: 2.2KOHM, SparkFun-Passives:RESISTOR0603-RES
- removed R10, R37, R38, R5, R6, R9: 500ohm, SparkFun-Passives:RESISTOR0603-RES
- removed R12, R22, R23: 3.3k, SparkFun-Passives:RESISTOR0603-RES
- removed R2, R4, R8: 100UOHMS, SparkFun-Passives:RESISTOR0603-RES
- removed R26, R27, R95: 1k, SparkFun-Passives:RESISTOR0603-RES
- removed R36, R39, R92: 560ohms, SparkFun-Passives:RESISTOR0603-RES
- removed SV3, SV4, SV5: (no value), con-lstb:MA03-2
- removed TP126, TP127, TP128, TP129: TPB2,54, testpad:TPB2,54
- removed U$1, U$2, U$3: (no value), freescalemod:MM912_637D1
- removed U10: SN65HVDA100-Q1_D_8, shit:SN65HVDA100-Q1_D_8
- removed X1, X2, X3: (no value), con-molex:KK-156-2
Connections:
- removed net 5V_SUP_J1: JP23.2, U$2.VSUP
- removed net 5V_SU_J123: JP25.2, U$3.VSUP
- removed net BKGND: R12.1, SV3.6, U$1.BKGD/MODC
- removed net BKGNDB: R22.1, SV4.6
- removed net BKGNDC: R23.1, SV5.6, U$3.BKGD/MODC
- removed net CON_MONA_+_J: JP3.2, LED8.A, R1.2
- removed net CON_MONB_+_J: JP2.2, LED7.A, R3.2
- removed net CON_MONC_+_J: JP1.2, LED6.A, R7.2
- removed net MCU_BATMON_LIN: C87.1, R95.1, TP129.TP, U$1.LIN, U$2.LIN, U$3.LIN, U10.LIN
- removed net MCU_BATMON_LINGND: C86.2, C87.2, U$1.LGND, U$2.LGND, U$3.LGND, U10.GND
- removed net MONA_AGND: C1.2, JP22.2, U$1.ADCGND, U$1.AGND
- removed net MONB_AGND: C6.2, JP24.2, U$2.ADCGND, U$2.AGND
- removed net MONC_AGND: C11.2, JP26.2, U$3.ADCGND, U$3.AGND
- removed net N$1: R1.1, U$1.VSENSE
- removed net N$116: R27.1, TP126.TP, U10.NWAKE
- removed net N$117: J3.4, U$3.PA1/MOSI
- removed net N$118: J3.3, U$3.PA2/SCK
- removed net N$119: J3.2, U$3.PA3/*SS
- removed net N$120: R7.1, U$3.VSENSE
- removed net N$121: C12.1, U$3.VDDRX, U$3.VDDX
- removed net N$122: C15.1, U$3.TSUP, X3-1.S
- removed net N$123: U$3.VTEMP, X3-2.S
- removed net N$125: R38.1, U$3.ISENSEH
- removed net N$126: C11.1, U$3.VDDA
- removed net N$127: R37.1, U$3.ISENSEL
- removed net N$129: LED6.C, R39.2
- removed net N$13: U$1.VTEMP, X1-2.S
- removed net N$14: JP28.2, SV3.3, U$1.*RESET
- removed net N$16: C3.1, U$1.VDDD2D, U$1.VDDH
- removed net N$17: J2.4, U$2.PA1/MOSI
- removed net N$19: JP30.1, U$3.*RESET_A
- removed net N$21: JP28.1, U$1.*RESET_A
- removed net N$233: LED8.C, R92.2
- removed net N$3: J2.5, U$2.PA0/MISO
- removed net N$30: J2.3, U$2.PA2/SCK
- removed net N$31: J2.2, U$2.PA3/*SS
- removed net N$32: R3.1, U$2.VSENSE
- removed net N$37: C10.1, U$2.TSUP, X2-1.S
- removed net N$38: U$2.VTEMP, X2-2.S
- removed net N$4: J1.5, U$1.PA0/MISO
- removed net N$40: JP29.2, SV4.3, U$2.*RESET
- removed net N$41: R6.1, U$2.ISENSEH
- removed net N$42: C6.1, U$2.VDDA
- removed net N$43: R5.1, U$2.ISENSEL
- removed net N$44: C8.1, U$2.VDDD2D, U$2.VDDH
- removed net N$45: R10.1, U$1.ISENSEH
- removed net N$46: R9.1, U$1.ISENSEL
- removed net N$47: C1.1, U$1.VDDA
- removed net N$5: J1.4, U$1.PA1/MOSI
- removed net N$6: J1.3, U$1.PA2/SCK
- removed net N$7: J1.2, U$1.PA3/*SS
- removed net N$73: LED7.C, R36.2
- removed net N$79: J3.5, U$3.PA0/MISO
- removed net N$8: C4.1, U$1.TSUP, X1-1.S
- removed net N$9: JP29.1, U$2.*RESET_A
- removed net VDDX: C2.1, R12.2, SV3.1, U$1.VDDRX, U$1.VDDX
- removed net VDDXB: C7.1, R22.2, SV4.1, U$2.VDDRX, U$2.VDDX
- removed net VDDXC: C13.1, R23.2, SV5.1, U$3.VDDD2D, U$3.VDDH
- removed net VSUP: JP21.2, U$1.VSUP
- net 5V_SUPERVISED: no longer C14.1, C5.1, C86.1, C9.1, JP21.1, JP23.1, JP25.1, R26.2, R95.2, TP127.TP, TP128.TP, U10.INH, U10.VSUP
- net CON_MONA_+: no longer JP3.1
- net CON_MONA_-: no longer JP22.1, R2.2, R9.2
- net CON_MONB_+: no longer JP2.1, R10.2, R2.1
- net CON_MONB_-: no longer JP24.1, R4.2, R5.2, U18.EPAD
- net CON_MONC_+: no longer JP1.1, R4.1, R6.2
- net CON_MONC_-: no longer JP26.1, R37.2, R8.2
- net CON_MONC_SP: no longer R38.2, R8.1
- net GND: no longer C10.2, C12.2, C13.2, C14.2, C15.2, C2.2, C3.2, C4.2, C5.2, C7.2, C8.2, C9.2, JP22.3, JP24.3, JP26.3, R26.1, R27.2, R36.1, R39.1, R92.1, SV3.5, SV4.5, SV5.5, U$1.DGND, U$1.DGND1, U$1.GNDSUB, U$1.GNDSUB1, U$1.GNDSUB2, U$1.GNDSUB3, U$1.TEST, U$1.VSSD2D, U$1.VSSRX, U$2.DGND, U$2.DGND1, U$2.GNDSUB, U$2.GNDSUB1, U$2.GNDSUB2, U$2.GNDSUB3, U$2.TEST, U$2.VSSD2D, U$2.VSSRX, U$3.DGND, U$3.DGND1, U$3.GNDSUB, U$3.GNDSUB1, U$3.GNDSUB2, U$3.GNDSUB3, U$3.TEST, U$3.VSSD2D, U$3.VSSRX, U3.EPAD, U4.EPAD, U5.4, U7.EPAD
- net MCU_IO_RALAYA: no longer U$1.PA4
- net MCU_IO_RALAYB: no longer U$2.PA4
- net MCU_IO_RALAYC: no longer U$3.PA4
- net MCU_LINTX: no longer U10.TXD
- net MCU_LIN_EN: no longer U10.EN
- net MCU__LINRX: no longer U10.RXD
- net N$167: now also U5.4
- net N$169: now also U4.EPAD
- net N$2: now also JP88.2; no longer JP30.2, SV5.3, U$3.*RESET
- net N$25: now also U18.EPAD
- net N$261: now also U3.EPAD
- net N$262: now also U7.EPAD
- net VOLTAGEJMP_+_TO_INPUT_VREG: no longer JP88.2
Other:
- note removed: "Battery Monitor B"
- note removed: "Battery Monitoring Block A"
- note removed: "Battery Monitoring Block C"
- note removed: "TEMP CONNECTOR"
