File: Electrical Schematics/Version3/Schematics/boardv2a.sch (EAGLE design)
At the start: 629 parts, among them IC1 MCP41HVX1ST, IC2 ADUM4160BRW, IC3 SE555D, IC5 74LVC1G04DBV, IC6 74LVC1G04DBV, IC7 4030D, K1 G5V-2, K2 CP1SA-12V, Q1 IRLML2060TRPBFBSS123LT1G, Q10 IRLML2060TRPBFBSS123LT1G, Q11 IRLML2060TRPBFBSS123LT1G, Q12 IRLML2060TRPBFBSS123LT1G, Q13 IRLML2060TRPBFBSS123LT1G, Q17 IRLML2060TRPBFBSS123LT1G, Q18 MOSFET-PCHANNEL, Q19 IRLML2060TRPBFBSS123LT1G, Q2 IRLML2060TRPBFBSS123LT1G, Q3 IRLML2060TRPBFBSS123LT1G, Q4 MOSFET-PCHANNEL, Q5 MOSFET-PCHANNEL, Q6 IRLML2060TRPBFBSS123LT1G, Q7 ASFL1, Q8 IRLML2060TRPBFBSS123LT1G, Q9 IRLML2060TRPBFBSS123LT1G, U1 CP2130-GM, U10 SN65HVDA100-Q1_D_8, U11 ADUM3442CRWZ, U12 ADUM3442CRWZ, U13 ADUM3442CRWZ, U14 ADUM3442CRWZ, U15 ADUM3442CRWZ, U16 ADUM3442CRWZ, U17 ADUM3442CRWZ, U18 LM1085_KTT_3, U19 ADUM3442CRWZ, U2 TMS570LS0432_PZ_100, U20 ADUM3442CRWZ, U3 LM1085_KTT_3, U4 LM1085_KTT_3, U5 LM1084_KTT_3, U6 TPS3514_D_14, U7 LM1085_KTT_3, U9 ADUM3442CRWZ, X4 5566-4

Commit message: Motor Driver and MCU changes
Parts:
- added Q14: (no value), SparkFun-DiscreteSemi:IRF7509
- added R43, R44, R45, R46, R48: 1k, SparkFun-Passives:RESISTOR0603-RES
- added R47, R49: 3.3k, SparkFun-Passives:RESISTOR0603-RES
- added U$40: VNH3SP30, IGVC_vnh3sp30_motordriver:VNH3SP30
Connections:
- new net MCU_FPGA_RES1: TP61.TP, U$32G$1.P$1
- new net N$124: R47.1, R48.1, U$40.ENA/DIAGA
- new net N$134: R46.1, R49.1, U$40.ENB/DIAGB
- new net N$143: R44.1, U$40.PWM
- new net N$161: R45.2, U$40.INB
- new net N$168: R43.2, U$40.INA
- new net STEERCTRL_MCU_N2HET(0): R44.2
- new net STEERCTRL_MCU_N2HET(2): R43.1
- new net STEERCTRL_MCU_N2HET(4): R45.1
- new net STEERCTRL_MCU_N2HET(6): R48.2
- new net STEERCTRL_MCU_N2HET(8): R46.2
- new net VCC: Q14NMOS.G, R47.2, R49.2, U$40.VCC_1, U$40.VCC_2, U$40.VCC_3
- net FPGA_MCU_RES1: no longer TP61.TP, U$32G$1.P$1
- net GND: now also Q14NMOS.S, U$40.GNDA_1, U$40.GNDA_2, U$40.GNDA_3, U$40.GNDB_1, U$40.GNDB_2, U$40.GNDB_3
- net MCU_+1.2V: now also U2.VCC_4, U2.VCC_5, U2.VCC_6, U2.VCC_7
- net MCU_+3.3V: no longer U2.VCCIO_5, U2.VCCIO_6, U2.VCCIO_7, U2.VCCIO_8
